File: BMS-Master/Power.sch (KiCad schematic (older format))
At the start: 33 parts

Commit message: schematics
Parts:
- added C? (x2): 0.1u, Capacitors_SMD:C_0805_HandSoldering, symbol Device:C
- added C?: 1u, Capacitors_SMD:C_0805_HandSoldering, symbol Device:C
- added C?: 4.7u, Capacitors_SMD:C_1206_HandSoldering, symbol Device:C
- added C? (x4): 0.01u, Capacitors_SMD:C_0603_HandSoldering, symbol Device:C
- added C?: 22u, Capacitors_SMD:C_1812_HandSoldering, symbol Device:C
- added C?: 4.7u, symbol Device:C
- added C?: 330p, symbol Device:C
- added C?: 2.2u, symbol Device:C
- added D?: B180-13-F, Diodes_SMD:D_SMA, symbol Device:D_Zener
- added L?: 220u, symbol pspice:INDUCTOR
- added R?: 174k, Resistors_SMD:R_0603_HandSoldering, symbol Device:R
- added R?: 665k, Resistors_SMD:R_0603_HandSoldering, symbol Device:R
- added R?: 1.2k, Resistors_SMD:R_0603_HandSoldering, symbol Device:R
- added R? (x3): 10k, Resistors_SMD:R_0603_HandSoldering, symbol Device:R
- added R?: 1.5, Resistors_SMD:R_0805_HandSoldering, symbol Device:R
- added U?: LM5008MM, Package_SO:MSOP-8_3x3mm_P0.65mm, symbol Regulator_Switching:LM5008MM
- added U?: LP2985-3.3, Package_TO_SOT_SMD:SOT-23-5, symbol Regulator_Linear:LP2985-3.3
Connections:
- net BAT16: now also C?.1, C?.1, R?.1, U?.8 (VIN)
- net GND: now also C?.1, C?.2, C?.2, C?.2, C?.2, C?.2, D?.2 (A), R?.1, R?.2, U?.2 (GND), U?.4 (RTN)
- new net: R?.2, U?.6 (RON/SD)
- new net: R?.1, U?.3 (RCL)
- new net: C?.1, U?.7 (VCC)
- new net: C?.1, D?.1 (K), L?.1, R?.2, U?.1 (SW)
- new net: C?.2, U?.2 (BST)
- new net: C?.2, C?.2, R?.1
- new net: C?.1, C?.1, C?.2, R?.1, R?.2, U?.5 (FB)
- new net: C?.1, R?.1
- new net: C?.1, R?.1, U?.3 (ON/~OFF~)
- new net: C?.2, C?.2
- new net +3V3: C?.1, U?.5 (VOUT)
- new net +5V: C?.1, C?.1, C?.2, L?.2, R?.2, R?.2, R?.2, U?.1 (VIN)

Commit message: schematic update
Parts:
- removed C? (x2): 0.1u, Capacitors_SMD:C_0805_HandSoldering, symbol Device:C
- removed C?: 1u, Capacitors_SMD:C_0805_HandSoldering, symbol Device:C
- removed C? (x2): 4.7u, Capacitors_SMD:C_1206_HandSoldering, symbol Device:C
- removed C? (x4): 0.01u, Capacitors_SMD:C_0603_HandSoldering, symbol Device:C
- removed C?: 22u, Capacitors_SMD:C_1812_HandSoldering, symbol Device:C
- removed C?: 4.7u, symbol Device:C
- removed C?: 330p, symbol Device:C
- removed C?: 2.2u, symbol Device:C
- removed C? (x8): 0.1u, Capacitors_SMD:C_0603_HandSoldering, symbol Device:C
- removed C?: 1u, Capacitors_SMD:C_1206_HandSoldering, symbol Device:C
- removed D?: B180-13-F, Diodes_SMD:D_SMA, symbol Device:D_Zener
- removed J?: Conn_02x08_Counter_Clockwise, Pin_Headers:Pin_Header_Angled_2x08_Pitch2.54mm, symbol Connector_Generic:Conn_02x08_Counter_Clockwise
- removed L?: 220u, symbol pspice:INDUCTOR
- removed Q?: ZXTN4004KTC, TO_SOT_Packages_SMD:TO-252-2, symbol Device:Q_NPN_BCE
- removed R?: 174k, Resistors_SMD:R_0603_HandSoldering, symbol Device:R
- removed R?: 665k, Resistors_SMD:R_0603_HandSoldering, symbol Device:R
- removed R?: 1.2k, Resistors_SMD:R_0603_HandSoldering, symbol Device:R
- removed R? (x11): 10k, Resistors_SMD:R_0603_HandSoldering, symbol Device:R
- removed R?: 1.5, Resistors_SMD:R_0805_HandSoldering, symbol Device:R
- removed R? (x8): 10, Resistors_SMD:R_0603_HandSoldering, symbol Device:R
- removed R? (x2): 200, Resistors_SMD:R_2512, symbol Device:R
- removed R?: 0.39, Resistors_SMD:R_0603_HandSoldering, symbol Device:R
- removed R? (x2): 1, Resistors_SMD:R_0603_HandSoldering, symbol Device:R
- removed U?: LM5008MM, Package_SO:MSOP-8_3x3mm_P0.65mm, symbol Regulator_Switching:LM5008MM
- removed U?: LP2985-3.3, Package_TO_SOT_SMD:SOT-23-5, symbol Regulator_Linear:LP2985-3.3
- added C?: 1u, Capacitors_SMD:C_1206_HandSoldering, symbol Device:C
- added C? (x2): 4.7u, Capacitors_SMD:C_1206_HandSoldering, symbol Device:C
- added C? (x2): 0.1u, Capacitors_SMD:C_0805_HandSoldering, symbol Device:C
- added C?: 1u, Capacitors_SMD:C_0805_HandSoldering, symbol Device:C
- added C? (x4): 0.01u, Capacitors_SMD:C_0603_HandSoldering, symbol Device:C
- added C?: 22u, Capacitors_SMD:C_1812_HandSoldering, symbol Device:C
- added C?: 4.7u, symbol Device:C
- added C?: 330p, symbol Device:C
- added C?: 2.2u, symbol Device:C
- added D?: B180-13-F, Diodes_SMD:D_SMA, symbol Device:D_Zener
- added JP?: Jumper_NC_Dual, symbol Device:Jumper_NC_Dual
- added L?: 220u, symbol pspice:INDUCTOR
- added Q?: ZXTN4004KTC, TO_SOT_Packages_SMD:TO-252-2, symbol Device:Q_NPN_BCE
- added R? (x2): 200, Resistors_SMD:R_2512, symbol Device:R
- added R?: 0.39, Resistors_SMD:R_0603_HandSoldering, symbol Device:R
- added R? (x2): 1, Resistors_SMD:R_0603_HandSoldering, symbol Device:R
- added R?: 174k, Resistors_SMD:R_0603_HandSoldering, symbol Device:R
- added R?: 665k, Resistors_SMD:R_0603_HandSoldering, symbol Device:R
- added R?: 1.2k, Resistors_SMD:R_0603_HandSoldering, symbol Device:R
- added R? (x3): 10k, Resistors_SMD:R_0603_HandSoldering, symbol Device:R
- added R?: 1.5, Resistors_SMD:R_0805_HandSoldering, symbol Device:R
- added U?: LM5008MM, Package_SO:MSOP-8_3x3mm_P0.65mm, symbol Regulator_Switching:LM5008MM
- added U?: LP2985-3.3, Package_TO_SOT_SMD:SOT-23-5, symbol Regulator_Linear:LP2985-3.3
Connections:
- net +3V3: now also C?.1, U?.5 (VOUT)
- net +5V: now also C?.1, C?.1, C?.2, L?.2, R?.2, R?.2, R?.2, U?.1 (VIN)
- net BAT16: now also JP?.1, R?.2
- net GND: now also C?.1, C?.2, C?.2, C?.2, C?.2, C?.2, C?.2, C?.2, D?.2 (A), R?.1, R?.2, U?.2 (GND), U?.4 (RTN)
- net NPN_BASE: now also Q?.1 (B)
- net VDIG: now also R?.2
- net VIO: now also R?.2
- net VP1: now also Q?.3 (E), R?.1, R?.1, R?.1
- new net: C?.1, C?.1, JP?.2, R?.1, U?.8 (VIN)
- new net: R?.1, R?.2
- new net: C?.1, Q?.2 (C), R?.1
- new net: C?.1, R?.2
- new net: C?.1, D?.1 (K), L?.1, R?.2, U?.1 (SW)
- new net: C?.2, U?.2 (BST)
- new net: R?.1, U?.3 (RCL)
- new net: C?.1, C?.1, C?.2, R?.1, R?.2, U?.5 (FB)
- new net: R?.2, U?.6 (RON/SD)
- new net: C?.1, U?.7 (VCC)
- new net: C?.1, R?.1, U?.3 (ON/~OFF~)
- new net: C?.2, C?.2, R?.1
- new net: C?.1, R?.1
- new net: C?.2, C?.2
- new net +12V: JP?.3
