File: V0.2-LTC6813/BMS-Master/Connector.sch (KiCad schematic (older format))
At the start: 115 parts

Commit message: V0.2 LTC6813 block
Parts:
- C? (x16): symbol Device:C -> BMS-Master-rescue:C-Device
- D? (x17): symbol Device:D_Zener -> BMS-Master-rescue:D_Zener-Device
- J?: symbol Connector_Generic:Conn_01x22 -> BMS-Master-rescue:Conn_01x22-Connector_Generic
- Q? (x16): symbol Device:Q_NMOS_GSD -> BMS-Master-rescue:Q_NMOS_GSD-Device
- R? (x65): symbol Device:R -> BMS-Master-rescue:R-Device
