File: V0.2-LTC6813/BMS-Master/bq76PL455A-Q1.sch (KiCad schematic (older format))
At the start: 54 parts

Commit message: V0.2 LTC6813 block
Parts:
- C? (x23): symbol Device:C -> BMS-Master-rescue:C-Device
- D? (x4): symbol Diode:1N4148 -> BMS-Master-rescue:1N4148-Diode
- D? (x8): symbol Device:D_Zener -> BMS-Master-rescue:D_Zener-Device
- J? (x2): symbol Connector_Generic:Conn_01x04 -> BMS-Master-rescue:Conn_01x04-Connector_Generic
- R? (x14): symbol Device:R -> BMS-Master-rescue:R-Device
