File: V0.2-LTC6813/BMS-Master/BMS-Master.sch (KiCad schematic (older format))
At the start: 22 parts

Commit message: V0.2 LTC6813 block
Parts:
- BZ?: symbol Device:Buzzer -> BMS-Master-rescue:Buzzer-Device
- D?: symbol Diode:MBR0540 -> BMS-Master-rescue:MBR0540-Diode
- D? (x2): symbol Device:LED -> BMS-Master-rescue:LED-Device
- F?: symbol Device:Fuse -> BMS-Master-rescue:Fuse-Device
- J?: symbol Connector_Specialized:USB_B_Micro -> BMS-Master-rescue:USB_B_Micro-Connector_Specialized
- J? (x2): symbol Connector_Generic:Conn_01x04 -> BMS-Master-rescue:Conn_01x04-Connector_Generic
- J? (x4): symbol Connector_Generic:Conn_01x02 -> BMS-Master-rescue:Conn_01x02-Connector_Generic
- J?: symbol Connector_Generic:Conn_01x05 -> BMS-Master-rescue:Conn_01x05-Connector_Generic
- J? (x2): symbol Connector_Generic:Conn_01x01 -> BMS-Master-rescue:Conn_01x01-Connector_Generic
- Q?: symbol Transistor_FET:BSS138 -> BMS-Master-rescue:BSS138-Transistor_FET
- R? (x6): symbol Device:R -> BMS-Master-rescue:R-Device
Changed lines of the file:
@@
-$EndSheet
-$Sheet
-S 4900 2250 1800 4200
-U 5A8ACA42
-F0 "bq76PL455A-Q1" 50
-F1 "bq76PL455A-Q1.sch" 50
-F2 "VSENSE14" I L 4900 3500 50
-F3 "EQ14" O L 4900 3600 50
-F4 "VSENSE13" I L 4900 3700 50
-F5 "EQ13" O L 4900 3800 50
-F6 "VSENSE12" I L 4900 3900 50
-F7 "EQ12" O L 4900 4000 50
-F8 "VSENSE11" I L 4900 4100 50
-F9 "EQ11" O L 4900 4200 50
-F10 "VSENSE10" I L 4900 4300 50
-F11 "EQ10" O L 4900 4400 50
-F12 "EQ15" O L 4900 3400 50
-F13 "VSENSE15" I L 4900 3300 50
-F14 "EQ16" O L 4900 3200 50
-F15 "VSENSE16" I L 4900 3100 50
-F16 "BAT16" B L 4900 2400 50
-F17 "NPN_BASE" B R 6700 3850 50
-F18 "VP1" B R 6700 3650 50
-F19 "AUX0" I R 6700 3300 50
-F20 "AUX1" I R 6700 3200 50
-F21 "AUX2" I R 6700 3100 50
-F22 "AUX3" I R 6700 3000 50
-F23 "AUX4" I R 6700 2900 50
-F24 "AUX5" I R 6700 2800 50
-F25 "AUX6" I R 6700 2700 50
-F26 "AUX7" I R 6700 2600 50
-F27 "VSENSE9" I L 4900 4500 50
-F28 "EQ9" O L 4900 4600 50
-F29 "VSENSE8" I L 4900 4700 50
-F30 "EQ8" O L 4900 4800 50
-F31 "VSENSE7" I L 4900 4900 50
-F32 "EQ7" O L 4900 5000 50
-F33 "VSENSE6" I L 4900 5100 50
-F34 "EQ6" O L 4900 5200 50
-F35 "VSENSE5" I L 4900 5300 50
-F36 "EQ5" O L 4900 5400 50
-F37 "VSENSE4" I L 4900 5500 50
-F38 "EQ4" O L 4900 5600 50
-F39 "VSENSE3" I L 4900 5700 50
-F40 "EQ3" O L 4900 5800 50
-F41 "VSENSE2" I L 4900 5900 50
-F42 "EQ2" O L 4900 6000 50
-F43 "VSENSE1" I L 4900 6100 50
-F44 "EQ1" O L 4900 6200 50
-F45 "VSENSE0" I L 4900 6300 50
-F46 "VDIG" B R 6700 3750 50
-F47 "VIO" B R 6700 3550 50
-F48 "FAULT_N" O R 6700 5300 50
-F49 "RX" I R 6700 5150 50
-F50 "TX" O R 6700 5050 50
-F51 "GPIO0" B R 6700 6250 50
-F52 "GPIO1" B R 6700 6150 50
-F53 "GPIO2" B R 6700 6050 50
-F54 "GPIO3" B R 6700 5950 50
-F55 "GPIO4" B R 6700 5850 50
-F56 "GPIO5" B R 6700 5750 50
-F57 "BAT0" B L 4900 2500 50
-F58 "WAKEUP" O R 6700 5400 50
 $EndSheet
 $Sheet
@@
 $EndSheet
 $Comp
-L Connector_Specialized:USB_B_Micro J?
+L BMS-Master-rescue:USB_B_Micro-Connector_Specialized J?
 U 1 1 5A966632
 P 10850 7300
@@
 $EndComp
 $Comp
-L power:GND #PWR?
+L BMS-Master-rescue:GND-power #PWR?
 U 1 1 5A969833
 P 10900 7750
@@
 	9800 8550 9550 8550
 $Comp
-L Connector_Generic:Conn_01x04 J?
+L BMS-Master-rescue:Conn_01x04-Connector_Generic J?
 U 1 1 5A98621E
 P 11750 8500
@@
 	11400 8700 11550 8700
 $Comp
-L power:+5V #PWR?
+L BMS-Master-rescue:+5V-power #PWR?
 U 1 1 5A9B2FE8
 P 10050 7050
@@
 $EndComp
 $Comp
-L Diode:MBR0540 D?
+L BMS-Master-rescue:MBR0540-Diode D?
 U 1 1 5A9B3071
 P 10300 7100
@@
 	10450 7100 10550 7100
 $Comp
-L Device:R R?
+L BMS-Master-rescue:R-Device R?
 U 1 1 5A9B7063
 P 9900 7300
@@
 $EndComp
 $Comp
-L Device:R R?
+L BMS-Master-rescue:R-Device R?
 U 1 1 5A9B70E5
 P 9900 7400
@@
 	6700 5750 8000 5750
 $Comp
-L Device:LED D?
+L BMS-Master-rescue:LED-Device D?
 U 1 1 5ABAB322
 P 6700 9900
@@
 $EndComp
 $Comp
-L Device:R R?
+L BMS-Master-rescue:R-Device R?
 U 1 1 5ABAB411
 P 6700 9500
@@
 $EndComp
 $Comp
-L Device:R R?
+L BMS-Master-rescue:R-Device R?
 U 1 1 5ABB20CA
 P 5950 9500
@@
 $EndComp
 $Comp
-L Device:LED D?
+L BMS-Master-rescue:LED-Device D?
 U 1 1 5ABB20FE
 P 5950 9900
@@
 	6700 9750 6700 9650
 $Comp
-L power:GND #PWR?
+L BMS-Master-rescue:GND-power #PWR?
 U 1 1 5ABB698D
 P 5950 10150
@@
 $EndComp
 $Comp
-L power:GND #PWR?
+L BMS-Master-rescue:GND-power #PWR?
 U 1 1 5ABB69D7
 P 6700 10150
@@
 	6700 9150 8000 9150
 $Comp
-L power:+3.3V #PWR?
+L BMS-Master-rescue:+3.3V-power #PWR?
 U 1 1 5ABBDFF3
 P 5950 9250
@@
 Status LED
 $Comp
-L Device:R R?
+L BMS-Master-rescue:R-Device R?
 U 1 1 5ABC0C8F
 P 10100 9550
@@
 $EndComp
 $Comp
-L power:GND #PWR?
+L BMS-Master-rescue:GND-power #PWR?
 U 1 1 5ABC0CBB
 P 10100 9850
@@
 	10100 9250 10100 9400
 $Comp
-L Device:Buzzer BZ?
+L BMS-Master-rescue:Buzzer-Device BZ?
 U 1 1 5ABC5C93
 P 14100 8050
@@
 $EndComp
 $Comp
-L power:+3.3V #PWR?
+L BMS-Master-rescue:+3.3V-power #PWR?
 U 1 1 5ABC5D22
 P 14000 7800
@@
 	14000 7800 14000 7950
 $Comp
-L power:GND #PWR?
+L BMS-Master-rescue:GND-power #PWR?
 U 1 1 5ABCABB8
 P 14000 9050
@@
 $EndComp
 $Comp
-L Transistor_FET:BSS138 Q?
+L BMS-Master-rescue:BSS138-Transistor_FET Q?
 U 1 1 5ABCAC4F
 P 13900 8550
@@
 $EndSheet
 $Comp
-L Connector_Generic:Conn_01x05 J?
+L BMS-Master-rescue:Conn_01x05-Connector_Generic J?
 U 1 1 5ABE6776
 P 12250 4500
@@
 Power
 $Comp
-L power:+3.3V #PWR?
+L BMS-Master-rescue:+3.3V-power #PWR?
 U 1 1 5ABE6960
 P 11800 4250
@@
 $EndComp
 $Comp
-L Device:R R?
+L BMS-Master-rescue:R-Device R?
 U 1 1 5ABEC8F7
 P 11700 4600
@@
 	11550 4600 11400 4600
 $Comp
-L power:GND #PWR?
+L BMS-Master-rescue:GND-power #PWR?
 U 1 1 5ABF492B
 P 11950 4800
@@
 	3700 2500 4900 2500
 $Comp
-L Connector_Generic:Conn_01x04 J?
+L BMS-Master-rescue:Conn_01x04-Connector_Generic J?
 U 1 1 5AB6317C
 P 4400 8650
@@
 $EndComp
 $Comp
-L power:+5V #PWR?
+L BMS-Master-rescue:+5V-power #PWR?
 U 1 1 5AB69DA9
 P 4650 8500
@@
 	4650 8550 4650 8500
 $Comp
-L power:GND #PWR?
+L BMS-Master-rescue:GND-power #PWR?
 U 1 1 5AB6D538
 P 4700 8900
@@
 	10050 5450 9550 5450
 $Comp
-L Connector_Generic:Conn_01x02 J?
+L BMS-Master-rescue:Conn_01x02-Connector_Generic J?
 U 1 1 5AB7AB5E
 P 13700 3600
@@
 $EndComp
 $Comp
-L power:GND #PWR?
+L BMS-Master-rescue:GND-power #PWR?
 U 1 1 5AB80FEA
 P 13450 3750
@@
 	13450 3700 13500 3700
 $Comp
-L Connector_Generic:Conn_01x02 J?
+L BMS-Master-rescue:Conn_01x02-Connector_Generic J?
 U 1 1 5ABBEF45
 P 13050 5050
@@
 $EndComp
 $Comp
-L Connector_Generic:Conn_01x02 J?
+L BMS-Master-rescue:Conn_01x02-Connector_Generic J?
 U 1 1 5ABBF131
 P 13050 5350
@@
 $EndComp
 $Comp
-L Connector_Generic:Conn_01x02 J?
+L BMS-Master-rescue:Conn_01x02-Connector_Generic J?
 U 1 1 5ABBF293
 P 13050 5650
@@
 $EndComp
 $Comp
-L power:GND #PWR?
+L BMS-Master-rescue:GND-power #PWR?
 U 1 1 5ABBF581
 P 12550 5850
@@
 	12250 5650 12850 5650
 $Comp
-L Connector_Generic:Conn_01x01 J?
+L BMS-Master-rescue:Conn_01x01-Connector_Generic J?
 U 1 1 5AC75917
 P 12250 2600
@@
 $EndComp
 $Comp
-L Connector_Generic:Conn_01x01 J?
+L BMS-Master-rescue:Conn_01x01-Connector_Generic J?
 U 1 1 5AC7F25B
 P 12250 2900
@@
 	11250 3600 12550 3600
 $Comp
-L Device:Fuse F?
+L BMS-Master-rescue:Fuse-Device F?
 U 1 1 5ACF057B
 P 13100 3600
@@
 	12950 3600 12550 3600
 Connection ~ 12550 3600
+$Sheet
+S 4900 2200 1800 4500
+U 5B4A196B
+F0 "ltc6813" 50
+F1 "ltc6813.sch" 50
+$EndSheet
 $EndSCHEMATC

Commit message: V0.2 update
Connections:
- wire segments 147 -> 112
Changed lines of the file:
@@
 $Descr A3 16535 11693
 encoding utf-8
-Sheet 1 8
+Sheet 1 25
 Title "BMS-Master"
 Date ""
@@
 Comment4 ""
 $EndDescr
-$Sheet
-S 2450 2150 1250 4300
-U 5A8ACA25
-F0 "connector" 50
-F1 "Connector.sch" 50
-F2 "VSENSE16" O R 3700 3100 50
-F3 "VSENSE15" O R 3700 3300 50
-F4 "EQ16" I R 3700 3200 50
-F5 "VSENSE14" O R 3700 3500 50
-F6 "EQ15" I R 3700 3400 50
-F7 "VSENSE13" O R 3700 3700 50
-F8 "EQ14" I R 3700 3600 50
-F9 "VSENSE12" O R 3700 3900 50
-F10 "EQ13" I R 3700 3800 50
-F11 "VSENSE11" O R 3700 4100 50
-F12 "EQ12" I R 3700 4000 50
-F13 "VSENSE10" O R 3700 4300 50
-F14 "EQ11" I R 3700 4200 50
-F15 "VSENSE9" O R 3700 4500 50
-F16 "EQ10" I R 3700 4400 50
-F17 "VSENSE8" O R 3700 4700 50
-F18 "EQ9" I R 3700 4600 50
-F19 "VSENSE7" O R 3700 4900 50
-F20 "EQ8" I R 3700 4800 50
-F21 "VSENSE6" O R 3700 5100 50
-F22 "EQ7" I R 3700 5000 50
-F23 "VSENSE5" O R 3700 5300 50
-F24 "EQ6" I R 3700 5200 50
-F25 "VSENSE4" O R 3700 5500 50
-F26 "EQ5" I R 3700 5400 50
-F27 "VSENSE3" O R 3700 5700 50
-F28 "EQ4" I R 3700 5600 50
-F29 "VSENSE2" O R 3700 5900 50
-F30 "EQ3" I R 3700 5800 50
-F31 "VSENSE1" O R 3700 6100 50
-F32 "EQ2" I R 3700 6000 50
-F33 "VSENSE0" O R 3700 6300 50
-F34 "EQ1" I R 3700 6200 50
-F35 "BAT16" B R 3700 2400 50
-F36 "BAT0" B R 3700 2500 50
-$EndSheet
 $Sheet
 S 7250 2250 1150 1150
@@
 $EndSheet
 Wire Wire Line
-	3700 3100 4900 3100
-Wire Wire Line
-	3700 3200 4900 3200
-Wire Wire Line
-	3700 3300 4900 3300
-Wire Wire Line
-	3700 3400 4900 3400
-Wire Wire Line
-	3700 3500 4900 3500
-Wire Wire Line
-	4900 3600 3700 3600
-Wire Wire Line
-	3700 3700 4900 3700
-Wire Wire Line
-	4900 3800 3700 3800
-Wire Wire Line
-	3700 3900 4900 3900
-Wire Wire Line
-	4900 4000 3700 4000
-Wire Wire Line
-	3700 4100 4900 4100
-Wire Wire Line
-	4900 4200 3700 4200
-Wire Wire Line
-	3700 4300 4900 4300
-Wire Wire Line
-	4900 4400 3700 4400
-Wire Wire Line
-	3700 4500 4900 4500
-Wire Wire Line
-	4900 4600 3700 4600
-Wire Wire Line
-	3700 4700 4900 4700
-Wire Wire Line
-	4900 4800 3700 4800
-Wire Wire Line
-	3700 4900 4900 4900
-Wire Wire Line
-	4900 5000 3700 5000
-Wire Wire Line
-	3700 5100 4900 5100
-Wire Wire Line
-	4900 5200 3700 5200
-Wire Wire Line
-	3700 5300 4900 5300
-Wire Wire Line
-	4900 5400 3700 5400
-Wire Wire Line
-	3700 5500 4900 5500
-Wire Wire Line
-	4900 5600 3700 5600
-Wire Wire Line
-	3700 5700 4900 5700
-Wire Wire Line
-	4900 5800 3700 5800
-Wire Wire Line
-	3700 5900 4900 5900
-Wire Wire Line
-	4900 6000 3700 6000
-Wire Wire Line
-	3700 6100 4900 6100
-Wire Wire Line
-	4900 6200 3700 6200
-Wire Wire Line
-	3700 6300 4900 6300
-Wire Wire Line
-	3700 2400 4650 2400
-Wire Wire Line
 	6700 3300 7250 3300
 Wire Wire Line
@@
 Wire Wire Line
 	7250 2600 6700 2600
-Wire Wire Line
-	4650 2000 4650 2400
-Connection ~ 4650 2400
-Wire Wire Line
-	4650 2400 4900 2400
 Wire Wire Line
 	6700 5050 8000 5050
@@
 Wire Wire Line
 	11800 4500 12050 4500
-Wire Wire Line
-	3700 2500 4900 2500
 $Comp
 L BMS-Master-rescue:Conn_01x04-Connector_Generic J?
@@
 F0 "power" 50
 F1 "power.sch" 50
-F2 "BAT16" I L 10050 2450 50
+F2 "BAT+" I L 10050 2450 50
 F3 "NPN_BASE" B L 10050 3850 50
 F4 "VP1" B L 10050 3650 50
@@
 Wire Wire Line
 	9800 2450 10050 2450
-Wire Wire Line
-	4650 2000 9800 2000
 Wire Wire Line
 	6700 3550 10050 3550
@@
 F0 "ltc6813" 50
 F1 "ltc6813.sch" 50
+F2 "MA" I L 4900 2850 50
+F3 "PA" I L 4900 3000 50
+F4 "MB" I L 4900 3200 50
+F5 "PB" I L 4900 3400 50
+F6 "BAT+" I L 4900 2400 50
 $EndSheet
+Wire Wire Line
+	4650 2000 9800 2000
+Wire Wire Line
+	4650 2000 4650 2400
+Wire Wire Line
+	4650 2400 4900 2400
 $EndSCHEMATC

Commit message: schematics 50% complete3d
Parts:
- removed D?: MBR0540, Diode_SMD:D_SOD-123, symbol BMS-Master-rescue:MBR0540-Diode
- removed J?: CANBUS, symbol BMS-Master-rescue:Conn_01x04-Connector_Generic
- removed Q?: BSS138, Package_TO_SOT_SMD:SOT-23, symbol BMS-Master-rescue:BSS138-Transistor_FET
- removed R? (x2): 22, Resistors_SMD:R_0603_HandSoldering, symbol BMS-Master-rescue:R-Device
- added DaisyChain: J?, symbol BMS-Master-rescue:Conn_01x02-Connector_Generic
- added J?: Conn_01x05-Connector_Generic, symbol BMS-Master-rescue:Conn_01x05-Connector_Generic
- added J?: Common, symbol BMS-Master-rescue:Conn_01x01-Connector_Generic
- added J?: Temperature, symbol Connector_Generic:Conn_02x09_Counter_Clockwise
- added J?: Cells, symbol Connector_Generic:Conn_01x19
- added Q?: BSS138, Package_TO_SOT_SMD:SOT-23, symbol Transistor_FET:BSS138
- added R?: 15, Resistors_SMD:R_2512_HandSoldering, symbol BMS-Master-rescue:R-Device
- J?: value +12V -> ExternalPower
Connections:
- wire segments 112 -> 157
- no-connect marks 1 -> 2
Other:
- moved on the sheet: BZ?, J?

Commit message: Schematics 75% completed
Connections:
- net GND: no longer J?.10 (Pin_10), J?.11 (Pin_11), J?.12 (Pin_12), J?.13 (Pin_13), J?.14 (Pin_14), J?.15 (Pin_15), J?.16 (Pin_16), J?.17 (Pin_17), J?.18 (Pin_18), R?.2
- net Power/Bat+: no longer J?.1 (Pin_1)
- net Power/Charge+: no longer J?.1 (Pin_1)
- net CurrentMonitor/IN renamed PowerMonitor/I
- new net GNDA: J?.10 (Pin_10), J?.11 (Pin_11), J?.12 (Pin_12), J?.13 (Pin_13), J?.14 (Pin_14), J?.15 (Pin_15), J?.16 (Pin_16), J?.17 (Pin_17), J?.18 (Pin_18), R?.2
Other:
- moved on the sheet: J?, R?

Commit message: Schematics 80% completed
Parts:
- removed R?: 15, Resistors_SMD:R_2512_HandSoldering, symbol BMS-Master-rescue:R-Device
- added J?: Discharge+, symbol BMS-Master-rescue:Conn_01x01-Connector_Generic
- added J?: Common, symbol BMS-Master-rescue:Conn_01x01-Connector_Generic
- added R?: 15, Resistors_SMD:R_2512_HandSoldering, symbol BMS-Master-rescue:R-Device
- J?: value Charge + -> Charge+
- J?: value Common -> BAT-
Connections:
- net GNDA: now also J?.1 (Pin_1), R?.1
- net MCU/PowerLED: no longer R?.2
- net PowerMonitor/Charge+: now reaches J?.1 (Pin_1)
- net PowerMonitor/BAT+: now reaches J?.1 (Pin_1)
- net Power/ExternalPower renamed PowerSupply/ExternalPower
- net Power/PushButton: no longer names the net of J?.2 (Pin_2)
- new net: J?.1 (Pin_1), R?.2
- new net PowerMonitor/Discharge+: J?.1 (Pin_1)
Other:
- moved on the sheet: BZ?, D?, DaisyChain, F?, J?, Q?, R?
