File: V0.2-LTC6813/BMS-Master/switches.sch (KiCad schematic (older format))
At the start: 15 parts

Commit message: V0.2 LTC6813 block
Parts:
- Q? (x3): symbol Transistor_FET:BSS138 -> BMS-Master-rescue:BSS138-Transistor_FET
- R? (x9): symbol Device:R -> BMS-Master-rescue:R-Device
- U? (x3): symbol Isolator:SFH617A-2X009T -> BMS-Master-rescue:SFH617A-2X009T-Isolator
Changed lines of the file:
@@
 Charge
 $Comp
-L Isolator:SFH617A-2X009T U?
+L BMS-Master-rescue:SFH617A-2X009T-Isolator U?
 U 1 1 5ACC44C1
 P 5150 1950
@@
 $EndComp
 $Comp
-L Isolator:SFH617A-2X009T U?
+L BMS-Master-rescue:SFH617A-2X009T-Isolator U?
 U 1 1 5ACC48D9
 P 5150 4150
@@
 $EndComp
 $Comp
-L Isolator:SFH617A-2X009T U?
+L BMS-Master-rescue:SFH617A-2X009T-Isolator U?
 U 1 1 5ACC490F
 P 5150 5600
@@
 Connection ~ 5850 4050
 $Comp
-L power:+3.3V #PWR?
+L BMS-Master-rescue:+3.3V-power #PWR?
 U 1 1 5ACFE468
 P 4550 1500
@@
 	4550 1850 4850 1850
 $Comp
-L power:+3.3V #PWR?
+L BMS-Master-rescue:+3.3V-power #PWR?
 U 1 1 5ACFE5C5
 P 4600 3850
@@
 	4600 4050 4850 4050
 $Comp
-L power:+3.3V #PWR?
+L BMS-Master-rescue:+3.3V-power #PWR?
 U 1 1 5ACFE760
 P 4550 5250
@@
 	4550 5500 4850 5500
 $Comp
-L Transistor_FET:BSS138 Q?
+L BMS-Master-rescue:BSS138-Transistor_FET Q?
 U 1 1 5AD010B8
 P 3900 2350
@@
 $EndComp
 $Comp
-L Device:R R?
+L BMS-Master-rescue:R-Device R?
 U 1 1 5AD011B7
 P 4350 2050
@@
 $EndComp
 $Comp
-L Device:R R?
+L BMS-Master-rescue:R-Device R?
 U 1 1 5AD01241
 P 2950 2350
@@
 $EndComp
 $Comp
-L Device:R R?
+L BMS-Master-rescue:R-Device R?
 U 1 1 5AD01290
 P 3400 2550
@@
 	2300 2350 2800 2350
 $Comp
-L power:GND #PWR?
+L BMS-Master-rescue:GND-power #PWR?
 U 1 1 5AD03C7A
 P 3750 2900
@@
 	4000 2050 4000 2150
 $Comp
-L Transistor_FET:BSS138 Q?
+L BMS-Master-rescue:BSS138-Transistor_FET Q?
 U 1 1 5AD06F84
 P 3900 4550
@@
 $EndComp
 $Comp
-L Device:R R?
+L BMS-Master-rescue:R-Device R?
 U 1 1 5AD06F8A
 P 4350 4250
@@
 $EndComp
 $Comp
-L Device:R R?
+L BMS-Master-rescue:R-Device R?
 U 1 1 5AD06F90
 P 2950 4550
@@
 $EndComp
 $Comp
-L Device:R R?
+L BMS-Master-rescue:R-Device R?
 U 1 1 5AD06F96
 P 3400 4750
@@
 	2300 4550 2800 4550
 $Comp
-L power:GND #PWR?
+L BMS-Master-rescue:GND-power #PWR?
 U 1 1 5AD06FA2
 P 3750 5100
@@
 	4000 4250 4000 4350
 $Comp
-L Transistor_FET:BSS138 Q?
+L BMS-Master-rescue:BSS138-Transistor_FET Q?
 U 1 1 5AD07A68
 P 4150 6000
@@
 $EndComp
 $Comp
-L Device:R R?
+L BMS-Master-rescue:R-Device R?
 U 1 1 5AD07A6E
 P 4600 5700
@@
 $EndComp
 $Comp
-L Device:R R?
+L BMS-Master-rescue:R-Device R?
 U 1 1 5AD07A74
 P 3200 6000
@@
 $EndComp
 $Comp
-L Device:R R?
+L BMS-Master-rescue:R-Device R?
 U 1 1 5AD07A7A
 P 3650 6200
@@
 	4250 5700 4450 5700
 $Comp
-L power:GND #PWR?
+L BMS-Master-rescue:GND-power #PWR?
 U 1 1 5AD07A86
 P 4000 6550

Commit message: Schematics 75% completed
Parts:
- removed R? (x3): 1k, Resistors_SMD:R_0603_HandSoldering, symbol BMS-Master-rescue:R-Device
- added C? (x3): 10n, symbol Device:C
- added C?: 2.2u, symbol Device:C
- added Q? (x2): BSS138, Package_TO_SOT_SMD:SOT-23, symbol Transistor_FET:BSS138
- added R?: 100, Resistors_SMD:R_0603_HandSoldering, symbol BMS-Master-rescue:R-Device
- added R? (x4): 10k, Resistors_SMD:R_0603_HandSoldering, symbol BMS-Master-rescue:R-Device
- added U?: BQ76200, symbol ENNOID:BQ76200
Connections:
- net +12V: no longer U?.4, U?.4
- net ChargeEnable: now also Q?.3 (D), R?.1; no longer R?.1
- net DischargeEnable: now also Q?.3 (D), R?.1; no longer R?.1
- net GND: now also C?.1, C?.1, C?.1, Q?.2 (S), Q?.2 (S), U?.9 (VSS)
- net PrechargeEnable: now also R?.1; no longer R?.1
- new net: R?.1, U?.12 (Discharge)
- new net: R?.1, U?.14 (Precharge)
- new net: R?.1, U?.16 (Charge)
- new net: C?.2, R?.1, U?.11 (Pack)
- new net: C?.1, U?.1 (VDDP)
- new net: R?.2, U?.4 (ChargeEnable)
- new net: R?.2, U?.5 (CP_Enable), U?.7 (PowerMonitorEnable)
- new net: R?.2, U?.6 (DischargeEnable)
- new net: R?.2, U?.8 (PrechargeEnable)
- new net Enable: R?.1
- new net Safety: Q?.1 (G), Q?.1 (G)
- new net V: C?.2, C?.2, C?.2, U?.2 (BAT)
- new net Vpack: R?.2
Other:
- moved on the sheet: Q?, R?, U?

Commit message: Schematics 80% completed
Parts:
- added C?: 100n, symbol Device:C
- added R?: 100, Resistors_SMD:R_0603_HandSoldering, symbol BMS-Master-rescue:R-Device
- added R?: 33k, Resistors_SMD:R_0603_HandSoldering, symbol BMS-Master-rescue:R-Device
- added R?: 2.2k, Resistors_SMD:R_0603_HandSoldering, symbol BMS-Master-rescue:R-Device
Connections:
- net GND: now also C?.1, R?.2
- net at U?.10 (PackDiv): now also R?.1
- net V: no longer names the net of C?.2, C?.2, C?.2, U?.2 (BAT)
- net V: now also R?.2
- new net Vbat: R?.1
- new net VoutSense: C?.2, R?.1, R?.2
Other:
- moved on the sheet: C?, R?
Changed lines of the file:
@@
 Vpack
 Text HLabel 4950 2000 0    50   Input ~ 0
-V
+Vbat
 Wire Wire Line
 	4950 2000 5300 2000
 Wire Wire Line
-	5300 2000 5300 3100
+	5300 2000 5300 2350
 $Comp
 L Device:C C?
@@
 L BMS-Master-rescue:R-Device R?
 U 1 1 5C2BC2E8
-P 10500 5300
-F 0 "R?" V 10707 5300 50  0000 C CNN
-F 1 "100" V 10616 5300 50  0000 C CNN
-F 2 "Resistors_SMD:R_0603_HandSoldering" V 10430 5300 50  0001 C CNN
-F 3 "~" H 10500 5300 50  0001 C CNN
-	1    10500 5300
+P 10650 5300
+F 0 "R?" V 10857 5300 50  0000 C CNN
+F 1 "100" V 10766 5300 50  0000 C CNN
+F 2 "Resistors_SMD:R_0603_HandSoldering" V 10580 5300 50  0001 C CNN
+F 3 "~" H 10650 5300 50  0001 C CNN
+	1    10650 5300
 	0    -1   -1   0
 $EndComp
 Wire Wire Line
-	10650 5300 10850 5300
-Wire Wire Line
-	8900 5300 10000 5300
+	10800 5300 10850 5300
 $Comp
 L Device:C C?
 U 1 1 5C2C3B76
-P 10000 5450
-F 0 "C?" H 9885 5359 50  0000 R CNN
-F 1 "10n" H 9885 5450 50  0000 R CNN
-F 2 "" H 10038 5300 50  0001 C CNN
-F 3 "~" H 10000 5450 50  0001 C CNN
-F 4 "100V" H 9885 5541 50  0000 R CNN "Voltage"
-	1    10000 5450
+P 10300 5450
+F 0 "C?" H 10185 5359 50  0000 R CNN
+F 1 "10n" H 10185 5450 50  0000 R CNN
+F 2 "" H 10338 5300 50  0001 C CNN
+F 3 "~" H 10300 5450 50  0001 C CNN
+F 4 "100V" H 10185 5541 50  0000 R CNN "Voltage"
+	1    10300 5450
 	-1   0    0    1
 $EndComp
-Connection ~ 10000 5300
-Wire Wire Line
-	10000 5300 10350 5300
 $Comp
 L BMS-Master-rescue:GND-power #PWR?
 U 1 1 5C2C40A6
-P 10000 5650
-F 0 "#PWR?" H 10000 5400 50  0001 C CNN
-F 1 "GND" H 10005 5477 50  0000 C CNN
-F 2 "" H 10000 5650 50  0001 C CNN
-F 3 "" H 10000 5650 50  0001 C CNN
-	1    10000 5650
+P 10300 5650
+F 0 "#PWR?" H 10300 5400 50  0001 C CNN
+F 1 "GND" H 10305 5477 50  0000 C CNN
+F 2 "" H 10300 5650 50  0001 C CNN
+F 3 "" H 10300 5650 50  0001 C CNN
+	1    10300 5650
 	1    0    0    -1
 $EndComp
 Wire Wire Line
-	10000 5600 10000 5650
+	10300 5600 10300 5650
+$Comp
+L BMS-Master-rescue:R-Device R?
+U 1 1 5C2CA2F9
+P 5300 2500
+F 0 "R?" V 5507 2500 50  0000 C CNN
+F 1 "100" V 5416 2500 50  0000 C CNN
+F 2 "Resistors_SMD:R_0603_HandSoldering" V 5230 2500 50  0001 C CNN
+F 3 "~" H 5300 2500 50  0001 C CNN
+	1    5300 2500
+	1    0    0    -1
+$EndComp
+Wire Wire Line
+	5300 2650 5300 3100
+Connection ~ 10300 5300
+Wire Wire Line
+	10300 5300 10500 5300
+Wire Wire Line
+	8900 5300 10300 5300
+$Comp
+L Device:C C?
+U 1 1 5C628F5F
+P 9950 6400
+F 0 "C?" H 9835 6309 50  0000 R CNN
+F 1 "100n" H 9835 6400 50  0000 R CNN
+F 2 "" H 9988 6250 50  0001 C CNN
+F 3 "~" H 9950 6400 50  0001 C CNN
+	1    9950 6400
+	-1   0    0    1
+$EndComp
+$Comp
+L BMS-Master-rescue:R-Device R?
+U 1 1 5C6297B1
+P 9150 5550
+F 0 "R?" V 9357 5550 50  0000 C CNN
+F 1 "33k" V 9266 5550 50  0000 C CNN
+F 2 "Resistors_SMD:R_0603_HandSoldering" V 9080 5550 50  0001 C CNN
+F 3 "~" H 9150 5550 50  0001 C CNN
+	1    9150 5550
+	0    -1   -1   0
+$EndComp
+Wire Wire Line
+	8900 5550 9000 5550
+Wire Wire Line
+	9300 5550 9500 5550
+$Comp
+L BMS-Master-rescue:R-Device R?
+U 1 1 5C62E63C
+P 9500 6400
+F 0 "R?" V 9707 6400 50  0000 C CNN
+F 1 "2.2k" V 9616 6400 50  0000 C CNN
+F 2 "Resistors_SMD:R_0603_HandSoldering" V 9430 6400 50  0001 C CNN
+F 3 "~" H 9500 6400 50  0001 C CNN
+	1    9500 6400
+	1    0    0    -1
+$EndComp
+$Comp
+L BMS-Master-rescue:GND-power #PWR?
+U 1 1 5C6339EA
+P 9500 7050
+F 0 "#PWR?" H 9500 6800 50  0001 C CNN
+F 1 "GND" H 9505 6877 50  0000 C CNN
+F 2 "" H 9500 7050 50  0001 C CNN
+F 3 "" H 9500 7050 50  0001 C CNN
+	1    9500 7050
+	1    0    0    -1
+$EndComp
+Wire Wire Line
+	9500 6550 9500 7050
+$Comp
+L BMS-Master-rescue:GND-power #PWR?
+U 1 1 5C636778
+P 9950 7050
+F 0 "#PWR?" H 9950 6800 50  0001 C CNN
+F 1 "GND" H 9955 6877 50  0000 C CNN
+F 2 "" H 9950 7050 50  0001 C CNN
+F 3 "" H 9950 7050 50  0001 C CNN
+	1    9950 7050
+	1    0    0    -1
+$EndComp
+Wire Wire Line
+	9950 6550 9950 7050
+Text HLabel 10150 6100 2    50   Input ~ 0
+VoutSense
+Wire Wire Line
+	9500 5550 9500 6100
+Wire Wire Line
+	9950 6250 9950 6100
+Wire Wire Line
+	9950 6100 9500 6100
+Connection ~ 9500 6100
+Wire Wire Line
+	9500 6100 9500 6250
+Wire Wire Line
+	9950 6100 10150 6100
+Connection ~ 9950 6100
 $EndSCHEMATC

Commit message: Schematics 90% completed
Parts:
- added TH?: Thermistor_NTC, symbol Device:Thermistor_NTC
Connections:
- net +12V: now also U?.4, U?.4
- net GND: now also TH?.1
- new net NTC_Switch: TH?.2
Changed lines of the file:
@@
 	9950 6100 10150 6100
 Connection ~ 9950 6100
+Text HLabel 14450 4300 2    50   Input ~ 0
++12V
+Text HLabel 14550 2350 2    50   Input ~ 0
++12V
+$Comp
+L Device:Thermistor_NTC TH?
+U 1 1 5C84F4B0
+P 3300 9350
+F 0 "TH?" H 3147 9304 50  0000 R CNN
+F 1 "Thermistor_NTC" H 3147 9395 50  0000 R CNN
+F 2 "" H 3300 9400 50  0001 C CNN
+F 3 "~" H 3300 9400 50  0001 C CNN
+	1    3300 9350
+	-1   0    0    1
+$EndComp
+Text HLabel 3300 8850 1    50   Input ~ 0
+NTC_Switch
+Wire Wire Line
+	3300 8850 3300 9200
+$Comp
+L BMS-Master-rescue:GND-power #PWR?
+U 1 1 5C85297F
+P 3300 9700
+F 0 "#PWR?" H 3300 9450 50  0001 C CNN
+F 1 "GND" H 3305 9527 50  0000 C CNN
+F 2 "" H 3300 9700 50  0001 C CNN
+F 3 "" H 3300 9700 50  0001 C CNN
+	1    3300 9700
+	1    0    0    -1
+$EndComp
+Wire Wire Line
+	3300 9500 3300 9700
 $EndSCHEMATC

Commit message: Schematics 90% completed
Parts:
- U1: renamed from U?; footprint (none) -> Housings_SSOP:TSSOP-16_4.4x5mm_Pitch0.65mm
- gave numbers to parts that had none: 28
