File: V0.2-LTC6813/BMS-Master/CAN.sch (KiCad schematic (older format))
At the start: 10 parts

Commit message: V0.2 LTC6813 block
Parts:
- C? (x5): symbol Device:C -> BMS-Master-rescue:C-Device
- D?: symbol Diode:MBR0540 -> BMS-Master-rescue:MBR0540-Diode
- Q?: symbol Transistor_FET:2N7002 -> BMS-Master-rescue:2N7002-Transistor_FET
- R? (x2): symbol Device:R -> BMS-Master-rescue:R-Device
Changed lines of the file:
@@
 	4750 3550 5200 3550
 $Comp
-L power:+3.3V #PWR?
+L BMS-Master-rescue:+3.3V-power #PWR?
 U 1 1 5A91EA58
 P 5050 3250
@@
 	5050 3350 5200 3350
 $Comp
-L power:GND #PWR?
+L BMS-Master-rescue:GND-power #PWR?
 U 1 1 5A91EADF
 P 5000 3850
@@
 	5000 3650 5000 3850
 $Comp
-L Device:C C?
+L BMS-Master-rescue:C-Device C?
 U 1 1 5A91EB41
 P 3750 3500
@@
 $EndComp
 $Comp
-L power:+3.3V #PWR?
+L BMS-Master-rescue:+3.3V-power #PWR?
 U 1 1 5A91EB6B
 P 3750 3050
@@
 	3750 3050 3750 3350
 $Comp
-L power:GND #PWR?
+L BMS-Master-rescue:GND-power #PWR?
 U 1 1 5A91EBA8
 P 3750 3750
@@
 	5650 2350 5650 4850
 $Comp
-L power:GNDD #PWR?
+L BMS-Master-rescue:GNDD-power #PWR?
 U 1 1 5A91F28A
 P 6100 3850
@@
 	6100 3650 6100 3850
 $Comp
-L Device:C C?
+L BMS-Master-rescue:C-Device C?
 U 1 1 5A91F3C0
 P 7300 3500
@@
 $EndComp
 $Comp
-L Device:R R?
+L BMS-Master-rescue:R-Device R?
 U 1 1 5A91F45F
 P 6900 3050
@@
 $EndComp
 $Comp
-L Device:R R?
+L BMS-Master-rescue:R-Device R?
 U 1 1 5A91F4AE
 P 6900 3900
@@
 	6900 4150 7550 4150
 $Comp
-L power:GNDD #PWR?
+L BMS-Master-rescue:GNDD-power #PWR?
 U 1 1 5A91F76E
 P 7650 3650
@@
 Connection ~ 6900 2700
 $Comp
-L power:GNDD #PWR?
+L BMS-Master-rescue:GNDD-power #PWR?
 U 1 1 5A91FE8A
 P 7650 2150
@@
 $EndComp
 $Comp
-L Device:C C?
+L BMS-Master-rescue:C-Device C?
 U 1 1 5A91FEEA
 P 7650 1900
@@
 	7650 2150 7650 2050
 $Comp
-L Device:C C?
+L BMS-Master-rescue:C-Device C?
 U 1 1 5A92018C
 P 8150 1900
@@
 $EndComp
 $Comp
-L power:GNDD #PWR?
+L BMS-Master-rescue:GNDD-power #PWR?
 U 1 1 5A9201EB
 P 8150 2150
@@
 	8150 2050 8150 2150
 $Comp
-L Diode:MBR0540 D?
+L BMS-Master-rescue:MBR0540-Diode D?
 U 1 1 5A92055E
 P 9000 1600
@@
 $EndComp
 $Comp
-L Transistor_FET:2N7002 Q?
+L BMS-Master-rescue:2N7002-Transistor_FET Q?
 U 1 1 5A92061C
 P 9000 950
@@
 	8150 750  8150 1600
 $Comp
-L power:GNDD #PWR?
+L BMS-Master-rescue:GNDD-power #PWR?
 U 1 1 5A921C15
 P 8700 1800
@@
 Reverse polarity protection\n
 $Comp
-L Device:C C?
+L BMS-Master-rescue:C-Device C?
 U 1 1 5A924642
 P 3300 3500
@@
 $EndComp
 $Comp
-L power:+3.3V #PWR?
+L BMS-Master-rescue:+3.3V-power #PWR?
 U 1 1 5A924C1D
 P 3300 3050
@@
 	3300 3050 3300 3350
 $Comp
-L power:GND #PWR?
+L BMS-Master-rescue:GND-power #PWR?
 U 1 1 5A925217
 P 3300 3750

Commit message: schematics 50% complete3d
Parts:
- removed C? (x2): 100n, Capacitors_SMD:C_0603_HandSoldering, symbol BMS-Master-rescue:C-Device
- removed C?: 4.7u, Capacitors_SMD:C_0805_HandSoldering, symbol BMS-Master-rescue:C-Device
- removed D?: MBR0540, Diode_SMD:D_SOD-123, symbol BMS-Master-rescue:MBR0540-Diode
- removed Q?: 2N7002, Package_TO_SOT_SMD:SOT-23, symbol BMS-Master-rescue:2N7002-Transistor_FET
- removed R? (x2): 60.4, Capacitors_SMD:C_0603_HandSoldering, symbol BMS-Master-rescue:R-Device
- added C?: 100n, Capacitors_SMD:C_0603_HandSoldering, symbol BMS-Master-rescue:C-Device
- added C?: 1u, Capacitors_SMD:C_0805_HandSoldering, symbol BMS-Master-rescue:C-Device
- added C?: 10n, Capacitors_SMD:C_0805_HandSoldering, symbol BMS-Master-rescue:C-Device
- added D?: SZNUP2105L, Package_TO_SOT_SMD:SOT-23, symbol Power_Protection:SZNUP2105L
- added R?: 4.7M, Capacitors_SMD:C_0805_HandSoldering, symbol BMS-Master-rescue:R-Device
- added R?: 2.2k, Capacitors_SMD:C_0603_HandSoldering, symbol BMS-Master-rescue:R-Device
- added U?: SFH617A-2X017T, Package_DIP:SMDIP-4_W9.53mm_Clearance8mm, symbol Isolator:SFH617A-2X017T
Connections:
- net labels added: CAN_GND, EnableRequest, Enable_CAN
- net labels removed: GNDD, GND_CAN
- wire segments 43 -> 45
Other:
- note removed: "Reverse polarity protection\n"

Commit message: Schematics 90% completed
Parts:
- gave numbers to parts that had none: 10
Changed lines of the file:
@@
 $EndDescr
 $Comp
-L ENNOID:ISO1050DUBR U?
+L ENNOID:ISO1050DUBR U8
 U 1 1 5A91E99C
 P 5600 3500
-F 0 "U?" H 5600 3915 50  0000 C CNN
+F 0 "U8" H 5600 3915 50  0000 C CNN
 F 1 "ISO1050DUBR" H 5600 3824 50  0000 C CNN
 F 2 "" H 5500 3150 50  0001 C CNN
@@
 	4750 3550 5200 3550
 $Comp
-L BMS-Master-rescue:+3.3V-power #PWR?
+L BMS-Master-rescue:+3.3V-power #PWR0183
 U 1 1 5A91EA58
 P 5050 3250
-F 0 "#PWR?" H 5050 3100 50  0001 C CNN
+F 0 "#PWR0183" H 5050 3100 50  0001 C CNN
 F 1 "+3.3V" H 5065 3423 50  0000 C CNN
 F 2 "" H 5050 3250 50  0001 C CNN
@@
 	5050 3350 5200 3350
 $Comp
-L BMS-Master-rescue:GND-power #PWR?
+L BMS-Master-rescue:GND-power #PWR0184
 U 1 1 5A91EADF
 P 5000 5150
-F 0 "#PWR?" H 5000 4900 50  0001 C CNN
+F 0 "#PWR0184" H 5000 4900 50  0001 C CNN
 F 1 "GND" H 5005 4977 50  0000 C CNN
 F 2 "" H 5000 5150 50  0001 C CNN
@@
 	5000 3650 5000 4300
 $Comp
-L BMS-Master-rescue:C-Device C?
+L BMS-Master-rescue:C-Device C44
 U 1 1 5A91EB41
 P 3750 3500
-F 0 "C?" H 3865 3546 50  0000 L CNN
+F 0 "C44" H 3865 3546 50  0000 L CNN
 F 1 "100n" H 3865 3455 50  0000 L CNN
 F 2 "Capacitors_SMD:C_0603_HandSoldering" H 3788 3350 50  0001 C CNN
@@
 $EndComp
 $Comp
-L BMS-Master-rescue:+3.3V-power #PWR?
+L BMS-Master-rescue:+3.3V-power #PWR0185
 U 1 1 5A91EB6B
 P 3750 3050
-F 0 "#PWR?" H 3750 2900 50  0001 C CNN
+F 0 "#PWR0185" H 3750 2900 50  0001 C CNN
 F 1 "+3.3V" H 3765 3223 50  0000 C CNN
 F 2 "" H 3750 3050 50  0001 C CNN
@@
 	3750 3050 3750 3350
 $Comp
-L BMS-Master-rescue:GND-power #PWR?
+L BMS-Master-rescue:GND-power #PWR0186
 U 1 1 5A91EBA8
 P 3750 3750
-F 0 "#PWR?" H 3750 3500 50  0001 C CNN
+F 0 "#PWR0186" H 3750 3500 50  0001 C CNN
 F 1 "GND" H 3755 3577 50  0000 C CNN
 F 2 "" H 3750 3750 50  0001 C CNN
@@
 	6000 3450 7100 3450
 $Comp
-L BMS-Master-rescue:C-Device C?
+L BMS-Master-rescue:C-Device C43
 U 1 1 5A924642
 P 3300 3500
-F 0 "C?" H 3415 3546 50  0000 L CNN
+F 0 "C43" H 3415 3546 50  0000 L CNN
 F 1 "1u" H 3415 3455 50  0000 L CNN
 F 2 "Capacitors_SMD:C_0805_HandSoldering" H 3338 3350 50  0001 C CNN
@@
 $EndComp
 $Comp
-L BMS-Master-rescue:+3.3V-power #PWR?
+L BMS-Master-rescue:+3.3V-power #PWR0187
 U 1 1 5A924C1D
 P 3300 3050
-F 0 "#PWR?" H 3300 2900 50  0001 C CNN
+F 0 "#PWR0187" H 3300 2900 50  0001 C CNN
 F 1 "+3.3V" H 3315 3223 50  0000 C CNN
 F 2 "" H 3300 3050 50  0001 C CNN
@@
 	3300 3050 3300 3350
 $Comp
-L BMS-Master-rescue:GND-power #PWR?
+L BMS-Master-rescue:GND-power #PWR0188
 U 1 1 5A925217
 P 3300 3750
-F 0 "#PWR?" H 3300 3500 50  0001 C CNN
+F 0 "#PWR0188" H 3300 3500 50  0001 C CNN
 F 1 "GND" H 3305 3577 50  0000 C CNN
 F 2 "" H 3300 3750 50  0001 C CNN
@@
 5V_CAN
 $Comp
-L BMS-Master-rescue:C-Device C?
+L BMS-Master-rescue:C-Device C47
 U 1 1 5C24AE55
 P 7000 1850
-F 0 "C?" V 6748 1850 50  0000 C CNN
+F 0 "C47" V 6748 1850 50  0000 C CNN
 F 1 "100n" V 6839 1850 50  0000 C CNN
 F 2 "Capacitors_SMD:C_0603_HandSoldering" H 7038 1700 50  0001 C CNN
@@
 $EndComp
 $Comp
-L BMS-Master-rescue:C-Device C?
+L BMS-Master-rescue:C-Device C46
 U 1 1 5C24B678
 P 6650 1850
-F 0 "C?" H 6765 1896 50  0000 L CNN
+F 0 "C46" H 6765 1896 50  0000 L CNN
 F 1 "1u" H 6765 1805 50  0000 L CNN
 F 2 "Capacitors_SMD:C_0805_HandSoldering" H 6688 1700 50  0001 C CNN
@@
 $EndComp
 $Comp
-L BMS-Master-rescue:R-Device R?
+L BMS-Master-rescue:R-Device R115
 U 1 1 5C24E192
 P 5600 4300
-F 0 "R?" V 5550 4000 50  0000 L CNN
+F 0 "R115" V 5550 4000 50  0000 L CNN
 F 1 "4.7M" V 5450 4000 50  0000 L CNN
 F 2 "Capacitors_SMD:C_0805_HandSoldering" V 5530 4300 50  0001 C CNN
@@
 $EndComp
 $Comp
-L BMS-Master-rescue:C-Device C?
+L BMS-Master-rescue:C-Device C45
 U 1 1 5C24E7DA
 P 5600 4950
-F 0 "C?" V 5350 4750 50  0000 C CNN
+F 0 "C45" V 5350 4750 50  0000 C CNN
 F 1 "10n" V 5450 4800 50  0000 C CNN
 F 2 "Capacitors_SMD:C_0805_HandSoldering" H 5638 4800 50  0001 C CNN
@@
 Connection ~ 6000 5150
 $Comp
-L Power_Protection:SZNUP2105L D?
+L Power_Protection:SZNUP2105L D4
 U 1 1 5C258D40
 P 7000 3900
-F 0 "D?" H 7205 3946 50  0000 L CNN
+F 0 "D4" H 7205 3946 50  0000 L CNN
 F 1 "SZNUP2105L" H 7205 3855 50  0000 L CNN
 F 2 "Package_TO_SOT_SMD:SOT-23" H 7225 3850 50  0001 L CNN
@@
 	5550 2350 5550 6300
 $Comp
-L Isolator:SFH617A-2X017T U?
+L Isolator:SFH617A-2X017T U9
 U 1 1 5C25CD2F
 P 5600 6100
-F 0 "U?" H 5600 6425 50  0000 C CNN
+F 0 "U9" H 5600 6425 50  0000 C CNN
 F 1 "SFH617A-2X017T" H 5600 6334 50  0000 C CNN
 F 2 "Package_DIP:SMDIP-4_W9.53mm_Clearance8mm" H 5600 5750 50  0001 C CIN
@@
 $EndComp
 $Comp
-L BMS-Master-rescue:GND-power #PWR?
+L BMS-Master-rescue:GND-power #PWR0189
 U 1 1 5C25DB56
 P 5100 6400
-F 0 "#PWR?" H 5100 6150 50  0001 C CNN
+F 0 "#PWR0189" H 5100 6150 50  0001 C CNN
 F 1 "GND" H 5105 6227 50  0000 C CNN
 F 2 "" H 5100 6400 50  0001 C CNN
@@
 	5100 6200 5100 6400
 $Comp
-L BMS-Master-rescue:R-Device R?
+L BMS-Master-rescue:R-Device R116
 U 1 1 5C25FA4A
 P 6450 6000
-F 0 "R?" V 6400 5700 50  0000 L CNN
+F 0 "R116" V 6400 5700 50  0000 L CNN
 F 1 "2.2k" V 6300 5700 50  0000 L CNN
 F 2 "Capacitors_SMD:C_0603_HandSoldering" V 6380 6000 50  0001 C CNN

Commit message: Schematics under revision
Parts:
- U8: footprint (none) -> ENNOID:ISO1050
Changed lines of the file:
@@
 F 0 "U8" H 5600 3915 50  0000 C CNN
 F 1 "ISO1050DUBR" H 5600 3824 50  0000 C CNN
-F 2 "" H 5500 3150 50  0001 C CNN
+F 2 "ENNOID:ISO1050" H 5500 3150 50  0001 C CNN
 F 3 "" H 5500 3150 50  0001 C CNN
 	1    5600 3500
