File: V0.2-LTC6813/BMS-Master/MCU.sch (KiCad schematic (older format))
At the start: 16 parts

Commit message: V0.2 LTC6813 block
Parts:
- C? (x8): symbol Device:C -> BMS-Master-rescue:C-Device
- J?: symbol Connector_Generic:Conn_01x05 -> BMS-Master-rescue:Conn_01x05-Connector_Generic
- J?: symbol Connector_Specialized:Micro_SD_Card_Det_Hirose_DM3AT -> BMS-Master-rescue:Micro_SD_Card_Det_Hirose_DM3AT-Connector_Specialized
- L?: symbol Device:L -> BMS-Master-rescue:L-Device
- Q?: symbol Transistor_FET:BSS138 -> BMS-Master-rescue:BSS138-Transistor_FET
- R?: symbol Device:R -> BMS-Master-rescue:R-Device
- SW?: symbol Switch:SW_MEC_5G -> BMS-Master-rescue:SW_MEC_5G-Switch
- U?: symbol MCU_ST_STM32:STM32F303CCTx -> BMS-Master-rescue:STM32F303CCTx-MCU_ST_STM32
- Y?: symbol Device:Crystal -> BMS-Master-rescue:Crystal-Device
Changed lines of the file:
@@
 	16400 11900 16450 11900
 $Comp
-L power:GND #PWR?
+L BMS-Master-rescue:GND-power #PWR?
 U 1 1 5A921A89
 P 16450 12100
@@
 	16450 11900 16500 11900
 $Comp
-L Device:C C?
+L BMS-Master-rescue:C-Device C?
 U 1 1 5A921BA9
 P 7000 9400
@@
 $EndComp
 $Comp
-L Device:C C?
+L BMS-Master-rescue:C-Device C?
 U 1 1 5A921C07
 P 6000 9400
@@
 $EndComp
 $Comp
-L Device:Crystal Y?
+L BMS-Master-rescue:Crystal-Device Y?
 U 1 1 5A921CE8
 P 6500 9200
@@
 	7000 9200 7000 9100
 $Comp
-L power:GND #PWR?
+L BMS-Master-rescue:GND-power #PWR?
 U 1 1 5A92281A
 P 6000 9600
@@
 $EndComp
 $Comp
-L power:GND #PWR?
+L BMS-Master-rescue:GND-power #PWR?
 U 1 1 5A92287D
 P 7000 9600
@@
 	9200 9000 6000 9000
 $Comp
-L power:GND #PWR?
+L BMS-Master-rescue:GND-power #PWR?
 U 1 1 5A9256C5
 P 8150 9650
@@
 	7800 9650 7750 9650
 $Comp
-L Connector_Specialized:Micro_SD_Card_Det_Hirose_DM3AT J?
+L BMS-Master-rescue:Micro_SD_Card_Det_Hirose_DM3AT-Connector_Specialized J?
 U 1 1 5A92F51A
 P 4800 11400
@@
 	4000 12300 4000 11900
 $Comp
-L power:GND #PWR?
+L BMS-Master-rescue:GND-power #PWR?
 U 1 1 5A933A6F
 P 5700 12450
@@
 	7400 11100 5700 11100
 $Comp
-L Device:C C?
+L BMS-Master-rescue:C-Device C?
 U 1 1 5A934D3C
 P 7050 12250
@@
 	7050 11300 5700 11300
 $Comp
-L power:+3.3V #PWR?
+L BMS-Master-rescue:+3.3V-power #PWR?
 U 1 1 5A9358BF
 P 7900 12000
@@
 $EndComp
 $Comp
-L power:GND #PWR?
+L BMS-Master-rescue:GND-power #PWR?
 U 1 1 5A9358DF
 P 7050 12450
@@
 	5700 11900 5700 12300
 $Comp
-L Device:L L?
+L BMS-Master-rescue:L-Device L?
 U 1 1 5A93EB70
 P 7500 12000
@@
 	9200 10500 8950 10500
 $Comp
-L Device:C C?
+L BMS-Master-rescue:C-Device C?
 U 1 1 5A95E11B
 P 7050 8350
@@
 $EndComp
 $Comp
-L power:GND #PWR?
+L BMS-Master-rescue:GND-power #PWR?
 U 1 1 5A95E15B
 P 7050 8550
@@
 	7050 8500 7050 8550
 $Comp
-L power:+3.3V #PWR?
+L BMS-Master-rescue:+3.3V-power #PWR?
 U 1 1 5A964008
 P 16450 7650
@@
 	25500 10900 23800 10900
 $Comp
-L power:+3.3V #PWR?
+L BMS-Master-rescue:+3.3V-power #PWR?
 U 1 1 5AA4D323
 P 20600 7150
@@
 $EndComp
 $Comp
-L Device:C C?
+L BMS-Master-rescue:C-Device C?
 U 1 1 5AA4D32A
 P 20600 7350
@@
 	20600 7200 20600 7150
 $Comp
-L power:GND #PWR?
+L BMS-Master-rescue:GND-power #PWR?
 U 1 1 5AA51178
 P 20600 7600
@@
 	20600 7600 20600 7500
 $Comp
-L power:+3.3V #PWR?
+L BMS-Master-rescue:+3.3V-power #PWR?
 U 1 1 5AA550BE
 P 21200 7150
@@
 $EndComp
 $Comp
-L Device:C C?
+L BMS-Master-rescue:C-Device C?
 U 1 1 5AA550C5
 P 21200 7350
@@
 	21200 7200 21200 7150
 $Comp
-L power:GND #PWR?
+L BMS-Master-rescue:GND-power #PWR?
 U 1 1 5AA550CC
 P 21200 7600
@@
 	21200 7600 21200 7500
 $Comp
-L power:+3.3V #PWR?
+L BMS-Master-rescue:+3.3V-power #PWR?
 U 1 1 5AA591BA
 P 21800 7150
@@
 $EndComp
 $Comp
-L Device:C C?
+L BMS-Master-rescue:C-Device C?
 U 1 1 5AA591C1
 P 21800 7350
@@
 	21800 7200 21800 7150
 $Comp
-L power:GND #PWR?
+L BMS-Master-rescue:GND-power #PWR?
 U 1 1 5AA591C8
 P 21800 7600
@@
 	21800 7600 21800 7500
 $Comp
-L power:+3.3V #PWR?
+L BMS-Master-rescue:+3.3V-power #PWR?
 U 1 1 5AA591CF
 P 22400 7150
@@
 $EndComp
 $Comp
-L Device:C C?
+L BMS-Master-rescue:C-Device C?
 U 1 1 5AA591D6
 P 22400 7350
@@
 	22400 7200 22400 7150
 $Comp
-L power:GND #PWR?
+L BMS-Master-rescue:GND-power #PWR?
 U 1 1 5AA591DD
 P 22400 7600
@@
 	7050 8200 9200 8200
 $Comp
-L Device:R R?
+L BMS-Master-rescue:R-Device R?
 U 1 1 5AA7B298
 P 8500 8550
@@
 $EndComp
 $Comp
-L power:GND #PWR?
+L BMS-Master-rescue:GND-power #PWR?
 U 1 1 5AA7B2E6
 P 8500 8800
@@
 Connection ~ 8500 8300
 $Comp
-L power:+3.3V #PWR?
+L BMS-Master-rescue:+3.3V-power #PWR?
 U 1 1 5AA8A218
 P 7500 8500
@@
 	7500 8550 7700 8550
 $Comp
-L Switch:SW_MEC_5G SW?
+L BMS-Master-rescue:SW_MEC_5G-Switch SW?
 U 1 1 5A8F5FFE
 P 7900 8550
@@
 $EndComp
 $Comp
-L Connector_Generic:Conn_01x05 J?
+L BMS-Master-rescue:Conn_01x05-Connector_Generic J?
 U 1 1 5A92BF2C
 P 27400 11350
@@
 	27000 11550 27200 11550
 $Comp
-L power:GND #PWR?
+L BMS-Master-rescue:GND-power #PWR?
 U 1 1 5A959924
 P 26600 11400
@@
 	26600 11350 27200 11350
 $Comp
-L power:+3.3V #PWR?
+L BMS-Master-rescue:+3.3V-power #PWR?
 U 1 1 5A95ED28
 P 26600 11150
@@
 	23800 10000 25050 10000
 $Comp
-L Transistor_FET:BSS138 Q?
+L BMS-Master-rescue:BSS138-Transistor_FET Q?
 U 1 1 5ABE0CA0
 P 8050 9450
@@
 $EndComp
 $Comp
-L MCU_ST_STM32:STM32F303CCTx U?
+L BMS-Master-rescue:STM32F303CCTx-MCU_ST_STM32 U?
 U 1 1 5A92186F
 P 16500 9800

Commit message: schematics 50% complete3d
Parts:
- added C?: 100n, Capacitors_SMD:C_0603_HandSoldering, symbol BMS-Master-rescue:C-Device
- added R?: 1k, Resistors_SMD:R_0603_HandSoldering, symbol BMS-Master-rescue:R-Device
Connections:
- net labels added: MISO, MOSI, NTC_Switch, OLED_RST, OLED_SCL, OLED_SDA, RX_USB, SAFETY, SCK, SCL, SDA, SPI_WT_SS, SS, TX_USB, VoutSense, Wireless_GDO0
- net labels removed: FAULT_N, GPIO0, GPIO1, GPIO2, GPIO3, GPIO4, GPIO5, I+, I-, RX, TX, USB_DM, USB_DP, V+
Other:
- moved on the sheet: Q?

Commit message: Schematics 80% completed
Parts:
- removed R?: 1k, Resistors_SMD:R_0603_HandSoldering, symbol BMS-Master-rescue:R-Device
- removed SW?: B3U-1000P, symbol BMS-Master-rescue:SW_MEC_5G-Switch
- added R? (x2): 10k, Resistors_SMD:R_0603_HandSoldering, symbol BMS-Master-rescue:R-Device
- added R?: 1.5k, Resistors_SMD:R_0603_HandSoldering, symbol BMS-Master-rescue:R-Device
Connections:
- net labels added: Safety, SwitchEnable
- net labels removed: SAFETY, WAKEUP
- wire segments 121 -> 122
Changed lines of the file:
@@
 $Descr A1 33110 23386
 encoding utf-8
-Sheet 23 27
+Sheet 27 27
 Title ""
 Date ""
@@
 RX_USB
 Text HLabel 9100 9300 0    50   Input ~ 0
-SAFETY
-Text HLabel 8950 9900 0    50   Input ~ 0
-WAKEUP
+Safety
+Text HLabel 8100 9900 0    50   Input ~ 0
+SwitchEnable
 Wire Wire Line
 	16300 11600 16300 11900
@@
 Wire Wire Line
 	9100 9300 9200 9300
-Text HLabel 7500 9950 0    50   BiDi ~ 0
+Text HLabel 7200 9950 0    50   BiDi ~ 0
 ChargeDetect
 Wire Wire Line
@@
 	7050 8200 9200 8200
 $Comp
-L BMS-Master-rescue:R-Device R?
-U 1 1 5AA7B298
-P 8500 8550
-F 0 "R?" H 8570 8596 50  0000 L CNN
-F 1 "1k" H 8570 8505 50  0000 L CNN
-F 2 "Resistors_SMD:R_0603_HandSoldering" V 8430 8550 50  0001 C CNN
-F 3 "~" H 8500 8550 50  0001 C CNN
-	1    8500 8550
-	1    0    0    -1
-$EndComp
-$Comp
 L BMS-Master-rescue:GND-power #PWR?
 U 1 1 5AA7B2E6
-P 8500 8800
-F 0 "#PWR?" H 8500 8550 50  0001 C CNN
-F 1 "GND" H 8505 8627 50  0000 C CNN
-F 2 "" H 8500 8800 50  0001 C CNN
-F 3 "" H 8500 8800 50  0001 C CNN
-	1    8500 8800
-	1    0    0    -1
-$EndComp
-Wire Wire Line
-	8500 8700 8500 8800
-Wire Wire Line
-	9200 8600 8850 8600
-Wire Wire Line
-	8850 8600 8850 8300
-Wire Wire Line
-	8850 8300 8500 8300
-Wire Wire Line
-	8500 8300 8500 8400
-Wire Wire Line
-	8100 8550 8300 8550
-Wire Wire Line
-	8300 8550 8300 8300
-Wire Wire Line
-	8300 8300 8500 8300
-Connection ~ 8500 8300
-$Comp
-L BMS-Master-rescue:+3.3V-power #PWR?
-U 1 1 5AA8A218
-P 7500 8500
-F 0 "#PWR?" H 7500 8350 50  0001 C CNN
-F 1 "+3.3V" H 7515 8673 50  0000 C CNN
-F 2 "" H 7500 8500 50  0001 C CNN
-F 3 "" H 7500 8500 50  0001 C CNN
-	1    7500 8500
-	1    0    0    -1
-$EndComp
-Wire Wire Line
-	7500 8500 7500 8550
-Wire Wire Line
-	7500 8550 7700 8550
-$Comp
-L BMS-Master-rescue:SW_MEC_5G-Switch SW?
-U 1 1 5A8F5FFE
-P 7900 8550
-F 0 "SW?" H 7900 8835 50  0000 C CNN
-F 1 "B3U-1000P" H 7900 8744 50  0000 C CNN
-F 2 "" H 7900 8750 50  0001 C CNN
-F 3 "http://www.apem.com/int/index.php?controller=attachment&id_attachment=488" H 7900 8750 50  0001 C CNN
-	1    7900 8550
-	-1   0    0    -1
+P 8500 8650
+F 0 "#PWR?" H 8500 8400 50  0001 C CNN
+F 1 "GND" H 8505 8477 50  0000 C CNN
+F 2 "" H 8500 8650 50  0001 C CNN
+F 3 "" H 8500 8650 50  0001 C CNN
+	1    8500 8650
+	1    0    0    -1
 $EndComp
 $Comp
@@
 	7800 9200 8600 9200
 Wire Wire Line
-	7500 9400 7500 9950
-Wire Wire Line
 	7800 9600 7800 9650
 Wire Wire Line
 	23800 9800 24450 9800
 Wire Wire Line
-	9200 9900 8950 9900
+	9200 9900 8200 9900
 Text HLabel 25050 9700 2    50   BiDi ~ 0
 NTC_Switch
@@
 Text Label 8450 10600 2    50   ~ 0
 SDCardDetect
-Wire Wire Line
-	5700 11800 6500 11800
-Text Label 6500 11800 2    50   ~ 0
+Text Label 6500 11900 2    50   ~ 0
 SDCardDetect
 Wire Wire Line
@@
 $EndComp
 Wire Wire Line
-	5700 11900 5700 12300
-Wire Wire Line
 	7050 12400 7050 12450
 $Comp
@@
 Wire Wire Line
 	9200 10900 7400 10900
-Wire Wire Line
-	5700 12300 4000 12300
-Connection ~ 5700 12300
-Wire Wire Line
-	5700 12450 5700 12300
 $Comp
 L BMS-Master-rescue:GND-power #PWR?
 U 1 1 5A933A6F
-P 5700 12450
-F 0 "#PWR?" H 5700 12200 50  0001 C CNN
-F 1 "GND" H 5705 12277 50  0000 C CNN
-F 2 "" H 5700 12450 50  0001 C CNN
-F 3 "" H 5700 12450 50  0001 C CNN
-	1    5700 12450
+P 6550 12450
+F 0 "#PWR?" H 6550 12200 50  0001 C CNN
+F 1 "GND" H 6555 12277 50  0000 C CNN
+F 2 "" H 6550 12450 50  0001 C CNN
+F 3 "" H 6550 12450 50  0001 C CNN
+	1    6550 12450
 	1    0    0    -1
 $EndComp
@@
 	4000 12300 4000 11900
 Wire Wire Line
-	6900 12300 5700 12300
+	6900 12300 6550 12300
 Wire Wire Line
 	6900 11500 6900 12300
@@
 $EndComp
 Wire Wire Line
-	23800 10300 24450 10300
-Text HLabel 24450 10300 2    50   Input ~ 0
+	23800 10300 26100 10300
+Text HLabel 26350 10300 2    50   Input ~ 0
 MISO
+$Comp
+L BMS-Master-rescue:+3.3V-power #PWR?
+U 1 1 5C66533B
+P 7050 7550
+F 0 "#PWR?" H 7050 7400 50  0001 C CNN
+F 1 "+3.3V" H 7065 7723 50  0000 C CNN
+F 2 "" H 7050 7550 50  0001 C CNN
+F 3 "" H 7050 7550 50  0001 C CNN
+	1    7050 7550
+	1    0    0    -1
+$EndComp
+$Comp
+L BMS-Master-rescue:R-Device R?
+U 1 1 5C665C3A
+P 7050 7800
+F 0 "R?" H 7120 7846 50  0000 L CNN
+F 1 "10k" H 7120 7755 50  0000 L CNN
+F 2 "Resistors_SMD:R_0603_HandSoldering" V 6980 7800 50  0001 C CNN
+F 3 "~" H 7050 7800 50  0001 C CNN
+	1    7050 7800
+	1    0    0    -1
+$EndComp
+Wire Wire Line
+	7050 7550 7050 7650
+Wire Wire Line
+	7050 7950 7050 8200
+Connection ~ 7050 8200
+Wire Wire Line
+	8500 8600 8500 8650
+Wire Wire Line
+	8500 8600 9200 8600
+Wire Wire Line
+	5700 11900 6500 11900
+Wire Wire Line
+	5700 11800 6550 11800
+Wire Wire Line
+	6550 11800 6550 12300
+Connection ~ 6550 12300
+Wire Wire Line
+	4000 12300 6550 12300
+Wire Wire Line
+	6550 12300 6550 12450
+$Comp
+L BMS-Master-rescue:R-Device R?
+U 1 1 5C6988CA
+P 8200 10050
+F 0 "R?" H 8270 10096 50  0000 L CNN
+F 1 "10k" H 8270 10005 50  0000 L CNN
+F 2 "Resistors_SMD:R_0603_HandSoldering" V 8130 10050 50  0001 C CNN
+F 3 "~" H 8200 10050 50  0001 C CNN
+	1    8200 10050
+	1    0    0    -1
+$EndComp
+Connection ~ 8200 9900
+Wire Wire Line
+	8200 9900 8100 9900
+$Comp
+L BMS-Master-rescue:GND-power #PWR?
+U 1 1 5C699041
+P 8200 10250
+F 0 "#PWR?" H 8200 10000 50  0001 C CNN
+F 1 "GND" H 8205 10077 50  0000 C CNN
+F 2 "" H 8200 10250 50  0001 C CNN
+F 3 "" H 8200 10250 50  0001 C CNN
+	1    8200 10250
+	1    0    0    -1
+$EndComp
+Wire Wire Line
+	8200 10200 8200 10250
+Wire Wire Line
+	7200 9950 7400 9950
+Wire Wire Line
+	7400 9950 7400 9400
+Wire Wire Line
+	7400 9400 7500 9400
+$Comp
+L BMS-Master-rescue:R-Device R?
+U 1 1 5C6AE41B
+P 26100 10150
+F 0 "R?" H 26170 10196 50  0000 L CNN
+F 1 "1.5k" H 26170 10105 50  0000 L CNN
+F 2 "Resistors_SMD:R_0603_HandSoldering" V 26030 10150 50  0001 C CNN
+F 3 "~" H 26100 10150 50  0001 C CNN
+	1    26100 10150
+	1    0    0    -1
+$EndComp
+$Comp
+L BMS-Master-rescue:+3.3V-power #PWR?
+U 1 1 5C6AE421
+P 26100 9950
+F 0 "#PWR?" H 26100 9800 50  0001 C CNN
+F 1 "+3.3V" H 26115 10123 50  0000 C CNN
+F 2 "" H 26100 9950 50  0001 C CNN
+F 3 "" H 26100 9950 50  0001 C CNN
+	1    26100 9950
+	1    0    0    -1
+$EndComp
+Wire Wire Line
+	26100 9950 26100 10000
+Connection ~ 26100 10300
+Wire Wire Line
+	26100 10300 26350 10300
 $EndSCHEMATC

Commit message: Schematics 90% completed
Parts:
- J16: renamed from J?; value Micro_SD_Card_Det_Hirose_DM3AT -> J
- J17: renamed from J?; footprint (none) -> Connectors_Molex:Molex_KK-6410-05_05x2.54mm_Straight
- gave numbers to parts that had none: 17
Connections:
- no-connect marks 0 -> 3

Commit message: Bootloader from DieBieMS added
Parts:
- J16: footprint (none) -> Connectors_Card:Hirose_DM3AT-SF-PEJM5
Changed lines of the file:
@@
 F 0 "J16" H 4750 12217 50  0000 C CNN
 F 1 "J" H 4750 12126 50  0000 C CNN
-F 2 "" H 6850 12100 50  0001 C CNN
+F 2 "Connectors_Card:Hirose_DM3AT-SF-PEJM5" H 6850 12100 50  0001 C CNN
 F 3 "" H 4800 11500 50  0001 C CNN
 	1    4800 11400
