File: V0.2-LTC6813/BMS-Master/PowerSupply.sch (KiCad schematic (older format))
At the start: 48 parts

Commit message: Schematics 85% completed
Parts:
- removed D? (x2): 5V zener, symbol BMS-Master-rescue:D_Zener-Device
- removed R? (x12): 1M, Resistors_SMD:R_1206, symbol BMS-Master-rescue:R-Device
- removed R? (x2): 100k, Resistors_SMD:R_1206, symbol BMS-Master-rescue:R-Device
Connections:
- net labels removed: Bat+, Charge+, GNDA
- wire segments 147 -> 113

Commit message: Schematics 90% completed
Parts:
- removed C?: 1u, Capacitors_SMD:C_1206_HandSoldering, symbol BMS-Master-rescue:C-Device
- removed C? (x2): 4.7u, Capacitors_SMD:C_1206_HandSoldering, symbol BMS-Master-rescue:C-Device
- removed C? (x2): 0.1u, Capacitors_SMD:C_0805_HandSoldering, symbol BMS-Master-rescue:C-Device
- removed C?: 1u, Capacitors_SMD:C_0805_HandSoldering, symbol BMS-Master-rescue:C-Device
- removed C? (x4): 0.01u, Capacitors_SMD:C_0603_HandSoldering, symbol BMS-Master-rescue:C-Device
- removed C?: 22u, Capacitors_SMD:C_1812_HandSoldering, symbol BMS-Master-rescue:C-Device
- removed C?: 4.7u, symbol BMS-Master-rescue:C-Device
- removed C?: 330p, symbol BMS-Master-rescue:C-Device
- removed C?: 2.2u, symbol BMS-Master-rescue:C-Device
- removed D?: B180-13-F, Diodes_SMD:D_SMA, symbol BMS-Master-rescue:D_Zener-Device
- removed L?: 220u, symbol BMS-Master-rescue:INDUCTOR-pspice
- removed Q?: ZXTN4004KTC, TO_SOT_Packages_SMD:TO-252-2, symbol BMS-Master-rescue:Q_NPN_BCE-Device
- removed R? (x2): 200, Resistors_SMD:R_2512, symbol BMS-Master-rescue:R-Device
- removed R?: 0.39, Resistors_SMD:R_0603_HandSoldering, symbol BMS-Master-rescue:R-Device
- removed R? (x2): 1, Resistors_SMD:R_0603_HandSoldering, symbol BMS-Master-rescue:R-Device
- removed R?: 174k, Resistors_SMD:R_0603_HandSoldering, symbol BMS-Master-rescue:R-Device
- removed R?: 665k, Resistors_SMD:R_0603_HandSoldering, symbol BMS-Master-rescue:R-Device
- removed R?: 1.2k, Resistors_SMD:R_0603_HandSoldering, symbol BMS-Master-rescue:R-Device
- removed R? (x3): 10k, Resistors_SMD:R_0603_HandSoldering, symbol BMS-Master-rescue:R-Device
- removed R?: 1.5, Resistors_SMD:R_0805_HandSoldering, symbol BMS-Master-rescue:R-Device
- removed U?: LM5008MM, Package_SO:MSOP-8_3x3mm_P0.65mm, symbol BMS-Master-rescue:LM5008MM-Regulator_Switching
- removed U?: LP2985-3.3, Package_TO_SOT_SMD:SOT-23-5, symbol BMS-Master-rescue:LP2985-3.3-Regulator_Linear
- added C? (x3): C, Capacitors_SMD:C_1206_HandSoldering, symbol BMS-Master-rescue:C-Device
- added C? (x2): 1u, Capacitors_SMD:C_0603_HandSoldering, symbol BMS-Master-rescue:C-Device
- added C? (x3): 10u, Capacitors_SMD:C_0603_HandSoldering, symbol BMS-Master-rescue:C-Device
- added C?: 47n, Capacitors_SMD:C_0603_HandSoldering, symbol BMS-Master-rescue:C-Device
- added C?: 2.2u, Capacitors_SMD:C_0603_HandSoldering, symbol BMS-Master-rescue:C-Device
- added D? (x7): D, symbol Device:D
- added F? (x2): Fuse, symbol Device:Fuse
- added L? (x2): L, symbol Device:L
- added Q? (x3): BSS138, Package_TO_SOT_SMD:SOT-23, symbol Transistor_FET:BSS138
- added R? (x2): 4.7M, Resistors_SMD:R_0805_HandSoldering, symbol BMS-Master-rescue:R-Device
- added R?: 130k, Resistors_SMD:R_0603_HandSoldering, symbol BMS-Master-rescue:R-Device
- added R? (x3): 10k, Resistors_SMD:R_0603_HandSoldering, symbol BMS-Master-rescue:R-Device
- added R? (x4): 1, Resistors_SMD:R_0603_HandSoldering, symbol BMS-Master-rescue:R-Device
- added R?: 1M, Resistors_SMD:R_0603_HandSoldering, symbol BMS-Master-rescue:R-Device
- added R?: 100, Resistors_SMD:R_0603_HandSoldering, symbol BMS-Master-rescue:R-Device
- added U?: EPM2405SJ, symbol ENNOID:EPM2405SJ
- added U?: LM5165, Package_SON:Texas_S-PVSON-N10_ThermalVias, symbol Regulator_Switching:LM5165
Connections:
- net labels added: +12V, +3V3, ChargeDetect, EnableFromExt, GNDA
- net labels removed: +3.3V, +5V, NPN_BASE, VDIG, VIO, VP1
- no-connect marks 0 -> 10
Other:
- moved on the sheet: JP?

Commit message: Schematics 90% completed
Parts:
- JP22: renamed from JP?; footprint (none) -> Pin_Headers:Pin_Header_Straight_1x03_Pitch2.54mm
- gave numbers to parts that had none: 38
Connections:
- no-connect marks 10 -> 12

Commit message: 90% schematics completed
Parts:
- C85: value C -> 33u
- C86: value C -> 10n; footprint Capacitors_SMD:C_1206_HandSoldering -> Capacitors_SMD:C_0603_HandSoldering
- C87: value C -> 220u; footprint Capacitors_SMD:C_1206_HandSoldering -> Capacitors_SMD:CP_Elec_8x10
- L2: value L -> 2.2uH - 4Amps
Changed lines of the file:
@@
 P 3100 6850
 F 0 "C85" H 3215 6896 50  0000 L CNN
-F 1 "C" H 3215 6805 50  0000 L CNN
+F 1 "33u" H 3215 6805 50  0000 L CNN
 F 2 "Capacitors_SMD:C_1206_HandSoldering" H 3138 6700 50  0001 C CNN
 F 3 "~" H 3100 6850 50  0001 C CNN
@@
 P 5650 6650
 F 0 "L2" V 5840 6650 50  0000 C CNN
-F 1 "L" V 5749 6650 50  0000 C CNN
+F 1 "2.2uH - 4Amps" V 5749 6650 50  0000 C CNN
 F 2 "" H 5650 6650 50  0001 C CNN
-F 3 "~" H 5650 6650 50  0001 C CNN
+F 3 "https://www.google.com/url?sa=t&rct=j&q=&esrc=s&source=web&cd=3&cad=rja&uact=8&ved=2ahUKEwjF8sbF6NLfAhVPqlkKHfcADH4QFjACegQICBAC&url=http%3A%2F%2Fwww.korin.co.jp%2Fproduct%2Fpdf%2FCat09501Sa.pdf&usg=AOvVaw3C9mpYL_KrwIiBYSZfq788" H 5650 6650 50  0001 C CNN
 	1    5650 6650
 	0    -1   -1   0
@@
 P 5300 6900
 F 0 "C86" H 5415 6946 50  0000 L CNN
-F 1 "C" H 5415 6855 50  0000 L CNN
-F 2 "Capacitors_SMD:C_1206_HandSoldering" H 5338 6750 50  0001 C CNN
+F 1 "10n" H 5415 6855 50  0000 L CNN
+F 2 "Capacitors_SMD:C_0603_HandSoldering" H 5338 6750 50  0001 C CNN
 F 3 "~" H 5300 6900 50  0001 C CNN
 F 4 "" H 5500 6750 50  0001 C CNN "Volatge"
@@
 P 6000 6950
 F 0 "C87" H 6115 6996 50  0000 L CNN
-F 1 "C" H 6115 6905 50  0000 L CNN
-F 2 "Capacitors_SMD:C_1206_HandSoldering" H 6038 6800 50  0001 C CNN
-F 3 "~" H 6000 6950 50  0001 C CNN
-F 4 "" H 6200 6800 50  0001 C CNN "Volatge"
+F 1 "220u" H 6115 6905 50  0000 L CNN
+F 2 "Capacitors_SMD:CP_Elec_8x10" H 6038 6800 50  0001 C CNN
+F 3 "UWT1V221MNL1GS" H 6000 6950 50  0001 C CNN
 	1    6000 6950
 	1    0    0    -1

Commit message: 92.5% schematics completed
Parts:
- removed F2, F3: Fuse, symbol Device:Fuse
- L2: footprint (none) -> ENNOID:TDK_Inductor
Connections:
- net BAT+: now also C85.1, U18.12 (+DC_IN)
- net ExternalPower: now also JP22.3
Changed lines of the file:
@@
 ExternalPower
-Wire Wire Line
-	7900 5800 8050 5800
 Wire Wire Line
 	8650 5800 8650 6150
@@
 	2350 7150 3100 7150
 Connection ~ 3100 7150
-Wire Wire Line
-	1700 6650 2150 6650
 Connection ~ 3100 6650
 $Comp
@@
 F 0 "L2" V 5840 6650 50  0000 C CNN
 F 1 "2.2uH - 4Amps" V 5749 6650 50  0000 C CNN
-F 2 "" H 5650 6650 50  0001 C CNN
+F 2 "ENNOID:TDK_Inductor" H 5650 6650 50  0001 C CNN
 F 3 "https://www.google.com/url?sa=t&rct=j&q=&esrc=s&source=web&cd=3&cad=rja&uact=8&ved=2ahUKEwjF8sbF6NLfAhVPqlkKHfcADH4QFjACegQICBAC&url=http%3A%2F%2Fwww.korin.co.jp%2Fproduct%2Fpdf%2FCat09501Sa.pdf&usg=AOvVaw3C9mpYL_KrwIiBYSZfq788" H 5650 6650 50  0001 C CNN
 	1    5650 6650
@@
 Wire Wire Line
 	11000 5900 11200 5900
-$Comp
-L Device:Fuse F2
-U 1 1 5C5F7134
-P 2300 6650
-F 0 "F2" V 2103 6650 50  0000 C CNN
-F 1 "Fuse" V 2194 6650 50  0000 C CNN
-F 2 "" V 2230 6650 50  0001 C CNN
-F 3 "~" H 2300 6650 50  0001 C CNN
-	1    2300 6650
-	0    1    1    0
-$EndComp
-Wire Wire Line
-	2450 6650 3100 6650
-$Comp
-L Device:Fuse F3
-U 1 1 5C5F84F5
-P 8200 5800
-F 0 "F3" V 8003 5800 50  0000 C CNN
-F 1 "Fuse" V 8094 5800 50  0000 C CNN
-F 2 "" V 8130 5800 50  0001 C CNN
-F 3 "~" H 8200 5800 50  0001 C CNN
-	1    8200 5800
-	0    1    1    0
-$EndComp
-Wire Wire Line
-	8350 5800 8650 5800
 $Comp
 L Regulator_Switching:LM5165 U19
@@
 Wire Notes Line
 	4400 5400 4400 9750
+Wire Wire Line
+	7900 5800 8650 5800
+Wire Wire Line
+	1700 6650 3100 6650
 $EndSCHEMATC

Commit message: Schematics under revision
Parts:
- removed D10, D11, D12, D13, D7, D8, D9: D, symbol Device:D
- added D? (x5): 1N4148W, Diode_SMD:D_SOD-123, symbol Diode:1N4148W
- added D? (x2): BZT52C16, Diode_SMD:D_SOD-123, symbol Diode:BZT52Bxx
- L2: value 2.2uH - 4Amps -> 2.2uH - 4Amps - CLF6045T-2R2N-D
- L3: value L -> 744043151; footprint (none) -> Inductors_SMD:L_Wuerth_WE-PD2-Typ-MS
- U18: footprint (none) -> ENNOID:EPM2405SJ
Connections:
- net +3V3: now also D?.2 (A), D?.2 (A)
- net ChargeDetect: now also D?.1 (K)
- net EnableFromExt: now also D?.1 (K)
- net GND: now also D?.2 (A), D?.2 (A)
- net at Q29.3 (D), Q30.1 (G), R175.1: now also D?.1 (K), D?.2 (A), D?.2 (A), D?.2 (A)
- net at R178.1: now also D?.1 (K)
- net at C88.2, R174.2: now also D?.1 (K)
- net at C88.1, Q28.1 (G), R172.2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: now also D?.1 (K)
- net at R173.2: now also D?.1 (K)
Changed lines of the file:
@@
 F 0 "U18" H 3800 8550 50  0000 C CNN
 F 1 "EPM2405SJ" H 3950 8450 50  0000 C CNN
-F 2 "" H 4300 7350 50  0001 C CNN
+F 2 "ENNOID:EPM2405SJ" H 4300 7350 50  0001 C CNN
 F 3 "" H 4300 7350 50  0001 C CNN
 	1    4300 7350
@@
 P 5650 6650
 F 0 "L2" V 5840 6650 50  0000 C CNN
-F 1 "2.2uH - 4Amps" V 5749 6650 50  0000 C CNN
+F 1 "2.2uH - 4Amps - CLF6045T-2R2N-D" V 5749 6650 50  0000 C CNN
 F 2 "ENNOID:TDK_Inductor" H 5650 6650 50  0001 C CNN
 F 3 "https://www.google.com/url?sa=t&rct=j&q=&esrc=s&source=web&cd=3&cad=rja&uact=8&ved=2ahUKEwjF8sbF6NLfAhVPqlkKHfcADH4QFjACegQICBAC&url=http%3A%2F%2Fwww.korin.co.jp%2Fproduct%2Fpdf%2FCat09501Sa.pdf&usg=AOvVaw3C9mpYL_KrwIiBYSZfq788" H 5650 6650 50  0001 C CNN
@@
 	11000 6400 11900 6400
 Connection ~ 11000 6400
-$Comp
-L Device:D D10
-U 1 1 5C68AB63
-P 13350 7400
-F 0 "D10" V 13304 7479 50  0000 L CNN
-F 1 "D" V 13395 7479 50  0000 L CNN
-F 2 "" H 13350 7400 50  0001 C CNN
-F 3 "~" H 13350 7400 50  0001 C CNN
-	1    13350 7400
-	0    1    1    0
-$EndComp
 Wire Wire Line
 	12400 6400 13350 6400
@@
 Wire Wire Line
 	13350 7550 13350 7600
-$Comp
-L Device:D D11
-U 1 1 5C6ABFB0
-P 13550 8500
-F 0 "D11" H 13550 8284 50  0000 C CNN
-F 1 "D" H 13550 8375 50  0000 C CNN
-F 2 "" H 13550 8500 50  0001 C CNN
-F 3 "~" H 13550 8500 50  0001 C CNN
-	1    13550 8500
-	-1   0    0    1
-$EndComp
 Text HLabel 14650 8500 2    50   Input ~ 0
 EnableFromExt
@@
 Wire Wire Line
 	13700 8500 14650 8500
-$Comp
-L Device:D D12
-U 1 1 5C6F3738
-P 13600 9100
-F 0 "D12" H 13600 8884 50  0000 C CNN
-F 1 "D" H 13600 8975 50  0000 C CNN
-F 2 "" H 13600 9100 50  0001 C CNN
-F 3 "~" H 13600 9100 50  0001 C CNN
-	1    13600 9100
-	-1   0    0    1
-$EndComp
 $Comp
 L BMS-Master-rescue:R-Device R178
@@
 	0    -1   -1   0
 $EndComp
-$Comp
-L Device:D D13
-U 1 1 5C6F4DA4
-P 13600 9800
-F 0 "D13" H 13600 9584 50  0000 C CNN
-F 1 "D" H 13600 9675 50  0000 C CNN
-F 2 "" H 13600 9800 50  0001 C CNN
-F 3 "~" H 13600 9800 50  0001 C CNN
-	1    13600 9800
-	-1   0    0    1
-$EndComp
 Wire Wire Line
 	13750 9800 14600 9800
@@
 P 15700 6400
 F 0 "L3" V 15890 6400 50  0000 C CNN
-F 1 "L" V 15799 6400 50  0000 C CNN
-F 2 "" H 15700 6400 50  0001 C CNN
+F 1 "744043151" V 15799 6400 50  0000 C CNN
+F 2 "Inductors_SMD:L_Wuerth_WE-PD2-Typ-MS" H 15700 6400 50  0001 C CNN
 F 3 "~" H 15700 6400 50  0001 C CNN
 	1    15700 6400
@@
 Wire Wire Line
 	13350 9100 13450 9100
-$Comp
-L Device:D D9
-U 1 1 5C7AB1AF
-P 12450 9800
-F 0 "D9" H 12450 10016 50  0000 C CNN
-F 1 "D" H 12450 9925 50  0000 C CNN
-F 2 "" H 12450 9800 50  0001 C CNN
-F 3 "~" H 12450 9800 50  0001 C CNN
-	1    12450 9800
-	1    0    0    -1
-$EndComp
 $Comp
 L BMS-Master-rescue:R-Device R174
@@
 Wire Wire Line
 	9650 10100 9650 10200
-$Comp
-L Device:D D7
-U 1 1 5C7CE51F
-P 10900 10550
-F 0 "D7" V 10854 10629 50  0000 L CNN
-F 1 "D" V 10945 10629 50  0000 L CNN
-F 2 "" H 10900 10550 50  0001 C CNN
-F 3 "~" H 10900 10550 50  0001 C CNN
-	1    10900 10550
-	0    1    1    0
-$EndComp
 Wire Wire Line
 	11400 10150 11200 10150
@@
 Wire Wire Line
 	9950 10400 10900 10400
-Connection ~ 10900 10400
 $Comp
 L BMS-Master-rescue:GND-power #PWR0264
@@
 Wire Wire Line
 	9650 10600 9650 10800
-$Comp
-L Device:D D8
-U 1 1 5C8020CB
-P 11250 9150
-F 0 "D8" H 11250 9366 50  0000 C CNN
-F 1 "D" H 11250 9275 50  0000 C CNN
-F 2 "" H 11250 9150 50  0001 C CNN
-F 3 "~" H 11250 9150 50  0001 C CNN
-	1    11250 9150
-	1    0    0    -1
-$EndComp
 $Comp
 L BMS-Master-rescue:R-Device R172
@@
 Wire Wire Line
 	1700 6650 3100 6650
+$Comp
+L Diode:1N4148W D?
+U 1 1 5C331B88
+P 13550 8500
+F 0 "D?" H 13550 8283 50  0000 C CNN
+F 1 "1N4148W" H 13550 8374 50  0000 C CNN
+F 2 "Diode_SMD:D_SOD-123" H 13550 8325 50  0001 C CNN
+F 3 "https://www.vishay.com/docs/85748/1n4148w.pdf" H 13550 8500 50  0001 C CNN
+	1    13550 8500
+	-1   0    0    1
+$EndComp
+$Comp
+L Diode:1N4148W D?
+U 1 1 5C332A77
+P 13600 9100
+F 0 "D?" H 13600 8883 50  0000 C CNN
+F 1 "1N4148W" H 13600 8974 50  0000 C CNN
+F 2 "Diode_SMD:D_SOD-123" H 13600 8925 50  0001 C CNN
+F 3 "https://www.vishay.com/docs/85748/1n4148w.pdf" H 13600 9100 50  0001 C CNN
+	1    13600 9100
+	-1   0    0    1
+$EndComp
+$Comp
+L Diode:1N4148W D?
+U 1 1 5C3330A4
+P 13600 9800
+F 0 "D?" H 13600 9583 50  0000 C CNN
+F 1 "1N4148W" H 13600 9674 50  0000 C CNN
+F 2 "Diode_SMD:D_SOD-123" H 13600 9625 50  0001 C CNN
+F 3 "https://www.vishay.com/docs/85748/1n4148w.pdf" H 13600 9800 50  0001 C CNN
+	1    13600 9800
+	-1   0    0    1
+$EndComp
+$Comp
+L Diode:1N4148W D?
+U 1 1 5C333552
+P 12450 9800
+F 0 "D?" H 12450 10017 50  0000 C CNN
+F 1 "1N4148W" H 12450 9926 50  0000 C CNN
+F 2 "Diode_SMD:D_SOD-123" H 12450 9625 50  0001 C CNN
+F 3 "https://www.vishay.com/docs/85748/1n4148w.pdf" H 12450 9800 50  0001 C CNN
+	1    12450 9800
+	1    0    0    -1
+$EndComp
+$Comp
+L Diode:1N4148W D?
+U 1 1 5C333C1D
+P 11250 9150
+F 0 "D?" H 11250 9367 50  0000 C CNN
+F 1 "1N4148W" H 11250 9276 50  0000 C CNN
+F 2 "Diode_SMD:D_SOD-123" H 11250 8975 50  0001 C CNN
+F 3 "https://www.vishay.com/docs/85748/1n4148w.pdf" H 11250 9150 50  0001 C CNN
+	1    11250 9150
+	1    0    0    -1
+$EndComp
+$Comp
+L Diode:BZT52Bxx D?
+U 1 1 5C334781
+P 10900 10550
+F 0 "D?" V 10854 10629 50  0000 L CNN
+F 1 "BZT52C16" V 10945 10629 50  0000 L CNN
+F 2 "Diode_SMD:D_SOD-123" H 10900 10375 50  0001 C CNN
+F 3 "https://diotec.com/tl_files/diotec/files/pdf/datasheets/bzt52b2v4.pdf" H 10900 10550 50  0001 C CNN
+	1    10900 10550
+	0    1    1    0
+$EndComp
+Connection ~ 10900 10400
+$Comp
+L Diode:BZT52Bxx D?
+U 1 1 5C339837
+P 13350 7400
+F 0 "D?" V 13304 7479 50  0000 L CNN
+F 1 "BZT52C16" V 13395 7479 50  0000 L CNN
+F 2 "Diode_SMD:D_SOD-123" H 13350 7225 50  0001 C CNN
+F 3 "https://diotec.com/tl_files/diotec/files/pdf/datasheets/bzt52b2v4.pdf" H 13350 7400 50  0001 C CNN
+	1    13350 7400
+	0    1    1    0
+$EndComp
 $EndSCHEMATC

Commit message: Schematics 99% completed
Only need to review everything &
Parts:
- gave numbers to parts that had none: 7
Connections:
- net +12V: now also C87.1
- net at JP22.1, L2.2: no longer C87.1
Other:
- moved on the sheet: C87
Changed lines of the file:
@@
 $EndComp
 Wire Wire Line
-	8750 6400 11000 6400
+	8750 6400 9250 6400
 Text HLabel 7900 5800 0    50   Input ~ 0
 ExternalPower
@@
 L BMS-Master-rescue:C-Device C87
 U 1 1 5C55039B
-P 6000 6950
-F 0 "C87" H 6115 6996 50  0000 L CNN
-F 1 "220u" H 6115 6905 50  0000 L CNN
-F 2 "Capacitors_SMD:CP_Elec_8x10" H 6038 6800 50  0001 C CNN
-F 3 "UWT1V221MNL1GS" H 6000 6950 50  0001 C CNN
-	1    6000 6950
-	1    0    0    -1
-$EndComp
-Wire Wire Line
-	6000 6650 6000 6800
-Wire Wire Line
-	5800 6650 6000 6650
-Wire Wire Line
-	5300 7150 6000 7150
-Wire Wire Line
-	6000 7150 6000 7100
+P 9250 6750
+F 0 "C87" H 9365 6796 50  0000 L CNN
+F 1 "220u" H 9365 6705 50  0000 L CNN
+F 2 "Capacitors_SMD:CP_Elec_8x10" H 9288 6600 50  0001 C CNN
+F 3 "UWT1V221MNL1GS" H 9250 6750 50  0001 C CNN
+	1    9250 6750
+	1    0    0    -1
+$EndComp
 Connection ~ 5300 7150
 $Comp
 L BMS-Master-rescue:GND-power #PWR0250
 U 1 1 5C580B9E
-P 6450 7200
-F 0 "#PWR0250" H 6450 6950 50  0001 C CNN
-F 1 "GND" H 6455 7027 50  0000 C CNN
-F 2 "" H 6450 7200 50  0001 C CNN
-F 3 "" H 6450 7200 50  0001 C CNN
-	1    6450 7200
-	1    0    0    -1
-$EndComp
-Wire Wire Line
-	6000 7150 6450 7150
-Wire Wire Line
-	6450 7150 6450 7200
-Connection ~ 6000 7150
-Connection ~ 6000 6650
+P 9650 7150
+F 0 "#PWR0250" H 9650 6900 50  0001 C CNN
+F 1 "GND" H 9655 6977 50  0000 C CNN
+F 2 "" H 9650 7150 50  0001 C CNN
+F 3 "" H 9650 7150 50  0001 C CNN
+	1    9650 7150
+	1    0    0    -1
+$EndComp
 Text HLabel 11200 5900 2    50   Input ~ 0
 +12V
@@
 Wire Wire Line
 	10950 9150 11100 9150
-Wire Wire Line
-	6000 6650 8650 6650
 NoConn ~ 14500 6700
 NoConn ~ 14500 6800
@@
 	1700 6650 3100 6650
 $Comp
-L Diode:1N4148W D?
+L Diode:1N4148W D11
 U 1 1 5C331B88
 P 13550 8500
-F 0 "D?" H 13550 8283 50  0000 C CNN
+F 0 "D11" H 13550 8283 50  0000 C CNN
 F 1 "1N4148W" H 13550 8374 50  0000 C CNN
 F 2 "Diode_SMD:D_SOD-123" H 13550 8325 50  0001 C CNN
@@
 $EndComp
 $Comp
-L Diode:1N4148W D?
+L Diode:1N4148W D12
 U 1 1 5C332A77
 P 13600 9100
-F 0 "D?" H 13600 8883 50  0000 C CNN
+F 0 "D12" H 13600 8883 50  0000 C CNN
 F 1 "1N4148W" H 13600 8974 50  0000 C CNN
 F 2 "Diode_SMD:D_SOD-123" H 13600 8925 50  0001 C CNN
@@
 $EndComp
 $Comp
-L Diode:1N4148W D?
+L Diode:1N4148W D13
 U 1 1 5C3330A4
 P 13600 9800
-F 0 "D?" H 13600 9583 50  0000 C CNN
+F 0 "D13" H 13600 9583 50  0000 C CNN
 F 1 "1N4148W" H 13600 9674 50  0000 C CNN
 F 2 "Diode_SMD:D_SOD-123" H 13600 9625 50  0001 C CNN
@@
 $EndComp
 $Comp
-L Diode:1N4148W D?
+L Diode:1N4148W D9
 U 1 1 5C333552
 P 12450 9800
-F 0 "D?" H 12450 10017 50  0000 C CNN
+F 0 "D9" H 12450 10017 50  0000 C CNN
 F 1 "1N4148W" H 12450 9926 50  0000 C CNN
 F 2 "Diode_SMD:D_SOD-123" H 12450 9625 50  0001 C CNN
@@
 $EndComp
 $Comp
-L Diode:1N4148W D?
+L Diode:1N4148W D8
 U 1 1 5C333C1D
 P 11250 9150
-F 0 "D?" H 11250 9367 50  0000 C CNN
+F 0 "D8" H 11250 9367 50  0000 C CNN
 F 1 "1N4148W" H 11250 9276 50  0000 C CNN
 F 2 "Diode_SMD:D_SOD-123" H 11250 8975 50  0001 C CNN
@@
 $EndComp
 $Comp
-L Diode:BZT52Bxx D?
+L Diode:BZT52Bxx D7
 U 1 1 5C334781
 P 10900 10550
-F 0 "D?" V 10854 10629 50  0000 L CNN
+F 0 "D7" V 10854 10629 50  0000 L CNN
 F 1 "BZT52C16" V 10945 10629 50  0000 L CNN
 F 2 "Diode_SMD:D_SOD-123" H 10900 10375 50  0001 C CNN
@@
 Connection ~ 10900 10400
 $Comp
-L Diode:BZT52Bxx D?
+L Diode:BZT52Bxx D10
 U 1 1 5C339837
 P 13350 7400
-F 0 "D?" V 13304 7479 50  0000 L CNN
+F 0 "D10" V 13304 7479 50  0000 L CNN
 F 1 "BZT52C16" V 13395 7479 50  0000 L CNN
 F 2 "Diode_SMD:D_SOD-123" H 13350 7225 50  0001 C CNN
@@
 	0    1    1    0
 $EndComp
+Wire Wire Line
+	9250 6400 9250 6600
+Connection ~ 9250 6400
+Wire Wire Line
+	9250 6400 11000 6400
+Wire Wire Line
+	9250 6900 9250 7150
+Connection ~ 9250 7150
+Wire Wire Line
+	9250 7150 9650 7150
+Wire Wire Line
+	5800 6650 8650 6650
+Wire Wire Line
+	5300 7150 9250 7150
 $EndSCHEMATC
