File: V0.2-LTC6813/BMS-Master/Temperature.sch (KiCad schematic (older format))
At the start: 25 parts

Commit message: V0.2 LTC6813 block
Parts:
- C? (x8): symbol Device:C -> BMS-Master-rescue:C-Device
- J?: symbol Connector_Generic:Conn_02x08_Counter_Clockwise -> BMS-Master-rescue:Conn_02x08_Counter_Clockwise-Connector_Generic
- R? (x16): symbol Device:R -> BMS-Master-rescue:R-Device
Changed lines of the file:
@@
 $EndDescr
 $Comp
-L Connector_Generic:Conn_02x08_Counter_Clockwise J?
+L BMS-Master-rescue:Conn_02x08_Counter_Clockwise-Connector_Generic J?
 U 1 1 5AEA9148
 P 8500 9050
@@
 $EndComp
 $Comp
-L power:GND #PWR?
+L BMS-Master-rescue:GND-power #PWR?
 U 1 1 5AEA9211
 P 7850 9650
@@
 	7850 9450 7850 9350
 $Comp
-L Device:R R?
+L BMS-Master-rescue:R-Device R?
 U 1 1 5AEA9568
 P 11450 3150
@@
 $EndComp
 $Comp
-L Device:R R?
+L BMS-Master-rescue:R-Device R?
 U 1 1 5AEA95F3
 P 10950 3350
@@
 	11450 3350 11100 3350
 $Comp
-L Device:C C?
+L BMS-Master-rescue:C-Device C?
 U 1 1 5AEA973B
 P 11450 3700
@@
 VP1
 $Comp
-L power:GND #PWR?
+L BMS-Master-rescue:GND-power #PWR?
 U 1 1 5AEA9CA3
 P 11450 3950
@@
 	11450 3850 11450 3950
 $Comp
-L Device:R R?
+L BMS-Master-rescue:R-Device R?
 U 1 1 5AEAA2B3
 P 11450 4600
@@
 $EndComp
 $Comp
-L Device:R R?
+L BMS-Master-rescue:R-Device R?
 U 1 1 5AEAA2B9
 P 10950 4800
@@
 	11450 4800 11100 4800
 $Comp
-L Device:C C?
+L BMS-Master-rescue:C-Device C?
 U 1 1 5AEAA2C2
 P 11450 5150
@@
 VP1
 $Comp
-L power:GND #PWR?
+L BMS-Master-rescue:GND-power #PWR?
 U 1 1 5AEAA2CF
 P 11450 5400
@@
 	11450 5300 11450 5400
 $Comp
-L Device:R R?
+L BMS-Master-rescue:R-Device R?
 U 1 1 5AEAA88D
 P 11450 5950
@@
 $EndComp
 $Comp
-L Device:R R?
+L BMS-Master-rescue:R-Device R?
 U 1 1 5AEAA893
 P 10950 6150
@@
 	11450 6150 11100 6150
 $Comp
-L Device:C C?
+L BMS-Master-rescue:C-Device C?
 U 1 1 5AEAA89C
 P 11450 6500
@@
 VP1
 $Comp
-L power:GND #PWR?
+L BMS-Master-rescue:GND-power #PWR?
 U 1 1 5AEAA8A9
 P 11450 6750
@@
 	11450 6650 11450 6750
 $Comp
-L Device:R R?
+L BMS-Master-rescue:R-Device R?
 U 1 1 5AEAA8B0
 P 11450 7400
@@
 $EndComp
 $Comp
-L Device:R R?
+L BMS-Master-rescue:R-Device R?
 U 1 1 5AEAA8B6
 P 10950 7600
@@
 	11450 7600 11100 7600
 $Comp
-L Device:C C?
+L BMS-Master-rescue:C-Device C?
 U 1 1 5AEAA8BF
 P 11450 7950
@@
 VP1
 $Comp
-L power:GND #PWR?
+L BMS-Master-rescue:GND-power #PWR?
 U 1 1 5AEAA8CC
 P 11450 8200
@@
 	11450 8100 11450 8200
 $Comp
-L Device:R R?
+L BMS-Master-rescue:R-Device R?
 U 1 1 5AEAB9E1
 P 11450 8750
@@
 $EndComp
 $Comp
-L Device:R R?
+L BMS-Master-rescue:R-Device R?
 U 1 1 5AEAB9E7
 P 10950 8950
@@
 	11450 8950 11100 8950
 $Comp
-L Device:C C?
+L BMS-Master-rescue:C-Device C?
 U 1 1 5AEAB9F0
 P 11450 9300
@@
 VP1
 $Comp
-L power:GND #PWR?
+L BMS-Master-rescue:GND-power #PWR?
 U 1 1 5AEAB9FD
 P 11450 9550
@@
 	11450 9450 11450 9550
 $Comp
-L Device:R R?
+L BMS-Master-rescue:R-Device R?
 U 1 1 5AEABA04
 P 11450 10200
@@
 $EndComp
 $Comp
-L Device:R R?
+L BMS-Master-rescue:R-Device R?
 U 1 1 5AEABA0A
 P 10950 10400
@@
 	11450 10400 11100 10400
 $Comp
-L Device:C C?
+L BMS-Master-rescue:C-Device C?
 U 1 1 5AEABA13
 P 11450 10750
@@
 VP1
 $Comp
-L power:GND #PWR?
+L BMS-Master-rescue:GND-power #PWR?
 U 1 1 5AEABA20
 P 11450 11000
@@
 	11450 10900 11450 11000
 $Comp
-L Device:R R?
+L BMS-Master-rescue:R-Device R?
 U 1 1 5AEABA27
 P 11450 11550
@@
 $EndComp
 $Comp
-L Device:R R?
+L BMS-Master-rescue:R-Device R?
 U 1 1 5AEABA2D
 P 10950 11750
@@
 	11450 11750 11100 11750
 $Comp
-L Device:C C?
+L BMS-Master-rescue:C-Device C?
 U 1 1 5AEABA36
 P 11450 12100
@@
 VP1
 $Comp
-L power:GND #PWR?
+L BMS-Master-rescue:GND-power #PWR?
 U 1 1 5AEABA43
 P 11450 12350
@@
 	11450 12250 11450 12350
 $Comp
-L Device:R R?
+L BMS-Master-rescue:R-Device R?
 U 1 1 5AEABA4A
 P 11450 13000
@@
 $EndComp
 $Comp
-L Device:R R?
+L BMS-Master-rescue:R-Device R?
 U 1 1 5AEABA50
 P 10950 13200
@@
 	11450 13200 11100 13200
 $Comp
-L Device:C C?
+L BMS-Master-rescue:C-Device C?
 U 1 1 5AEABA59
 P 11450 13550
@@
 VP1
 $Comp
-L power:GND #PWR?
+L BMS-Master-rescue:GND-power #PWR?
 U 1 1 5AEABA66
 P 11450 13800

Commit message: schematics 50% complete3d
Parts:
- removed J?: Conn_02x08_Counter_Clockwise, Pin_Headers:Pin_Header_Angled_2x08_Pitch2.54mm, symbol BMS-Master-rescue:Conn_02x08_Counter_Clockwise-Connector_Generic
- removed R? (x8): 10, Resistors_SMD:R_0603_HandSoldering, symbol BMS-Master-rescue:R-Device
- added C?: 0.1u, Capacitors_SMD:C_0603_HandSoldering, symbol BMS-Master-rescue:C-Device
- added R?: 10k, Resistors_SMD:R_0603_HandSoldering, symbol BMS-Master-rescue:R-Device
Connections:
- net labels added: AUX8, T0, T1, T2, T3, T4, T5, T6, T7, T8, VREF2
- wire segments 96 -> 81
Changed lines of the file:
@@
 EESchema Schematic File Version 4
 LIBS:BMS-Master-cache
-EELAYER 26 0
+EELAYER 29 0
 EELAYER END
 $Descr A2 23386 16535
 encoding utf-8
-Sheet 2 25
+Sheet 2 27
 Title "BMS-Master"
 Date ""
@@
 $EndDescr
 $Comp
-L BMS-Master-rescue:Conn_02x08_Counter_Clockwise-Connector_Generic J?
-U 1 1 5AEA9148
-P 8500 9050
-F 0 "J?" H 8550 9567 50  0000 C CNN
-F 1 "Conn_02x08_Counter_Clockwise" H 8550 9476 50  0000 C CNN
-F 2 "Pin_Headers:Pin_Header_Angled_2x08_Pitch2.54mm" H 8500 9050 50  0001 C CNN
-F 3 "~" H 8500 9050 50  0001 C CNN
-	1    8500 9050
-	1    0    0    -1
-$EndComp
-$Comp
-L BMS-Master-rescue:GND-power #PWR?
-U 1 1 5AEA9211
-P 7850 9650
-F 0 "#PWR?" H 7850 9400 50  0001 C CNN
-F 1 "GND" H 7855 9477 50  0000 C CNN
-F 2 "" H 7850 9650 50  0001 C CNN
-F 3 "" H 7850 9650 50  0001 C CNN
-	1    7850 9650
-	1    0    0    -1
-$EndComp
-Wire Wire Line
-	7850 9650 7850 9450
-Wire Wire Line
-	7850 8750 8300 8750
-Wire Wire Line
-	8300 8850 7850 8850
-Connection ~ 7850 8850
-Wire Wire Line
-	7850 8850 7850 8750
-Wire Wire Line
-	8300 8950 7850 8950
-Connection ~ 7850 8950
-Wire Wire Line
-	7850 8950 7850 8850
-Wire Wire Line
-	8300 9050 7850 9050
-Connection ~ 7850 9050
-Wire Wire Line
-	7850 9050 7850 8950
-Wire Wire Line
-	8300 9150 7850 9150
-Connection ~ 7850 9150
-Wire Wire Line
-	7850 9150 7850 9050
-Wire Wire Line
-	8300 9250 7850 9250
-Connection ~ 7850 9250
-Wire Wire Line
-	7850 9250 7850 9150
-Wire Wire Line
-	8300 9350 7850 9350
-Connection ~ 7850 9350
-Wire Wire Line
-	7850 9350 7850 9250
-Wire Wire Line
-	8300 9450 7850 9450
-Connection ~ 7850 9450
-Wire Wire Line
-	7850 9450 7850 9350
-$Comp
 L BMS-Master-rescue:R-Device R?
 U 1 1 5AEA9568
@@
 	1    0    0    -1
 $EndComp
-$Comp
-L BMS-Master-rescue:R-Device R?
-U 1 1 5AEA95F3
-P 10950 3350
-F 0 "R?" V 10743 3350 50  0000 C CNN
-F 1 "10" V 10834 3350 50  0000 C CNN
-F 2 "Resistors_SMD:R_0603_HandSoldering" V 10880 3350 50  0001 C CNN
-F 3 "~" H 10950 3350 50  0001 C CNN
-	1    10950 3350
-	0    1    1    0
-$EndComp
 Wire Wire Line
 	11450 3300 11450 3350
-Wire Wire Line
-	11450 3350 11100 3350
 $Comp
 L BMS-Master-rescue:C-Device C?
@@
 	1    0    0    -1
 $EndComp
-$Comp
-L BMS-Master-rescue:R-Device R?
-U 1 1 5AEAA2B9
-P 10950 4800
-F 0 "R?" V 10743 4800 50  0000 C CNN
-F 1 "10" V 10834 4800 50  0000 C CNN
-F 2 "Resistors_SMD:R_0603_HandSoldering" V 10880 4800 50  0001 C CNN
-F 3 "~" H 10950 4800 50  0001 C CNN
-	1    10950 4800
-	0    1    1    0
-$EndComp
 Wire Wire Line
 	11450 4750 11450 4800
-Wire Wire Line
-	11450 4800 11100 4800
 $Comp
 L BMS-Master-rescue:C-Device C?
@@
 	1    0    0    -1
 $EndComp
-$Comp
-L BMS-Master-rescue:R-Device R?
-U 1 1 5AEAA893
-P 10950 6150
-F 0 "R?" V 10743 6150 50  0000 C CNN
-F 1 "10" V 10834 6150 50  0000 C CNN
-F 2 "Resistors_SMD:R_0603_HandSoldering" V 10880 6150 50  0001 C CNN
-F 3 "~" H 10950 6150 50  0001 C CNN
-	1    10950 6150
-	0    1    1    0
-$EndComp
 Wire Wire Line
 	11450 6100 11450 6150
-Wire Wire Line
-	11450 6150 11100 6150
 $Comp
 L BMS-Master-rescue:C-Device C?
@@
 	1    0    0    -1
 $EndComp
-$Comp
-L BMS-Master-rescue:R-Device R?
-U 1 1 5AEAA8B6
-P 10950 7600
-F 0 "R?" V 10743 7600 50  0000 C CNN
-F 1 "10" V 10834 7600 50  0000 C CNN
-F 2 "Resistors_SMD:R_0603_HandSoldering" V 10880 7600 50  0001 C CNN
-F 3 "~" H 10950 7600 50  0001 C CNN
-	1    10950 7600
-	0    1    1    0
-$EndComp
 Wire Wire Line
 	11450 7550 11450 7600
-Wire Wire Line
-	11450 7600 11100 7600
 $Comp
 L BMS-Master-rescue:C-Device C?
@@
 	1    0    0    -1
 $EndComp
-$Comp
-L BMS-Master-rescue:R-Device R?
-U 1 1 5AEAB9E7
-P 10950 8950
-F 0 "R?" V 10743 8950 50  0000 C CNN
-F 1 "10" V 10834 8950 50  0000 C CNN
-F 2 "Resistors_SMD:R_0603_HandSoldering" V 10880 8950 50  0001 C CNN
-F 3 "~" H 10950 8950 50  0001 C CNN
-	1    10950 8950
-	0    1    1    0
-$EndComp
 Wire Wire Line
 	11450 8900 11450 8950
-Wire Wire Line
-	11450 8950 11100 8950
 $Comp
 L BMS-Master-rescue:C-Device C?
@@
 	1    0    0    -1
 $EndComp
-$Comp
-L BMS-Master-rescue:R-Device R?
-U 1 1 5AEABA0A
-P 10950 10400
-F 0 "R?" V 10743 10400 50  0000 C CNN
-F 1 "10" V 10834 10400 50  0000 C CNN
-F 2 "Resistors_SMD:R_0603_HandSoldering" V 10880 10400 50  0001 C CNN
-F 3 "~" H 10950 10400 50  0001 C CNN
-	1    10950 10400
-	0    1    1    0
-$EndComp
 Wire Wire Line
 	11450 10350 11450 10400
-Wire Wire Line
-	11450 10400 11100 10400
 $Comp
 L BMS-Master-rescue:C-Device C?
@@
 	1    0    0    -1
 $EndComp
-$Comp
-L BMS-Master-rescue:R-Device R?
-U 1 1 5AEABA2D
-P 10950 11750
-F 0 "R?" V 10743 11750 50  0000 C CNN
-F 1 "10" V 10834 11750 50  0000 C CNN
-F 2 "Resistors_SMD:R_0603_HandSoldering" V 10880 11750 50  0001 C CNN
-F 3 "~" H 10950 11750 50  0001 C CNN
-	1    10950 11750
-	0    1    1    0
-$EndComp
 Wire Wire Line
 	11450 11700 11450 11750
-Wire Wire Line
-	11450 11750 11100 11750
 $Comp
 L BMS-Master-rescue:C-Device C?
@@
 	1    0    0    -1
 $EndComp
-$Comp
-L BMS-Master-rescue:R-Device R?
-U 1 1 5AEABA50
-P 10950 13200
-F 0 "R?" V 10743 13200 50  0000 C CNN
-F 1 "10" V 10834 13200 50  0000 C CNN
-F 2 "Resistors_SMD:R_0603_HandSoldering" V 10880 13200 50  0001 C CNN
-F 3 "~" H 10950 13200 50  0001 C CNN
-	1    10950 13200
-	0    1    1    0
-$EndComp
 Wire Wire Line
 	11450 13150 11450 13200
-Wire Wire Line
-	11450 13200 11100 13200
 $Comp
 L BMS-Master-rescue:C-Device C?
@@
 	11450 13700 11450 13800
 Wire Wire Line
-	10800 3350 9350 3350
-Wire Wire Line
 	9350 3350 9350 8750
 Wire Wire Line
 	9350 8750 8800 8750
 Wire Wire Line
-	10800 4800 9450 4800
-Wire Wire Line
 	9450 4800 9450 8850
 Wire Wire Line
 	9450 8850 8800 8850
 Wire Wire Line
-	10800 6150 9550 6150
-Wire Wire Line
 	9550 6150 9550 8950
 Wire Wire Line
 	9550 8950 8800 8950
 Wire Wire Line
-	10800 7600 9650 7600
-Wire Wire Line
 	9650 7600 9650 9050
 Wire Wire Line
 	9650 9050 8800 9050
 Wire Wire Line
-	10800 8950 9750 8950
-Wire Wire Line
 	9750 8950 9750 9150
 Wire Wire Line
 	9750 9150 8800 9150
 Wire Wire Line
-	10800 10400 9750 10400
-Wire Wire Line
 	9750 10400 9750 9250
 Wire Wire Line
 	9750 9250 8800 9250
 Wire Wire Line
-	10800 11750 9650 11750
-Wire Wire Line
 	9650 11750 9650 9350
 Wire Wire Line
 	9650 9350 8800 9350
 Wire Wire Line
-	10800 13200 9550 13200
-Wire Wire Line
 	9550 13200 9550 9450
 Wire Wire Line
 	9550 9450 8800 9450
+$Comp
+L BMS-Master-rescue:R-Device R?
+U 1 1 5BF1E9E7
+P 11450 1750
+F 0 "R?" H 11520 1796 50  0000 L CNN
+F 1 "10k" H 11520 1705 50  0000 L CNN
+F 2 "Resistors_SMD:R_0603_HandSoldering" V 11380 1750 50  0001 C CNN
+F 3 "~" H 11450 1750 50  0001 C CNN
+	1    11450 1750
+	1    0    0    -1
+$EndComp
+Wire Wire Line
+	11450 1900 11450 1950
+$Comp
+L BMS-Master-rescue:C-Device C?
+U 1 1 5BF1E9F8
+P 11450 2300
+F 0 "C?" H 11565 2346 50  0000 L CNN
+F 1 "0.1u" H 11565 2255 50  0000 L CNN
+F 2 "Capacitors_SMD:C_0603_HandSoldering" H 11488 2150 50  0001 C CNN
+F 3 "~" H 11450 2300 50  0001 C CNN
+F 4 "50V" H 11450 2300 50  0001 C CNN "Volatge"
+	1    11450 2300
+	1    0    0    -1
+$EndComp
+Wire Wire Line
+	11450 2150 11450 1950
+Connection ~ 11450 1950
+Text HLabel 11850 1950 2    50   Output ~ 0
+AUX8
+Wire Wire Line
+	11450 1950 11850 1950
+Wire Wire Line
+	11450 1600 11450 1500
+Text Label 10900 1500 0    50   ~ 0
+VP1
+$Comp
+L BMS-Master-rescue:GND-power #PWR?
+U 1 1 5BF1EA06
+P 11450 2550
+F 0 "#PWR?" H 11450 2300 50  0001 C CNN
+F 1 "GND" H 11455 2377 50  0000 C CNN
+F 2 "" H 11450 2550 50  0001 C CNN
+F 3 "" H 11450 2550 50  0001 C CNN
+	1    11450 2550
+	1    0    0    -1
+$EndComp
+Wire Wire Line
+	11450 2450 11450 2550
+Wire Wire Line
+	9250 1950 9250 8650
+Wire Wire Line
+	9250 8650 8800 8650
+Text HLabel 8550 1500 0    50   Input ~ 0
+VREF2
+Wire Wire Line
+	8550 1500 11450 1500
+Wire Wire Line
+	9550 13200 11450 13200
+Wire Wire Line
+	9650 11750 11450 11750
+Wire Wire Line
+	9750 10400 11450 10400
+Wire Wire Line
+	9750 8950 11450 8950
+Wire Wire Line
+	9650 7600 11450 7600
+Wire Wire Line
+	9550 6150 11450 6150
+Wire Wire Line
+	9450 4800 11450 4800
+Wire Wire Line
+	9250 1950 11450 1950
+Wire Wire Line
+	9350 3350 11450 3350
+Text HLabel 8800 8650 0    50   Output ~ 0
+T8
+Text HLabel 8800 8750 0    50   Output ~ 0
+T7
+Text HLabel 8800 8850 0    50   Output ~ 0
+T6
+Text HLabel 8800 8950 0    50   Output ~ 0
+T5
+Text HLabel 8800 9050 0    50   Output ~ 0
+T4
+Text HLabel 8800 9150 0    50   Output ~ 0
+T3
+Text HLabel 8800 9250 0    50   Output ~ 0
+T2
+Text HLabel 8800 9350 0    50   Output ~ 0
+T1
+Text HLabel 8800 9450 0    50   Output ~ 0
+T0
 $EndSCHEMATC

Commit message: Schematics 75% completed
Connections:
- net GND renamed GNDA
Changed lines of the file:
@@
 Text Label 10900 2900 0    50   ~ 0
 VP1
-$Comp
-L BMS-Master-rescue:GND-power #PWR?
-U 1 1 5AEA9CA3
-P 11450 3950
-F 0 "#PWR?" H 11450 3700 50  0001 C CNN
-F 1 "GND" H 11455 3777 50  0000 C CNN
-F 2 "" H 11450 3950 50  0001 C CNN
-F 3 "" H 11450 3950 50  0001 C CNN
-	1    11450 3950
-	1    0    0    -1
-$EndComp
 Wire Wire Line
 	11450 3850 11450 3950
@@
 Text Label 10900 4350 0    50   ~ 0
 VP1
-$Comp
-L BMS-Master-rescue:GND-power #PWR?
-U 1 1 5AEAA2CF
-P 11450 5400
-F 0 "#PWR?" H 11450 5150 50  0001 C CNN
-F 1 "GND" H 11455 5227 50  0000 C CNN
-F 2 "" H 11450 5400 50  0001 C CNN
-F 3 "" H 11450 5400 50  0001 C CNN
-	1    11450 5400
-	1    0    0    -1
-$EndComp
 Wire Wire Line
 	11450 5300 11450 5400
@@
 Text Label 10900 5700 0    50   ~ 0
 VP1
-$Comp
-L BMS-Master-rescue:GND-power #PWR?
-U 1 1 5AEAA8A9
-P 11450 6750
-F 0 "#PWR?" H 11450 6500 50  0001 C CNN
-F 1 "GND" H 11455 6577 50  0000 C CNN
-F 2 "" H 11450 6750 50  0001 C CNN
-F 3 "" H 11450 6750 50  0001 C CNN
-	1    11450 6750
-	1    0    0    -1
-$EndComp
 Wire Wire Line
 	11450 6650 11450 6750
@@
 Text Label 10900 7150 0    50   ~ 0
 VP1
-$Comp
-L BMS-Master-rescue:GND-power #PWR?
-U 1 1 5AEAA8CC
-P 11450 8200
-F 0 "#PWR?" H 11450 7950 50  0001 C CNN
-F 1 "GND" H 11455 8027 50  0000 C CNN
-F 2 "" H 11450 8200 50  0001 C CNN
-F 3 "" H 11450 8200 50  0001 C CNN
-	1    11450 8200
-	1    0    0    -1
-$EndComp
 Wire Wire Line
 	11450 8100 11450 8200
@@
 Text Label 10900 8500 0    50   ~ 0
 VP1
-$Comp
-L BMS-Master-rescue:GND-power #PWR?
-U 1 1 5AEAB9FD
-P 11450 9550
-F 0 "#PWR?" H 11450 9300 50  0001 C CNN
-F 1 "GND" H 11455 9377 50  0000 C CNN
-F 2 "" H 11450 9550 50  0001 C CNN
-F 3 "" H 11450 9550 50  0001 C CNN
-	1    11450 9550
-	1    0    0    -1
-$EndComp
 Wire Wire Line
 	11450 9450 11450 9550
@@
 Text Label 10900 9950 0    50   ~ 0
 VP1
-$Comp
-L BMS-Master-rescue:GND-power #PWR?
-U 1 1 5AEABA20
-P 11450 11000
-F 0 "#PWR?" H 11450 10750 50  0001 C CNN
-F 1 "GND" H 11455 10827 50  0000 C CNN
-F 2 "" H 11450 11000 50  0001 C CNN
-F 3 "" H 11450 11000 50  0001 C CNN
-	1    11450 11000
-	1    0    0    -1
-$EndComp
 Wire Wire Line
 	11450 10900 11450 11000
@@
 Text Label 10900 11300 0    50   ~ 0
 VP1
-$Comp
-L BMS-Master-rescue:GND-power #PWR?
-U 1 1 5AEABA43
-P 11450 12350
-F 0 "#PWR?" H 11450 12100 50  0001 C CNN
-F 1 "GND" H 11455 12177 50  0000 C CNN
-F 2 "" H 11450 12350 50  0001 C CNN
-F 3 "" H 11450 12350 50  0001 C CNN
-	1    11450 12350
-	1    0    0    -1
-$EndComp
 Wire Wire Line
 	11450 12250 11450 12350
@@
 Text Label 10900 12750 0    50   ~ 0
 VP1
-$Comp
-L BMS-Master-rescue:GND-power #PWR?
-U 1 1 5AEABA66
-P 11450 13800
-F 0 "#PWR?" H 11450 13550 50  0001 C CNN
-F 1 "GND" H 11455 13627 50  0000 C CNN
-F 2 "" H 11450 13800 50  0001 C CNN
-F 3 "" H 11450 13800 50  0001 C CNN
-	1    11450 13800
-	1    0    0    -1
-$EndComp
 Wire Wire Line
 	11450 13700 11450 13800
@@
 Text Label 10900 1500 0    50   ~ 0
 VP1
-$Comp
-L BMS-Master-rescue:GND-power #PWR?
-U 1 1 5BF1EA06
-P 11450 2550
-F 0 "#PWR?" H 11450 2300 50  0001 C CNN
-F 1 "GND" H 11455 2377 50  0000 C CNN
-F 2 "" H 11450 2550 50  0001 C CNN
-F 3 "" H 11450 2550 50  0001 C CNN
-	1    11450 2550
-	1    0    0    -1
-$EndComp
 Wire Wire Line
 	11450 2450 11450 2550
@@
 Text HLabel 8800 9450 0    50   Output ~ 0
 T0
+$Comp
+L power:GNDA #PWR?
+U 1 1 5C8C5E65
+P 11450 2550
+F 0 "#PWR?" H 11450 2300 50  0001 C CNN
+F 1 "GNDA" H 11455 2377 50  0000 C CNN
+F 2 "" H 11450 2550 50  0001 C CNN
+F 3 "" H 11450 2550 50  0001 C CNN
+	1    11450 2550
+	1    0    0    -1
+$EndComp
+$Comp
+L power:GNDA #PWR?
+U 1 1 5C8C630F
+P 11450 3950
+F 0 "#PWR?" H 11450 3700 50  0001 C CNN
+F 1 "GNDA" H 11455 3777 50  0000 C CNN
+F 2 "" H 11450 3950 50  0001 C CNN
+F 3 "" H 11450 3950 50  0001 C CNN
+	1    11450 3950
+	1    0    0    -1
+$EndComp
+$Comp
+L power:GNDA #PWR?
+U 1 1 5C8C66F7
+P 11450 5400
+F 0 "#PWR?" H 11450 5150 50  0001 C CNN
+F 1 "GNDA" H 11455 5227 50  0000 C CNN
+F 2 "" H 11450 5400 50  0001 C CNN
+F 3 "" H 11450 5400 50  0001 C CNN
+	1    11450 5400
+	1    0    0    -1
+$EndComp
+$Comp
+L power:GNDA #PWR?
+U 1 1 5C8C69B9
+P 11450 6750
+F 0 "#PWR?" H 11450 6500 50  0001 C CNN
+F 1 "GNDA" H 11455 6577 50  0000 C CNN
+F 2 "" H 11450 6750 50  0001 C CNN
+F 3 "" H 11450 6750 50  0001 C CNN
+	1    11450 6750
+	1    0    0    -1
+$EndComp
+$Comp
+L power:GNDA #PWR?
+U 1 1 5C8C6C83
+P 11450 8200
+F 0 "#PWR?" H 11450 7950 50  0001 C CNN
+F 1 "GNDA" H 11455 8027 50  0000 C CNN
+F 2 "" H 11450 8200 50  0001 C CNN
+F 3 "" H 11450 8200 50  0001 C CNN
+	1    11450 8200
+	1    0    0    -1
+$EndComp
+$Comp
+L power:GNDA #PWR?
+U 1 1 5C8C6FDD
+P 11450 9550
+F 0 "#PWR?" H 11450 9300 50  0001 C CNN
+F 1 "GNDA" H 11455 9377 50  0000 C CNN
+F 2 "" H 11450 9550 50  0001 C CNN
+F 3 "" H 11450 9550 50  0001 C CNN
+	1    11450 9550
+	1    0    0    -1
+$EndComp
+$Comp
+L power:GNDA #PWR?
+U 1 1 5C8C726A
+P 11450 11000
+F 0 "#PWR?" H 11450 10750 50  0001 C CNN
+F 1 "GNDA" H 11455 10827 50  0000 C CNN
+F 2 "" H 11450 11000 50  0001 C CNN
+F 3 "" H 11450 11000 50  0001 C CNN
+	1    11450 11000
+	1    0    0    -1
+$EndComp
+$Comp
+L power:GNDA #PWR?
+U 1 1 5C8C7637
+P 11450 12350
+F 0 "#PWR?" H 11450 12100 50  0001 C CNN
+F 1 "GNDA" H 11455 12177 50  0000 C CNN
+F 2 "" H 11450 12350 50  0001 C CNN
+F 3 "" H 11450 12350 50  0001 C CNN
+	1    11450 12350
+	1    0    0    -1
+$EndComp
+$Comp
+L power:GNDA #PWR?
+U 1 1 5C8C7939
+P 11450 13800
+F 0 "#PWR?" H 11450 13550 50  0001 C CNN
+F 1 "GNDA" H 11455 13627 50  0000 C CNN
+F 2 "" H 11450 13800 50  0001 C CNN
+F 3 "" H 11450 13800 50  0001 C CNN
+	1    11450 13800
+	1    0    0    -1
+$EndComp
 $EndSCHEMATC
