File: V0.2-LTC6813/BMS-Master/Temperature.sch (KiCad schematic (older format))
At the start: 18 parts

Commit message: Schematics 90% completed
Parts:
- gave numbers to parts that had none: 18
Changed lines of the file:
@@
 $EndDescr
 $Comp
-L BMS-Master-rescue:R-Device R?
+L BMS-Master-rescue:R-Device R7
 U 1 1 5AEA9568
 P 11450 3150
-F 0 "R?" H 11520 3196 50  0000 L CNN
+F 0 "R7" H 11520 3196 50  0000 L CNN
 F 1 "10k" H 11520 3105 50  0000 L CNN
 F 2 "Resistors_SMD:R_0603_HandSoldering" V 11380 3150 50  0001 C CNN
@@
 	11450 3300 11450 3350
 $Comp
-L BMS-Master-rescue:C-Device C?
+L BMS-Master-rescue:C-Device C2
 U 1 1 5AEA973B
 P 11450 3700
-F 0 "C?" H 11565 3746 50  0000 L CNN
+F 0 "C2" H 11565 3746 50  0000 L CNN
 F 1 "0.1u" H 11565 3655 50  0000 L CNN
 F 2 "Capacitors_SMD:C_0603_HandSoldering" H 11488 3550 50  0001 C CNN
@@
 	11450 3850 11450 3950
 $Comp
-L BMS-Master-rescue:R-Device R?
+L BMS-Master-rescue:R-Device R8
 U 1 1 5AEAA2B3
 P 11450 4600
-F 0 "R?" H 11520 4646 50  0000 L CNN
+F 0 "R8" H 11520 4646 50  0000 L CNN
 F 1 "10k" H 11520 4555 50  0000 L CNN
 F 2 "Resistors_SMD:R_0603_HandSoldering" V 11380 4600 50  0001 C CNN
@@
 	11450 4750 11450 4800
 $Comp
-L BMS-Master-rescue:C-Device C?
+L BMS-Master-rescue:C-Device C3
 U 1 1 5AEAA2C2
 P 11450 5150
-F 0 "C?" H 11565 5196 50  0000 L CNN
+F 0 "C3" H 11565 5196 50  0000 L CNN
 F 1 "0.1u" H 11565 5105 50  0000 L CNN
 F 2 "Capacitors_SMD:C_0603_HandSoldering" H 11488 5000 50  0001 C CNN
@@
 	11450 5300 11450 5400
 $Comp
-L BMS-Master-rescue:R-Device R?
+L BMS-Master-rescue:R-Device R9
 U 1 1 5AEAA88D
 P 11450 5950
-F 0 "R?" H 11520 5996 50  0000 L CNN
+F 0 "R9" H 11520 5996 50  0000 L CNN
 F 1 "10k" H 11520 5905 50  0000 L CNN
 F 2 "Resistors_SMD:R_0603_HandSoldering" V 11380 5950 50  0001 C CNN
@@
 	11450 6100 11450 6150
 $Comp
-L BMS-Master-rescue:C-Device C?
+L BMS-Master-rescue:C-Device C4
 U 1 1 5AEAA89C
 P 11450 6500
-F 0 "C?" H 11565 6546 50  0000 L CNN
+F 0 "C4" H 11565 6546 50  0000 L CNN
 F 1 "0.1u" H 11565 6455 50  0000 L CNN
 F 2 "Capacitors_SMD:C_0603_HandSoldering" H 11488 6350 50  0001 C CNN
@@
 	11450 6650 11450 6750
 $Comp
-L BMS-Master-rescue:R-Device R?
+L BMS-Master-rescue:R-Device R10
 U 1 1 5AEAA8B0
 P 11450 7400
-F 0 "R?" H 11520 7446 50  0000 L CNN
+F 0 "R10" H 11520 7446 50  0000 L CNN
 F 1 "10k" H 11520 7355 50  0000 L CNN
 F 2 "Resistors_SMD:R_0603_HandSoldering" V 11380 7400 50  0001 C CNN
@@
 	11450 7550 11450 7600
 $Comp
-L BMS-Master-rescue:C-Device C?
+L BMS-Master-rescue:C-Device C5
 U 1 1 5AEAA8BF
 P 11450 7950
-F 0 "C?" H 11565 7996 50  0000 L CNN
+F 0 "C5" H 11565 7996 50  0000 L CNN
 F 1 "0.1u" H 11565 7905 50  0000 L CNN
 F 2 "Capacitors_SMD:C_0603_HandSoldering" H 11488 7800 50  0001 C CNN
@@
 	11450 8100 11450 8200
 $Comp
-L BMS-Master-rescue:R-Device R?
+L BMS-Master-rescue:R-Device R11
 U 1 1 5AEAB9E1
 P 11450 8750
-F 0 "R?" H 11520 8796 50  0000 L CNN
+F 0 "R11" H 11520 8796 50  0000 L CNN
 F 1 "10k" H 11520 8705 50  0000 L CNN
 F 2 "Resistors_SMD:R_0603_HandSoldering" V 11380 8750 50  0001 C CNN
@@
 	11450 8900 11450 8950
 $Comp
-L BMS-Master-rescue:C-Device C?
+L BMS-Master-rescue:C-Device C6
 U 1 1 5AEAB9F0
 P 11450 9300
-F 0 "C?" H 11565 9346 50  0000 L CNN
+F 0 "C6" H 11565 9346 50  0000 L CNN
 F 1 "0.1u" H 11565 9255 50  0000 L CNN
 F 2 "Capacitors_SMD:C_0603_HandSoldering" H 11488 9150 50  0001 C CNN
@@
 	11450 9450 11450 9550
 $Comp
-L BMS-Master-rescue:R-Device R?
+L BMS-Master-rescue:R-Device R12
 U 1 1 5AEABA04
 P 11450 10200
-F 0 "R?" H 11520 10246 50  0000 L CNN
+F 0 "R12" H 11520 10246 50  0000 L CNN
 F 1 "10k" H 11520 10155 50  0000 L CNN
 F 2 "Resistors_SMD:R_0603_HandSoldering" V 11380 10200 50  0001 C CNN
@@
 	11450 10350 11450 10400
 $Comp
-L BMS-Master-rescue:C-Device C?
+L BMS-Master-rescue:C-Device C7
 U 1 1 5AEABA13
 P 11450 10750
-F 0 "C?" H 11565 10796 50  0000 L CNN
+F 0 "C7" H 11565 10796 50  0000 L CNN
 F 1 "0.1u" H 11565 10705 50  0000 L CNN
 F 2 "Capacitors_SMD:C_0603_HandSoldering" H 11488 10600 50  0001 C CNN
@@
 Text Label 10900 9950 0    50   ~ 0
 VP1
-Wire Wire Line
-	11450 10900 11450 11000
-$Comp
-L BMS-Master-rescue:R-Device R?
+$Comp
+L BMS-Master-rescue:R-Device R13
 U 1 1 5AEABA27
 P 11450 11550
-F 0 "R?" H 11520 11596 50  0000 L CNN
+F 0 "R13" H 11520 11596 50  0000 L CNN
 F 1 "10k" H 11520 11505 50  0000 L CNN
 F 2 "Resistors_SMD:R_0603_HandSoldering" V 11380 11550 50  0001 C CNN
@@
 	11450 11700 11450 11750
 $Comp
-L BMS-Master-rescue:C-Device C?
+L BMS-Master-rescue:C-Device C8
 U 1 1 5AEABA36
 P 11450 12100
-F 0 "C?" H 11565 12146 50  0000 L CNN
+F 0 "C8" H 11565 12146 50  0000 L CNN
 F 1 "0.1u" H 11565 12055 50  0000 L CNN
 F 2 "Capacitors_SMD:C_0603_HandSoldering" H 11488 11950 50  0001 C CNN
@@
 	11450 12250 11450 12350
 $Comp
-L BMS-Master-rescue:R-Device R?
+L BMS-Master-rescue:R-Device R14
 U 1 1 5AEABA4A
 P 11450 13000
-F 0 "R?" H 11520 13046 50  0000 L CNN
+F 0 "R14" H 11520 13046 50  0000 L CNN
 F 1 "10k" H 11520 12955 50  0000 L CNN
 F 2 "Resistors_SMD:R_0603_HandSoldering" V 11380 13000 50  0001 C CNN
@@
 	11450 13150 11450 13200
 $Comp
-L BMS-Master-rescue:C-Device C?
+L BMS-Master-rescue:C-Device C9
 U 1 1 5AEABA59
 P 11450 13550
-F 0 "C?" H 11565 13596 50  0000 L CNN
+F 0 "C9" H 11565 13596 50  0000 L CNN
 F 1 "0.1u" H 11565 13505 50  0000 L CNN
 F 2 "Capacitors_SMD:C_0603_HandSoldering" H 11488 13400 50  0001 C CNN
@@
 	9550 9450 8800 9450
 $Comp
-L BMS-Master-rescue:R-Device R?
+L BMS-Master-rescue:R-Device R6
 U 1 1 5BF1E9E7
 P 11450 1750
-F 0 "R?" H 11520 1796 50  0000 L CNN
+F 0 "R6" H 11520 1796 50  0000 L CNN
 F 1 "10k" H 11520 1705 50  0000 L CNN
 F 2 "Resistors_SMD:R_0603_HandSoldering" V 11380 1750 50  0001 C CNN
@@
 	11450 1900 11450 1950
 $Comp
-L BMS-Master-rescue:C-Device C?
+L BMS-Master-rescue:C-Device C1
 U 1 1 5BF1E9F8
 P 11450 2300
-F 0 "C?" H 11565 2346 50  0000 L CNN
+F 0 "C1" H 11565 2346 50  0000 L CNN
 F 1 "0.1u" H 11565 2255 50  0000 L CNN
 F 2 "Capacitors_SMD:C_0603_HandSoldering" H 11488 2150 50  0001 C CNN
@@
 T0
 $Comp
-L power:GNDA #PWR?
+L power:GNDA #PWR0117
 U 1 1 5C8C5E65
 P 11450 2550
-F 0 "#PWR?" H 11450 2300 50  0001 C CNN
+F 0 "#PWR0117" H 11450 2300 50  0001 C CNN
 F 1 "GNDA" H 11455 2377 50  0000 C CNN
 F 2 "" H 11450 2550 50  0001 C CNN
@@
 $EndComp
 $Comp
-L power:GNDA #PWR?
+L power:GNDA #PWR0118
 U 1 1 5C8C630F
 P 11450 3950
-F 0 "#PWR?" H 11450 3700 50  0001 C CNN
+F 0 "#PWR0118" H 11450 3700 50  0001 C CNN
 F 1 "GNDA" H 11455 3777 50  0000 C CNN
 F 2 "" H 11450 3950 50  0001 C CNN
@@
 $EndComp
 $Comp
-L power:GNDA #PWR?
+L power:GNDA #PWR0119
 U 1 1 5C8C66F7
 P 11450 5400
-F 0 "#PWR?" H 11450 5150 50  0001 C CNN
+F 0 "#PWR0119" H 11450 5150 50  0001 C CNN
 F 1 "GNDA" H 11455 5227 50  0000 C CNN
 F 2 "" H 11450 5400 50  0001 C CNN
@@
 $EndComp
 $Comp
-L power:GNDA #PWR?
+L power:GNDA #PWR0120
 U 1 1 5C8C69B9
 P 11450 6750
-F 0 "#PWR?" H 11450 6500 50  0001 C CNN
+F 0 "#PWR0120" H 11450 6500 50  0001 C CNN
 F 1 "GNDA" H 11455 6577 50  0000 C CNN
 F 2 "" H 11450 6750 50  0001 C CNN
@@
 $EndComp
 $Comp
-L power:GNDA #PWR?
+L power:GNDA #PWR0121
 U 1 1 5C8C6C83
 P 11450 8200
-F 0 "#PWR?" H 11450 7950 50  0001 C CNN
+F 0 "#PWR0121" H 11450 7950 50  0001 C CNN
 F 1 "GNDA" H 11455 8027 50  0000 C CNN
 F 2 "" H 11450 8200 50  0001 C CNN
@@
 $EndComp
 $Comp
-L power:GNDA #PWR?
+L power:GNDA #PWR0122
 U 1 1 5C8C6FDD
 P 11450 9550
-F 0 "#PWR?" H 11450 9300 50  0001 C CNN
+F 0 "#PWR0122" H 11450 9300 50  0001 C CNN
 F 1 "GNDA" H 11455 9377 50  0000 C CNN
 F 2 "" H 11450 9550 50  0001 C CNN
@@
 $EndComp
 $Comp
-L power:GNDA #PWR?
+L power:GNDA #PWR0123
 U 1 1 5C8C726A
 P 11450 11000
-F 0 "#PWR?" H 11450 10750 50  0001 C CNN
+F 0 "#PWR0123" H 11450 10750 50  0001 C CNN
 F 1 "GNDA" H 11455 10827 50  0000 C CNN
 F 2 "" H 11450 11000 50  0001 C CNN
@@
 $EndComp
 $Comp
-L power:GNDA #PWR?
+L power:GNDA #PWR0124
 U 1 1 5C8C7637
 P 11450 12350
-F 0 "#PWR?" H 11450 12100 50  0001 C CNN
+F 0 "#PWR0124" H 11450 12100 50  0001 C CNN
 F 1 "GNDA" H 11455 12177 50  0000 C CNN
 F 2 "" H 11450 12350 50  0001 C CNN
@@
 $EndComp
 $Comp
-L power:GNDA #PWR?
+L power:GNDA #PWR0125
 U 1 1 5C8C7939
 P 11450 13800
-F 0 "#PWR?" H 11450 13550 50  0001 C CNN
+F 0 "#PWR0125" H 11450 13550 50  0001 C CNN
 F 1 "GNDA" H 11455 13627 50  0000 C CNN
 F 2 "" H 11450 13800 50  0001 C CNN
@@
 	1    0    0    -1
 $EndComp
+Wire Wire Line
+	11450 10900 11450 11000
 $EndSCHEMATC

Commit message: Now master & slave are on  separate boards
Connections:
- net GNDA renamed GNDREF
Changed lines of the file:
@@
 Text HLabel 8800 9450 0    50   Output ~ 0
 T0
+Wire Wire Line
+	11450 10900 11450 11000
 $Comp
-L power:GNDA #PWR0117
-U 1 1 5C8C5E65
+L power:GNDREF #PWR0117
+U 1 1 5C77BBEC
 P 11450 2550
 F 0 "#PWR0117" H 11450 2300 50  0001 C CNN
-F 1 "GNDA" H 11455 2377 50  0000 C CNN
+F 1 "GNDREF" H 11455 2377 50  0000 C CNN
 F 2 "" H 11450 2550 50  0001 C CNN
 F 3 "" H 11450 2550 50  0001 C CNN
@@
 $EndComp
 $Comp
-L power:GNDA #PWR0118
-U 1 1 5C8C630F
+L power:GNDREF #PWR0118
+U 1 1 5C77C4DE
 P 11450 3950
 F 0 "#PWR0118" H 11450 3700 50  0001 C CNN
-F 1 "GNDA" H 11455 3777 50  0000 C CNN
+F 1 "GNDREF" H 11455 3777 50  0000 C CNN
 F 2 "" H 11450 3950 50  0001 C CNN
 F 3 "" H 11450 3950 50  0001 C CNN
@@
 $EndComp
 $Comp
-L power:GNDA #PWR0119
-U 1 1 5C8C66F7
+L power:GNDREF #PWR0119
+U 1 1 5C77CE41
 P 11450 5400
 F 0 "#PWR0119" H 11450 5150 50  0001 C CNN
-F 1 "GNDA" H 11455 5227 50  0000 C CNN
+F 1 "GNDREF" H 11455 5227 50  0000 C CNN
 F 2 "" H 11450 5400 50  0001 C CNN
 F 3 "" H 11450 5400 50  0001 C CNN
@@
 $EndComp
 $Comp
-L power:GNDA #PWR0120
-U 1 1 5C8C69B9
+L power:GNDREF #PWR0120
+U 1 1 5C77D999
 P 11450 6750
 F 0 "#PWR0120" H 11450 6500 50  0001 C CNN
-F 1 "GNDA" H 11455 6577 50  0000 C CNN
+F 1 "GNDREF" H 11455 6577 50  0000 C CNN
 F 2 "" H 11450 6750 50  0001 C CNN
 F 3 "" H 11450 6750 50  0001 C CNN
@@
 $EndComp
 $Comp
-L power:GNDA #PWR0121
-U 1 1 5C8C6C83
+L power:GNDREF #PWR0121
+U 1 1 5C77E07A
 P 11450 8200
 F 0 "#PWR0121" H 11450 7950 50  0001 C CNN
-F 1 "GNDA" H 11455 8027 50  0000 C CNN
+F 1 "GNDREF" H 11455 8027 50  0000 C CNN
 F 2 "" H 11450 8200 50  0001 C CNN
 F 3 "" H 11450 8200 50  0001 C CNN
@@
 $EndComp
 $Comp
-L power:GNDA #PWR0122
-U 1 1 5C8C6FDD
+L power:GNDREF #PWR0122
+U 1 1 5C77E6D8
 P 11450 9550
 F 0 "#PWR0122" H 11450 9300 50  0001 C CNN
-F 1 "GNDA" H 11455 9377 50  0000 C CNN
+F 1 "GNDREF" H 11455 9377 50  0000 C CNN
 F 2 "" H 11450 9550 50  0001 C CNN
 F 3 "" H 11450 9550 50  0001 C CNN
@@
 $EndComp
 $Comp
-L power:GNDA #PWR0123
-U 1 1 5C8C726A
+L power:GNDREF #PWR0123
+U 1 1 5C77EC81
 P 11450 11000
 F 0 "#PWR0123" H 11450 10750 50  0001 C CNN
-F 1 "GNDA" H 11455 10827 50  0000 C CNN
+F 1 "GNDREF" H 11455 10827 50  0000 C CNN
 F 2 "" H 11450 11000 50  0001 C CNN
 F 3 "" H 11450 11000 50  0001 C CNN
@@
 $EndComp
 $Comp
-L power:GNDA #PWR0124
-U 1 1 5C8C7637
+L power:GNDREF #PWR0124
+U 1 1 5C77F278
 P 11450 12350
 F 0 "#PWR0124" H 11450 12100 50  0001 C CNN
-F 1 "GNDA" H 11455 12177 50  0000 C CNN
+F 1 "GNDREF" H 11455 12177 50  0000 C CNN
 F 2 "" H 11450 12350 50  0001 C CNN
 F 3 "" H 11450 12350 50  0001 C CNN
@@
 $EndComp
 $Comp
-L power:GNDA #PWR0125
-U 1 1 5C8C7939
+L power:GNDREF #PWR0125
+U 1 1 5C77F796
 P 11450 13800
 F 0 "#PWR0125" H 11450 13550 50  0001 C CNN
-F 1 "GNDA" H 11455 13627 50  0000 C CNN
+F 1 "GNDREF" H 11455 13627 50  0000 C CNN
 F 2 "" H 11450 13800 50  0001 C CNN
 F 3 "" H 11450 13800 50  0001 C CNN
@@
 	1    0    0    -1
 $EndComp
-Wire Wire Line
-	11450 10900 11450 11000
 $EndSCHEMATC
