File: Slave/PCB/ltc6813.sch (KiCad schematic (older format))
At the start: 19 parts, among them Q7 DZT5551, U5 LTC6813

Commit message: Slave PCB placement update
Changed lines of the file:
@@
 $Descr A2 23386 16535
 encoding utf-8
-Sheet 10 21
+Sheet 3 21
 Title "BMS-Slave"
 Date ""
@@
 	2900 5850 2900 12050
 Wire Wire Line
-	2900 12050 4350 12050
+	2900 12050 4300 12050
 Wire Wire Line
 	4350 12600 4300 12600
@@
 	1    0    0    -1
 $EndComp
+Wire Wire Line
+	4350 11700 4300 11700
+Wire Wire Line
+	4300 11700 4300 12050
+Connection ~ 4300 12050
+Wire Wire Line
+	4300 12050 4350 12050
 $EndSCHEMATC
