File: Master/PCB/_saved_BMS-Master.sch (KiCad schematic (older format))
At the start: 30 parts, among them J1 BAT, J10 Charge, J11 CAN, J12 USB, J13 Discharge, J14 Corner, J15 Corner, J18 OLED, J19 Master, J2 Charge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

Commit message: Master major PCB change
Connections:
- net GNDA: now also J2.2 (Pin_2); no longer J2.1 (Pin_1)
- net PowerMonitor/Charge+: now also J2.1 (Pin_1); no longer J2.2 (Pin_2)
Changed lines of the file:
@@
-$EndComp
-$Comp
-L Connector_Generic:Conn_01x02 J2
-U 1 1 5C3822E8
-P 14400 1050
-F 0 "J2" H 14480 1042 50  0000 L CNN
-F 1 "Charge" H 14480 951 50  0000 L CNN
-F 2 "TerminalBlock_RND:TerminalBlock_RND_205-00001_Pitch5.00mm" H 14400 1050 50  0001 C CNN
-F 3 "~" H 14400 1050 50  0001 C CNN
-	1    14400 1050
-	1    0    0    1
 $EndComp
 $Comp
@@
 	1    0    0    -1
 $EndComp
+$Comp
+L Connector_Generic:Conn_01x02 J2
+U 1 1 5C3822E8
+P 14400 950
+F 0 "J2" H 14480 942 50  0000 L CNN
+F 1 "Charge" H 14480 851 50  0000 L CNN
+F 2 "TerminalBlock_RND:TerminalBlock_RND_205-00001_Pitch5.00mm" H 14400 950 50  0001 C CNN
+F 3 "~" H 14400 950 50  0001 C CNN
+	1    14400 950
+	1    0    0    -1
+$EndComp
