File: Master/PCB/MCU.sch (KiCad schematic (older format))
At the start: 24 parts, among them J16 J, J17 SWD, Q27 BSS138, U17 STM32F303CCTx, U2 LTC6820, Y1 8MHz

Commit message: components placed on PCB
Parts:
- J16: value J -> SD
- J17: value SWD -> DEBUG
Changed lines of the file:
@@
 $Descr A1 33110 23386
 encoding utf-8
-Sheet 9 8
+Sheet 8 8
 Title ""
 Date ""
@@
 P 27400 11350
 F 0 "J17" H 27480 11392 50  0000 L CNN
-F 1 "SWD" H 27480 11301 50  0000 L CNN
+F 1 "DEBUG" H 27480 11301 50  0000 L CNN
 F 2 "Connectors_Molex:Molex_PicoBlade_53261-0571_05x1.25mm_Angled" H 27400 11350 50  0001 C CNN
 F 3 "~" H 27400 11350 50  0001 C CNN
@@
 P 4800 11400
 F 0 "J16" H 4750 12217 50  0000 C CNN
-F 1 "J" H 4750 12126 50  0000 C CNN
+F 1 "SD" H 4750 12126 50  0000 C CNN
 F 2 "Connectors_Card:Hirose_DM3AT-SF-PEJM5" H 6850 12100 50  0001 C CNN
 F 3 "" H 4800 11500 50  0001 C CNN

Commit message: PCB update
Parts:
- C76, C78: footprint Resistors_SMD:R_0603_HandSoldering -> Capacitors_SMD:C_0603_HandSoldering
Changed lines of the file:
@@
 F 0 "C76" H 6115 9446 50  0000 L CNN
 F 1 "18p" H 6115 9355 50  0000 L CNN
-F 2 "Resistors_SMD:R_0603_HandSoldering" H 6038 9250 50  0001 C CNN
+F 2 "Capacitors_SMD:C_0603_HandSoldering" H 6038 9250 50  0001 C CNN
 F 3 "~" H 6000 9400 50  0001 C CNN
 F 4 "50V" H 6000 9400 50  0001 C CNN "Voltage"
@@
 F 0 "C78" H 7165 8396 50  0000 L CNN
 F 1 "100n" H 7165 8305 50  0000 L CNN
-F 2 "Resistors_SMD:R_0603_HandSoldering" H 7088 8200 50  0001 C CNN
+F 2 "Capacitors_SMD:C_0603_HandSoldering" H 7088 8200 50  0001 C CNN
 F 3 "~" H 7050 8350 50  0001 C CNN
 	1    7050 8350

Commit message: PCB update master final
Parts:
- removed JP3: Jumper_NC_Dual, Pin_Headers:Pin_Header_Straight_1x03_Pitch2.54mm, symbol Device:Jumper_NC_Dual
Connections:
- net +3V3: now also U2.1 (EN)
Changed lines of the file:
@@
 	15500 3350 15500 3650
-Wire Wire Line
-	15500 3350 15800 3350
 Wire Wire Line
 	17250 3650 17250 3500
@@
 	18350 3200 17950 3200
 Connection ~ 17250 3200
-$Comp
-L Device:Jumper_NC_Dual JP?
-U 1 1 5C68B684
-P 15800 3600
-AR Path="/5B4A196B/5C68B684" Ref="JP?"  Part="1"
-AR Path="/5AB72D4D/5C68B684" Ref="JP3"  Part="1"
-F 0 "JP3" V 15800 3701 50  0000 L CNN
-F 1 "Jumper_NC_Dual" V 15845 3702 50  0001 L CNN
-F 2 "Pin_Headers:Pin_Header_Straight_1x03_Pitch2.54mm" H 15800 3600 50  0001 C CNN
-F 3 "~" H 15800 3600 50  0001 C CNN
-	1    15800 3600
-	0    -1   1    0
-$EndComp
-Connection ~ 15800 3350
-Wire Wire Line
-	15800 3350 16050 3350
-Wire Wire Line
-	15800 3850 15800 3900
 Wire Wire Line
 	15800 3900 16050 3900
 Connection ~ 16050 3900
-Wire Wire Line
-	15900 3600 16000 3600
 Wire Wire Line
 	16000 3600 16000 3500
@@
 Text Label 24450 10100 0    50   ~ 0
 SS
+Wire Wire Line
+	15500 3350 16050 3350
+Wire Wire Line
+	15800 3600 15800 3900
+Wire Wire Line
+	15800 3600 16000 3600
 $EndSCHEMATC

Commit message: Mistake correction in master with LTC6820
Parts:
- added C? (x2): 10n, Capacitors_SMD:C_0603_HandSoldering, symbol Device:C
- added R? (x2): 51, Resistors_SMD:R_0603_HandSoldering, symbol Device:R
- added TR?: HM2108NL, ENNOID:HM2108NL, symbol ENNOID:HM2108NL
Connections:
- net GND: now also C?.1, C?.2
- net MA: now also TR?.4; no longer U2.11 (IP)
- net PA: now also TR?.6; no longer U2.10 (IM)
- new net: C?.2, R?.1, R?.2
- new net: R?.2, TR?.3, U2.11 (IP)
- new net: R?.1, TR?.1, U2.10 (IM)
- new net: C?.1, TR?.2
- no-connect marks 4 -> 5
Changed lines of the file:
@@
 AR Path="/5B4A196B/5C68B63A" Ref="R?"  Part="1"
 AR Path="/5AB72D4D/5C68B63A" Ref="R36"  Part="1"
-F 0 "R36" V 15443 2900 50  0000 C CNN
+F 0 "R36" V 15750 2900 50  0000 C CNN
 F 1 "1k" V 15534 2900 50  0000 C CNN
 F 2 "Resistors_SMD:R_0603_HandSoldering" V 15580 2900 50  0001 C CNN
@@
 AR Path="/5B4A196B/5C68B640" Ref="R?"  Part="1"
 AR Path="/5AB72D4D/5C68B640" Ref="R5"  Part="1"
-F 0 "R5" V 14893 2900 50  0000 C CNN
+F 0 "R5" V 15200 2900 50  0000 C CNN
 F 1 "1k" V 14984 2900 50  0000 C CNN
 F 2 "Resistors_SMD:R_0603_HandSoldering" V 15030 2900 50  0001 C CNN
@@
 Wire Wire Line
 	15400 2900 15500 2900
-Wire Wire Line
-	14450 2600 15950 2600
-Wire Wire Line
-	15950 2600 15950 2750
-Wire Wire Line
-	15950 2750 16050 2750
-Wire Wire Line
-	16050 2600 16050 2450
-Wire Wire Line
-	14000 2450 16050 2450
 Wire Wire Line
 	16050 3650 16050 3900
@@
 Wire Wire Line
 	17950 3200 17250 3200
-Text HLabel 14000 2450 0    50   Input ~ 0
+Text HLabel 12550 2350 0    50   Input ~ 0
 MA
-Text HLabel 14450 2600 0    50   Input ~ 0
+Text HLabel 12550 2750 0    50   Input ~ 0
 PA
 Text Label 17650 3050 0    50   ~ 0
@@
 Wire Wire Line
 	15800 3600 16000 3600
+Wire Wire Line
+	12550 2350 12800 2350
+Wire Wire Line
+	12550 2750 12800 2750
+NoConn ~ 12800 2550
+$Comp
+L ENNOID:HM2108NL TR?
+U 1 1 5C441D43
+P 13400 2500
+F 0 "TR?" H 13200 2875 50  0000 C CNN
+F 1 "HM2108NL" H 13200 2784 50  0000 C CNN
+F 2 "ENNOID:HM2108NL" H 13450 2400 50  0001 C CNN
+F 3 "" H 13450 2400 50  0001 C CNN
+	1    13400 2500
+	1    0    0    -1
+$EndComp
+Wire Wire Line
+	13600 2750 15350 2750
+Wire Wire Line
+	16050 2050 15350 2050
+Wire Wire Line
+	13600 2050 13600 2350
+Wire Wire Line
+	16050 2050 16050 2600
+$Comp
+L Device:R R?
+U 1 1 5C424C06
+P 15350 2200
+AR Path="/5B4A196B/5C424C06" Ref="R?"  Part="1"
+AR Path="/5AB72D4D/5C424C06" Ref="R?"  Part="1"
+F 0 "R?" V 15450 2200 50  0000 C CNN
+F 1 "51" V 15234 2200 50  0000 C CNN
+F 2 "Resistors_SMD:R_0603_HandSoldering" V 15280 2200 50  0001 C CNN
+F 3 "~" H 15350 2200 50  0001 C CNN
+	1    15350 2200
+	-1   0    0    1
+$EndComp
+Connection ~ 15350 2050
+Wire Wire Line
+	15350 2050 13600 2050
+$Comp
+L Device:R R?
+U 1 1 5C4254A7
+P 15350 2600
+AR Path="/5B4A196B/5C4254A7" Ref="R?"  Part="1"
+AR Path="/5AB72D4D/5C4254A7" Ref="R?"  Part="1"
+F 0 "R?" V 15450 2600 50  0000 C CNN
+F 1 "51" V 15234 2600 50  0000 C CNN
+F 2 "Resistors_SMD:R_0603_HandSoldering" V 15280 2600 50  0001 C CNN
+F 3 "~" H 15350 2600 50  0001 C CNN
+	1    15350 2600
+	-1   0    0    1
+$EndComp
+Connection ~ 15350 2750
+Wire Wire Line
+	15350 2750 16050 2750
+$Comp
+L Device:C C?
+U 1 1 5C4257C3
+P 14850 2400
+AR Path="/5B4A196B/5C4257C3" Ref="C?"  Part="1"
+AR Path="/5AB72D4D/5C4257C3" Ref="C?"  Part="1"
+F 0 "C?" H 14735 2354 50  0000 R CNN
+F 1 "10n" H 14735 2445 50  0000 R CNN
+F 2 "Capacitors_SMD:C_0603_HandSoldering" H 14888 2250 50  0001 C CNN
+F 3 "~" H 14850 2400 50  0001 C CNN
+	1    14850 2400
+	0    -1   -1   0
+$EndComp
+$Comp
+L Device:C C?
+U 1 1 5C43CC1D
+P 14300 2400
+AR Path="/5B4A196B/5C43CC1D" Ref="C?"  Part="1"
+AR Path="/5AB72D4D/5C43CC1D" Ref="C?"  Part="1"
+F 0 "C?" H 14185 2354 50  0000 R CNN
+F 1 "10n" H 14185 2445 50  0000 R CNN
+F 2 "Capacitors_SMD:C_0603_HandSoldering" H 14338 2250 50  0001 C CNN
+F 3 "~" H 14300 2400 50  0001 C CNN
+	1    14300 2400
+	0    -1   -1   0
+$EndComp
+Wire Wire Line
+	15000 2400 15350 2400
+Wire Wire Line
+	15350 2400 15350 2350
+Wire Wire Line
+	15350 2400 15350 2450
+Connection ~ 15350 2400
+Wire Wire Line
+	14700 2400 14550 2400
+Wire Wire Line
+	14150 2400 13950 2400
+Wire Wire Line
+	13950 2400 13950 2550
+Wire Wire Line
+	13950 2550 13600 2550
+$Comp
+L power:GND #PWR?
+U 1 1 5C45D37F
+P 14550 2400
+AR Path="/5B4A196B/5C45D37F" Ref="#PWR?"  Part="1"
+AR Path="/5AB72D4D/5C45D37F" Ref="#PWR?"  Part="1"
+F 0 "#PWR?" H 14550 2150 50  0001 C CNN
+F 1 "GND" H 14555 2227 50  0000 C CNN
+F 2 "" H 14550 2400 50  0001 C CNN
+F 3 "" H 14550 2400 50  0001 C CNN
+	1    14550 2400
+	1    0    0    -1
+$EndComp
+Connection ~ 14550 2400
+Wire Wire Line
+	14550 2400 14450 2400
 $EndSCHEMATC

Commit message: Master major PCB change
Parts:
- gave numbers to parts that had none: 5
Changed lines of the file:
@@
 NoConn ~ 12800 2550
 $Comp
-L ENNOID:HM2108NL TR?
+L ENNOID:HM2108NL TR2
 U 1 1 5C441D43
 P 13400 2500
-F 0 "TR?" H 13200 2875 50  0000 C CNN
+F 0 "TR2" H 13200 2875 50  0000 C CNN
 F 1 "HM2108NL" H 13200 2784 50  0000 C CNN
 F 2 "ENNOID:HM2108NL" H 13450 2400 50  0001 C CNN
@@
 P 15350 2200
 AR Path="/5B4A196B/5C424C06" Ref="R?"  Part="1"
-AR Path="/5AB72D4D/5C424C06" Ref="R?"  Part="1"
-F 0 "R?" V 15450 2200 50  0000 C CNN
+AR Path="/5AB72D4D/5C424C06" Ref="R6"  Part="1"
+F 0 "R6" V 15450 2200 50  0000 C CNN
 F 1 "51" V 15234 2200 50  0000 C CNN
 F 2 "Resistors_SMD:R_0603_HandSoldering" V 15280 2200 50  0001 C CNN
@@
 P 15350 2600
 AR Path="/5B4A196B/5C4254A7" Ref="R?"  Part="1"
-AR Path="/5AB72D4D/5C4254A7" Ref="R?"  Part="1"
-F 0 "R?" V 15450 2600 50  0000 C CNN
+AR Path="/5AB72D4D/5C4254A7" Ref="R7"  Part="1"
+F 0 "R7" V 15450 2600 50  0000 C CNN
 F 1 "51" V 15234 2600 50  0000 C CNN
 F 2 "Resistors_SMD:R_0603_HandSoldering" V 15280 2600 50  0001 C CNN
@@
 P 14850 2400
 AR Path="/5B4A196B/5C4257C3" Ref="C?"  Part="1"
-AR Path="/5AB72D4D/5C4257C3" Ref="C?"  Part="1"
-F 0 "C?" H 14735 2354 50  0000 R CNN
+AR Path="/5AB72D4D/5C4257C3" Ref="C7"  Part="1"
+F 0 "C7" H 14735 2354 50  0000 R CNN
 F 1 "10n" H 14735 2445 50  0000 R CNN
 F 2 "Capacitors_SMD:C_0603_HandSoldering" H 14888 2250 50  0001 C CNN
@@
 P 14300 2400
 AR Path="/5B4A196B/5C43CC1D" Ref="C?"  Part="1"
-AR Path="/5AB72D4D/5C43CC1D" Ref="C?"  Part="1"
-F 0 "C?" H 14185 2354 50  0000 R CNN
+AR Path="/5AB72D4D/5C43CC1D" Ref="C6"  Part="1"
+F 0 "C6" H 14185 2354 50  0000 R CNN
 F 1 "10n" H 14185 2445 50  0000 R CNN
 F 2 "Capacitors_SMD:C_0603_HandSoldering" H 14338 2250 50  0001 C CNN
@@
 P 14550 2400
 AR Path="/5B4A196B/5C45D37F" Ref="#PWR?"  Part="1"
-AR Path="/5AB72D4D/5C45D37F" Ref="#PWR?"  Part="1"
-F 0 "#PWR?" H 14550 2150 50  0001 C CNN
+AR Path="/5AB72D4D/5C45D37F" Ref="#PWR0130"  Part="1"
+F 0 "#PWR0130" H 14550 2150 50  0001 C CNN
 F 1 "GND" H 14555 2227 50  0000 C CNN
 F 2 "" H 14550 2400 50  0001 C CNN

Commit message: PCB master update
Connections:
- net MA: now also TR2.6; no longer TR2.4
- net PA: now also TR2.4; no longer TR2.6
- net at R6.2, U2.11 (IP): now also TR2.1; no longer TR2.3
- net at R7.1, U2.10 (IM): now also TR2.3; no longer TR2.1
Changed lines of the file:
@@
 Wire Wire Line
 	17950 3200 17250 3200
-Text HLabel 12550 2350 0    50   Input ~ 0
-MA
-Text HLabel 12550 2750 0    50   Input ~ 0
-PA
 Text Label 17650 3050 0    50   ~ 0
 SS
@@
 L ENNOID:HM2108NL TR2
 U 1 1 5C441D43
-P 13400 2500
-F 0 "TR2" H 13200 2875 50  0000 C CNN
-F 1 "HM2108NL" H 13200 2784 50  0000 C CNN
-F 2 "ENNOID:HM2108NL" H 13450 2400 50  0001 C CNN
-F 3 "" H 13450 2400 50  0001 C CNN
-	1    13400 2500
-	1    0    0    -1
+P 13400 2600
+F 0 "TR2" H 13200 2975 50  0000 C CNN
+F 1 "HM2108NL" H 13200 2884 50  0000 C CNN
+F 2 "ENNOID:HM2108NL" H 13450 2500 50  0001 C CNN
+F 3 "" H 13450 2500 50  0001 C CNN
+	1    13400 2600
+	1    0    0    1
 $EndComp
 Wire Wire Line
@@
 	16050 2050 15350 2050
 Wire Wire Line
-	13600 2050 13600 2350
+	13600 2050 13600 2250
 Wire Wire Line
 	16050 2050 16050 2600
@@
 Wire Wire Line
 	14550 2400 14450 2400
+Text HLabel 12550 2750 0    50   Input ~ 0
+PA
+Text HLabel 12550 2350 0    50   Input ~ 0
+MA
+Connection ~ 13600 2250
+Wire Wire Line
+	13600 2250 13600 2350
 $EndSCHEMATC

Commit message: small corections
Changed lines of the file:
@@
 	16050 2050 15350 2050
-Wire Wire Line
-	13600 2050 13600 2250
 Wire Wire Line
 	16050 2050 16050 2600
@@
 Text HLabel 12550 2350 0    50   Input ~ 0
 MA
-Connection ~ 13600 2250
 Wire Wire Line
-	13600 2250 13600 2350
+	13600 2050 13600 2350
 $EndSCHEMATC

Commit message: BOM
Parts:
- C79: value C -> 10u
Changed lines of the file:
@@
 P 7050 12250
 F 0 "C79" H 7165 12296 50  0000 L CNN
-F 1 "C" H 7165 12205 50  0000 L CNN
+F 1 "10u" H 7165 12205 50  0000 L CNN
 F 2 "Capacitors_SMD:C_0603_HandSoldering" H 7088 12100 50  0001 C CNN
 F 3 "~" H 7050 12250 50  0001 C CNN
