File: Current_Sensor/current_sensor.kicad_pcb (KiCad board)
At the start: 2 copper layers, 58.5 x 25 mm, 47 parts, among them J2 DS conn, J3 Conn, J4 DS conn, T2 TRANS-2CT, U1 Buffer, U2 OPA376AID, U3 AMC1303, U4 SN74LVC2G17DBVR, U5 SN6501DBV, U7 TPS76350

Commit message: ltc6811 started
Parts:
- removed C2: 10uF, IPC7351-Nominal:CAPC1608X55
- removed C3: 470pF, IPC7351-Nominal:CAPC1608X55
- removed C4: 330pF, IPC7351-Nominal:CAPC1608X55
- removed C5: 150pF, IPC7351-Nominal:CAPC1608X55
- removed C6, C7: 100nF, IPC7351-Nominal:CAPC1608X55
- removed D1, D2: BAT54S, smd-semi:SOT-23
- removed HOLE1, HOLE2: MOUNTING_HOLE, mech:PTH-3MM-PLUS-SUPPORTED
- removed J2: DS conn, conn-100mil:CONN-100MIL-F-1x4
- removed J3: Conn, paltatech:DF13-3P-1.25H_50
- removed R11, R9: 220R, IPC7351-Nominal:RESC1608X50
- removed R4: 100k, IPC7351-Nominal:RESC1608X50
- removed R6: 910R, IPC7351-Nominal:RESC1608X50
- removed R7: 6.8k, IPC7351-Nominal:RESC1608X50
- removed R8: 5.1k, IPC7351-Nominal:RESC1608X50
- removed REF** (x2): routing_tab_2mm_slot, routing_tab_2mm_slot
- removed U2: OPA376AID, IPC7351-Nominal:SOIC127P600X175-8
- removed U4: SN74LVC2G17DBVR, smd-semi:SOT-23-6
Connections:
- J4 pad : GND -> (no net)
- U7 pad 4: Net-(U7-Pad4) -> (no net)
Routing:
- net +5: track 92.2 -> 36.0 mm, vias 1 -> 0
- net GND: track 99.5 -> 44.8 mm, vias 36 -> 25
- net Net-(R6-Pad2): track 23.7 -> 0.00 mm
- net Net-(D1-Pad3): track 23.7 -> 0.00 mm, vias 2 -> 0
- net Net-(C4-Pad1): track 18.5 -> 0.00 mm, vias 2 -> 0
- net /delta_sigma: track 21.6 -> 7.65 mm
- net Net-(C5-Pad1): track 5.91 -> 0.00 mm
- net Net-(C3-Pad1): track 5.41 -> 0.00 mm
- net /analog filter/OUT: track 3.15 -> 0.00 mm
- net Net-(C4-Pad2): track 3.00 -> 0.00 mm
Other:
- board size 58.5 x 25 mm -> 39 x 25 mm
- board text removed: "-o+"
