File: Slaves/LTC6813/PCB/Temperature.sch (KiCad schematic (older format))
At the start: 18 parts

Commit message: description on PCB
Parts:
- renumbered R6 to R1, R7 to R2, R8 to R3, R9 to R4, R10 to R5, R11 to R6, R12 to R7, R13 to R8, R14 to R9
Changed lines of the file:
@@
 $EndDescr
 $Comp
-L BMS-Slave-rescue:R-Device-BMS-Slave-rescue R7
+L BMS-Slave-rescue:R-Device-BMS-Slave-rescue R2
 U 1 1 5AEA9568
 P 11450 3150
-F 0 "R7" H 11520 3196 50  0000 L CNN
+F 0 "R2" H 11520 3196 50  0000 L CNN
 F 1 "10k" H 11520 3105 50  0000 L CNN
 F 2 "Resistors_SMD:R_0603_HandSoldering" V 11380 3150 50  0001 C CNN
@@
 	11450 3850 11450 3950
 $Comp
-L BMS-Slave-rescue:R-Device-BMS-Slave-rescue R8
+L BMS-Slave-rescue:R-Device-BMS-Slave-rescue R3
 U 1 1 5AEAA2B3
 P 11450 4600
-F 0 "R8" H 11520 4646 50  0000 L CNN
+F 0 "R3" H 11520 4646 50  0000 L CNN
 F 1 "10k" H 11520 4555 50  0000 L CNN
 F 2 "Resistors_SMD:R_0603_HandSoldering" V 11380 4600 50  0001 C CNN
@@
 	11450 5300 11450 5400
 $Comp
-L BMS-Slave-rescue:R-Device-BMS-Slave-rescue R9
+L BMS-Slave-rescue:R-Device-BMS-Slave-rescue R4
 U 1 1 5AEAA88D
 P 11450 5950
-F 0 "R9" H 11520 5996 50  0000 L CNN
+F 0 "R4" H 11520 5996 50  0000 L CNN
 F 1 "10k" H 11520 5905 50  0000 L CNN
 F 2 "Resistors_SMD:R_0603_HandSoldering" V 11380 5950 50  0001 C CNN
@@
 	11450 6650 11450 6750
 $Comp
-L BMS-Slave-rescue:R-Device-BMS-Slave-rescue R10
+L BMS-Slave-rescue:R-Device-BMS-Slave-rescue R5
 U 1 1 5AEAA8B0
 P 11450 7400
-F 0 "R10" H 11520 7446 50  0000 L CNN
+F 0 "R5" H 11520 7446 50  0000 L CNN
 F 1 "10k" H 11520 7355 50  0000 L CNN
 F 2 "Resistors_SMD:R_0603_HandSoldering" V 11380 7400 50  0001 C CNN
@@
 	11450 8100 11450 8200
 $Comp
-L BMS-Slave-rescue:R-Device-BMS-Slave-rescue R11
+L BMS-Slave-rescue:R-Device-BMS-Slave-rescue R6
 U 1 1 5AEAB9E1
 P 11450 8750
-F 0 "R11" H 11520 8796 50  0000 L CNN
+F 0 "R6" H 11520 8796 50  0000 L CNN
 F 1 "10k" H 11520 8705 50  0000 L CNN
 F 2 "Resistors_SMD:R_0603_HandSoldering" V 11380 8750 50  0001 C CNN
@@
 	11450 9450 11450 9550
 $Comp
-L BMS-Slave-rescue:R-Device-BMS-Slave-rescue R12
+L BMS-Slave-rescue:R-Device-BMS-Slave-rescue R7
 U 1 1 5AEABA04
 P 11450 10200
-F 0 "R12" H 11520 10246 50  0000 L CNN
+F 0 "R7" H 11520 10246 50  0000 L CNN
 F 1 "10k" H 11520 10155 50  0000 L CNN
 F 2 "Resistors_SMD:R_0603_HandSoldering" V 11380 10200 50  0001 C CNN
@@
 VP1
 $Comp
-L BMS-Slave-rescue:R-Device-BMS-Slave-rescue R13
+L BMS-Slave-rescue:R-Device-BMS-Slave-rescue R8
 U 1 1 5AEABA27
 P 11450 11550
-F 0 "R13" H 11520 11596 50  0000 L CNN
+F 0 "R8" H 11520 11596 50  0000 L CNN
 F 1 "10k" H 11520 11505 50  0000 L CNN
 F 2 "Resistors_SMD:R_0603_HandSoldering" V 11380 11550 50  0001 C CNN
@@
 	11450 12250 11450 12350
 $Comp
-L BMS-Slave-rescue:R-Device-BMS-Slave-rescue R14
+L BMS-Slave-rescue:R-Device-BMS-Slave-rescue R9
 U 1 1 5AEABA4A
 P 11450 13000
-F 0 "R14" H 11520 13046 50  0000 L CNN
+F 0 "R9" H 11520 13046 50  0000 L CNN
 F 1 "10k" H 11520 12955 50  0000 L CNN
 F 2 "Resistors_SMD:R_0603_HandSoldering" V 11380 13000 50  0001 C CNN
@@
 	9550 9450 8800 9450
 $Comp
-L BMS-Slave-rescue:R-Device-BMS-Slave-rescue R6
+L BMS-Slave-rescue:R-Device-BMS-Slave-rescue R1
 U 1 1 5BF1E9E7
 P 11450 1750
-F 0 "R6" H 11520 1796 50  0000 L CNN
+F 0 "R1" H 11520 1796 50  0000 L CNN
 F 1 "10k" H 11520 1705 50  0000 L CNN
 F 2 "Resistors_SMD:R_0603_HandSoldering" V 11380 1750 50  0001 C CNN
@@
 	11450 10900 11450 11000
 $Comp
-L power:GNDREF #PWR0117
+L power:GNDREF #PWR02
 U 1 1 5C77BBEC
 P 11450 2550
-F 0 "#PWR0117" H 11450 2300 50  0001 C CNN
+F 0 "#PWR02" H 11450 2300 50  0001 C CNN
 F 1 "GNDREF" H 11455 2377 50  0000 C CNN
 F 2 "" H 11450 2550 50  0001 C CNN
@@
 $EndComp
 $Comp
-L power:GNDREF #PWR0118
+L power:GNDREF #PWR03
 U 1 1 5C77C4DE
 P 11450 3950
-F 0 "#PWR0118" H 11450 3700 50  0001 C CNN
+F 0 "#PWR03" H 11450 3700 50  0001 C CNN
 F 1 "GNDREF" H 11455 3777 50  0000 C CNN
 F 2 "" H 11450 3950 50  0001 C CNN
@@
 $EndComp
 $Comp
-L power:GNDREF #PWR0119
+L power:GNDREF #PWR04
 U 1 1 5C77CE41
 P 11450 5400
-F 0 "#PWR0119" H 11450 5150 50  0001 C CNN
+F 0 "#PWR04" H 11450 5150 50  0001 C CNN
 F 1 "GNDREF" H 11455 5227 50  0000 C CNN
 F 2 "" H 11450 5400 50  0001 C CNN
@@
 $EndComp
 $Comp
-L power:GNDREF #PWR0120
+L power:GNDREF #PWR05
 U 1 1 5C77D999
 P 11450 6750
-F 0 "#PWR0120" H 11450 6500 50  0001 C CNN
+F 0 "#PWR05" H 11450 6500 50  0001 C CNN
 F 1 "GNDREF" H 11455 6577 50  0000 C CNN
 F 2 "" H 11450 6750 50  0001 C CNN
@@
 $EndComp
 $Comp
-L power:GNDREF #PWR0121
+L power:GNDREF #PWR06
 U 1 1 5C77E07A
 P 11450 8200
-F 0 "#PWR0121" H 11450 7950 50  0001 C CNN
+F 0 "#PWR06" H 11450 7950 50  0001 C CNN
 F 1 "GNDREF" H 11455 8027 50  0000 C CNN
 F 2 "" H 11450 8200 50  0001 C CNN
@@
 $EndComp
 $Comp
-L power:GNDREF #PWR0122
+L power:GNDREF #PWR07
 U 1 1 5C77E6D8
 P 11450 9550
-F 0 "#PWR0122" H 11450 9300 50  0001 C CNN
+F 0 "#PWR07" H 11450 9300 50  0001 C CNN
 F 1 "GNDREF" H 11455 9377 50  0000 C CNN
 F 2 "" H 11450 9550 50  0001 C CNN
@@
 $EndComp
 $Comp
-L power:GNDREF #PWR0123
+L power:GNDREF #PWR08
 U 1 1 5C77EC81
 P 11450 11000
-F 0 "#PWR0123" H 11450 10750 50  0001 C CNN
+F 0 "#PWR08" H 11450 10750 50  0001 C CNN
 F 1 "GNDREF" H 11455 10827 50  0000 C CNN
 F 2 "" H 11450 11000 50  0001 C CNN
@@
 $EndComp
 $Comp
-L power:GNDREF #PWR0124
+L power:GNDREF #PWR09
 U 1 1 5C77F278
 P 11450 12350
-F 0 "#PWR0124" H 11450 12100 50  0001 C CNN
+F 0 "#PWR09" H 11450 12100 50  0001 C CNN
 F 1 "GNDREF" H 11455 12177 50  0000 C CNN
 F 2 "" H 11450 12350 50  0001 C CNN
@@
 $EndComp
 $Comp
-L power:GNDREF #PWR0125
+L power:GNDREF #PWR010
 U 1 1 5C77F796
 P 11450 13800
-F 0 "#PWR0125" H 11450 13550 50  0001 C CNN
+F 0 "#PWR010" H 11450 13550 50  0001 C CNN
 F 1 "GNDREF" H 11455 13627 50  0000 C CNN
 F 2 "" H 11450 13800 50  0001 C CNN
