File: UPS/PCB/UPS.kicad_pcb (KiCad board)
At the start: 2 copper layers, 100 x 100 mm, 14 parts, among them J1 BAT, J2 ExtPower, J3 Conn_01x01, J4 Conn_01x01, J5 Conn_01x01, J6 Conn_01x01, U1 EPM2405SJ

Commit message: UPS update
Parts:
- added C10: 0.1u, Capacitors_SMD:C_0603_HandSoldering, F.Cu at (17.2, -13.9)
- added C11: 0.1u, Capacitors_SMD:C_0603_HandSoldering, F.Cu at (22.4, -19.0)
- added C4: 0.1u, Capacitors_SMD:C_0603_HandSoldering, F.Cu at (22.4, -21.3)
- added C5: 1u, Capacitors_SMD:C_0603_HandSoldering, F.Cu at (17.9, -9.18)
- added C6: 0.1u, Capacitors_SMD:C_0603_HandSoldering, F.Cu at (17.9, -11.5)
- added C7: 1u, Capacitors_SMD:C_0603_HandSoldering, F.Cu at (21.8, -13.9)
- added C8: 0.1u, Capacitors_SMD:C_0603_HandSoldering, F.Cu at (22.2, -16.4)
- added C9: 0.1u, Capacitors_SMD:C_0603_HandSoldering, F.Cu at (13.2, -9.63)
- added F1: Fuse, Fuse_Holders_and_Fuses:Fuseholder5x20_horiz_open_universal_Type-III, F.Cu at (32.0, 5.50)
- added R1: 1k, Resistors_SMD:R_0603_HandSoldering, F.Cu at (7.44, -17.0)
- added R10: 5.1k, Resistors_SMD:R_0603_HandSoldering, F.Cu at (7.44, -12.0)
- added R11: 5.1k, Resistors_SMD:R_0603_HandSoldering, F.Cu at (12.4, -12.0)
- added R12: 3M, Resistors_SMD:R_0603_HandSoldering, F.Cu at (8.41, -9.57)
- added R13: 470k, Resistors_SMD:R_0603_HandSoldering, F.Cu at (17.4, -16.3)
- added R2: 1k, Resistors_SMD:R_0603_HandSoldering, F.Cu at (17.6, -21.3)
- added R3: 1k, Resistors_SMD:R_0603_HandSoldering, F.Cu at (12.4, -17.0)
- added R4: 1k, Resistors_SMD:R_0603_HandSoldering, F.Cu at (7.44, -14.5)
- added R5: 100, Resistors_SMD:R_0603_HandSoldering, F.Cu at (-1.51, -9.03)
- added R6: 100, Resistors_SMD:R_0603_HandSoldering, F.Cu at (3.45, -9.03)
- added R7: 0.01, Resistors_SMD:R_2010_HandSoldering, F.Cu at (1.13, -20.5)
- added R8: 10k, Resistors_SMD:R_0603_HandSoldering, F.Cu at (17.6, -18.8)
- added R9: 1M, Resistors_SMD:R_0603_HandSoldering, F.Cu at (12.4, -14.5)
- added TH1: Thermistor 10k, Resistors_THT:R_Axial_DIN0207_L6.3mm_D2.5mm_P5.08mm_Vertical, F.Cu at (8.38, -20.4)
- added U2: BQ77904, Housings_SSOP:TSSOP-20_4.4x6.5mm_Pitch0.65mm, F.Cu at (0.48, -14.3)
- J2: moved to B.Cu
- moved C1 4.50 mm to (24.5, 16.5)
- moved J2 4.14 mm to (89.4, 5.90)
- moved U1 2.55 mm to (52.0, 16.0)
Connections:
- BT3 pad 2: GND -> GNDREF
- J1 pad 2: Net-(C1-Pad1) -> Net-(F1-Pad2)
Routing:
- net GNDREF: track 0.00 -> 54.4 mm, vias 0 -> 100
- net Net-(C1-Pad2): track 52.5 -> 0.00 mm
- net GND: track 115.1 -> 64.1 mm, vias 181 -> 80
- net Net-(C1-Pad1): track 42.5 -> 0.00 mm
- net Net-(C2-Pad1): track 51.7 -> 10.8 mm
- net +12V: track 100.6 -> 101.8 mm

Commit message: UPS completed
Parts:
- added Q1: CSD18534Q5A, TO_SOT_Packages_SMD:TDSON-8-1, B.Cu at (38.4, 68.2)
- added Q2: CSD18534Q5A, TO_SOT_Packages_SMD:TDSON-8-1, B.Cu at (27.4, 68.2)
- C10, C11, C4, C5, C6, C7, C8, C9, R1, R10, R11, R12, R13, R2, R3, R4, R5, R6, R7, R8, R9, TH1, U2: moved to B.Cu
- moved R7 104.7 mm to (61.4, 65.2)
- moved R5 96.3 mm to (64.4, 61.2), turned to 270 degrees
- moved R4 94.5 mm to (72.9, 53.7)
- moved R9 93.4 mm to (43.0, 73.7), turned to 180 degrees
- moved R3 89.3 mm to (72.9, 48.7)
- moved R6 89.2 mm to (58.4, 61.2), turned to 270 degrees
- moved C8 88.5 mm to (67.4, 59.7)
- moved R1 85.9 mm to (72.9, 38.7)
- moved C10 85.8 mm to (61.4, 59.7), turned to 180 degrees
- moved C9 85.7 mm to (69.9, 54.7), turned to 270 degrees
- moved R12 85.7 mm to (28.8, 73.7)
- moved R2 85.7 mm to (72.9, 44.2)
- moved U2 85.6 mm to (58.4, 48.7), turned to 180 degrees
- moved C11 85.0 mm to (54.4, 59.7), turned to 180 degrees
- moved R10 82.5 mm to (44.4, 61.7), turned to 90 degrees
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Routing:
- net GND: track 64.1 -> 138.9 mm, vias 80 -> 0
- net Net-(C1-Pad2): track 0.00 -> 59.0 mm
- net Net-(C1-Pad1): track 0.00 -> 52.1 mm
- net Net-(C2-Pad1): track 10.8 -> 53.6 mm
- net Net-(F1-Pad2): track 0.00 -> 31.0 mm
- net Net-(R11-Pad2): track 0.00 -> 30.2 mm
- net Net-(Q1-Pad1): track 0.00 -> 29.9 mm
- net +12V: track 101.8 -> 123.0 mm, vias 0 -> 1
- net Net-(R8-Pad2): track 0.00 -> 19.6 mm
- net Net-(Q1-Pad5): track 0.00 -> 16.8 mm
- net Net-(C10-Pad1): track 0.00 -> 15.4 mm
- net Net-(C5-Pad1): track 0.00 -> 15.2 mm
- net Net-(Q2-Pad4): track 0.00 -> 15.0 mm, vias 0 -> 2
- net Net-(R10-Pad2): track 0.00 -> 14.9 mm
- net Net-(C10-Pad2): track 0.00 -> 14.0 mm
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- added copper zone on B.Cu, net GNDREF
- removed copper zone on B.Cu, net GND
