File: UPS/PCB/UPS.sch (KiCad schematic (older format))
At the start: 17 parts, among them J1 BAT, J2 ExtPower, J3 Conn_01x01, J4 Conn_01x01, J5 Conn_01x01, J6 Conn_01x01, U1 EPM2405SJ

Commit message: UPS update
Parts:
- removed R? (x3): 1M, Resistors_SMD:R_0603_HandSoldering, symbol Device:R
- added C10, C11, C4, C6, C8, C9: 0.1u, Capacitors_SMD:C_0603_HandSoldering, symbol Device:C
- added C5, C7: 1u, Capacitors_SMD:C_0603_HandSoldering, symbol Device:C
- added F1: Fuse, Fuse_Holders_and_Fuses:Fuseholder5x20_horiz_open_universal_Type-III, symbol Device:Fuse
- added Q1, Q2: CSD18534Q5A, Package_TO_SOT_SMD:TDSON-8-1, symbol Transistor_FET:CSD18534Q5A
- added R1, R2, R3, R4: 1k, Resistors_SMD:R_0603_HandSoldering, symbol Device:R
- added R10, R11: 5.1k, Resistors_SMD:R_0603_HandSoldering, symbol Device:R
- added R12: 3M, Resistors_SMD:R_0603_HandSoldering, symbol Device:R
- added R13: 470k, Resistors_SMD:R_0603_HandSoldering, symbol Device:R
- added R5, R6: 100, Resistors_SMD:R_0603_HandSoldering, symbol Device:R
- added R7: 0.01, Resistors_SMD:R_2010_HandSoldering, symbol Device:R
- added R8: 10k, Resistors_SMD:R_0603_HandSoldering, symbol Device:R
- added R9: 1M, Resistors_SMD:R_0603_HandSoldering, symbol Device:R
- added TH1: Thermistor 10k, Resistors_THT:R_Axial_DIN0207_L6.3mm_D2.5mm_P5.08mm_Vertical, symbol Device:Thermistor
- added U2: BQ77904, Housings_SSOP:TSSOP-20_4.4x6.5mm_Pitch0.65mm, symbol ENNOID:BQ77904
Connections:
- net +12V: now also R1.2, R2.2
- net GND: now also Q2.5 (D), R12.1, R13.1; no longer BT3.2 (-)
- net at C1.1, U1.12 (+DC_IN): now also F1.1; no longer J1.2 (Pin_2)
- net at BT1.2 (-), BT2.1 (+): now also R3.2
- net at BT2.2 (-), BT3.1 (+): now also R4.2
- new net: F1.2, J1.2 (Pin_2)
- new net: C5.1, R1.1, U2.1 (VDD)
- new net: C10.2, C11.1, R6.1, U2.10 (SRN)
- new net: R10.2, U2.11 (DSG)
- new net: R11.2, U2.13 (CHG)
- new net: R13.2, U2.14 (LD)
- new net: R8.2, TH1.2, U2.15 (TS)
- new net: R8.1, U2.16 (VTB)
- new net: C7.1, U2.2 (AVDD)
- new net: C4.1, R2.1, U2.3 (VC5), U2.4 (VC4), U2.5 (VC3)
- new net: C6.1, R3.1, U2.6 (VC2)
- new net: C9.1, R4.1, U2.7 (VC1)
- new net: C10.1, C8.1, R5.1, U2.9 (SRP)
- new net: Q1.1 (S), Q1.2 (S), Q1.3 (S), R6.2, R7.1, R9.1
- new net: Q1.4 (G), R10.1, R9.2
- new net: Q1.5 (D), Q2.1 (S), Q2.2 (S), Q2.3 (S)
- new net: Q2.4 (G), R11.1, R12.2
- new net GNDREF: BT3.2 (-), C11.2, C4.2, C5.2, C6.2, C7.2, C8.2, C9.2, R5.2, R7.2, TH1.1, U2.17 (CCFG), U2.18 (CTRC), U2.19 (CTRD), U2.20 (DVSS), U2.8 (AVSS)
Other:
- moved on the sheet: BT1, BT2, BT3

Commit message: UPS completed
Parts:
- Q1, Q2: footprint Package_TO_SOT_SMD:TDSON-8-1 -> TO_SOT_Packages_SMD:TDSON-8-1
Changed lines of the file:
@@
 F 0 "Q1" V 8601 8400 50  0000 C CNN
 F 1 "CSD18534Q5A" V 8692 8400 50  0000 C CNN
-F 2 "Package_TO_SOT_SMD:TDSON-8-1" H 8550 8325 50  0001 L CIN
+F 2 "TO_SOT_Packages_SMD:TDSON-8-1" H 8550 8325 50  0001 L CIN
 F 3 "http://www.ti.com/lit/gpn/csd18534q5a" V 8350 8400 50  0001 L CNN
 	1    8350 8400
@@
 F 0 "Q2" V 9501 8400 50  0000 C CNN
 F 1 "CSD18534Q5A" V 9592 8400 50  0000 C CNN
-F 2 "Package_TO_SOT_SMD:TDSON-8-1" H 9450 8325 50  0001 L CIN
+F 2 "TO_SOT_Packages_SMD:TDSON-8-1" H 9450 8325 50  0001 L CIN
 F 3 "http://www.ti.com/lit/gpn/csd18534q5a" V 9250 8400 50  0001 L CNN
 	1    9250 8400
