File: Current_Sensor/PCB/isolated_current_sensor.sch (KiCad schematic (older format))
At the start: 7 parts, among them U3 AMC1303

Commit message: Software added
Changed lines of the file:
@@
 	5100 3450 5100 3500
 Wire Wire Line
-	4550 3450 5300 3450
+	4550 3450 5100 3450
 Wire Wire Line
 	5100 3750 5100 3700
 Wire Wire Line
-	4550 3750 5300 3750
+	4550 3750 5100 3750
 Wire Wire Line
 	4000 3950 4600 3950
 Wire Wire Line
-	4800 3950 5300 3950
+	4800 3950 5100 3950
 Wire Wire Line
 	5100 3950 5100 4000
 Wire Wire Line
-	4800 4250 5300 4250
+	4800 4250 5100 4250
 Wire Wire Line
 	5100 4250 5100 4200
@@
 	6700 3500 6700 3450
 Wire Wire Line
-	6500 3450 7450 3450
+	6500 3450 6700 3450
 Wire Wire Line
 	6700 3700 6700 3750
 Wire Wire Line
-	6500 3750 7450 3750
+	6500 3750 6700 3750
 Wire Wire Line
 	7150 3750 7150 3700
@@
 	-1   0    0    -1
 $EndComp
+Wire Wire Line
+	5100 3750 5300 3750
+Wire Wire Line
+	5100 3450 5300 3450
+Wire Wire Line
+	5100 3950 5300 3950
+Wire Wire Line
+	5100 4250 5300 4250
+Wire Wire Line
+	6700 3750 7150 3750
+Wire Wire Line
+	6700 3450 7150 3450
+Wire Wire Line
+	7150 3750 7450 3750
+Wire Wire Line
+	7150 3450 7450 3450
 $EndSCHEMATC
