File: Slaves/LTC6811/PCB/LTC6811.sch (KiCad schematic (older format))
At the start: 50 parts, among them J1 Cells, J2 Slave, J3 Master, J4 Temperature, J5 Conn_01x01, J6 Conn_01x01, J7 Conn_01x01, J8 Conn_01x01, Q1 NSV1C201MZ4, U1 LTC6811-1

Commit message: LTC6811 pcb update
Parts:
- F1, F10, F11, F12, F13, F2, F3, F4, F5, F6, F7, F8, F9: footprint Fuse_Holders_and_Fuses:Fuse_SMD1206_HandSoldering -> ENNOID:FUSE
Changed lines of the file:
@@
 F 0 "F1" V 2750 4950 50  0000 C CNN
 F 1 "0.25A" V 2750 4500 50  0000 C CNN
-F 2 "Fuse_Holders_and_Fuses:Fuse_SMD1206_HandSoldering" V 2730 4750 50  0001 C CNN
+F 2 "ENNOID:FUSE" V 2730 4750 50  0001 C CNN
 F 3 "~" H 2800 4750 50  0001 C CNN
 	1    2800 4750
@@
 F 0 "F2" V 2750 5050 50  0000 C CNN
 F 1 "0.25A" V 2750 4600 50  0000 C CNN
-F 2 "Fuse_Holders_and_Fuses:Fuse_SMD1206_HandSoldering" V 2730 4850 50  0001 C CNN
+F 2 "ENNOID:FUSE" V 2730 4850 50  0001 C CNN
 F 3 "~" H 2800 4850 50  0001 C CNN
 	1    2800 4850
@@
 F 0 "F3" V 2750 5150 50  0000 C CNN
 F 1 "0.25A" V 2750 4700 50  0000 C CNN
-F 2 "Fuse_Holders_and_Fuses:Fuse_SMD1206_HandSoldering" V 2730 4950 50  0001 C CNN
+F 2 "ENNOID:FUSE" V 2730 4950 50  0001 C CNN
 F 3 "~" H 2800 4950 50  0001 C CNN
 	1    2800 4950
@@
 F 0 "F4" V 2750 5250 50  0000 C CNN
 F 1 "0.25A" V 2750 4800 50  0000 C CNN
-F 2 "Fuse_Holders_and_Fuses:Fuse_SMD1206_HandSoldering" V 2730 5050 50  0001 C CNN
+F 2 "ENNOID:FUSE" V 2730 5050 50  0001 C CNN
 F 3 "~" H 2800 5050 50  0001 C CNN
 	1    2800 5050
@@
 F 0 "F5" V 2750 5350 50  0000 C CNN
 F 1 "0.25A" V 2750 4900 50  0000 C CNN
-F 2 "Fuse_Holders_and_Fuses:Fuse_SMD1206_HandSoldering" V 2730 5150 50  0001 C CNN
+F 2 "ENNOID:FUSE" V 2730 5150 50  0001 C CNN
 F 3 "~" H 2800 5150 50  0001 C CNN
 	1    2800 5150
@@
 F 0 "F6" V 2750 5450 50  0000 C CNN
 F 1 "0.25A" V 2750 5000 50  0000 C CNN
-F 2 "Fuse_Holders_and_Fuses:Fuse_SMD1206_HandSoldering" V 2730 5250 50  0001 C CNN
+F 2 "ENNOID:FUSE" V 2730 5250 50  0001 C CNN
 F 3 "~" H 2800 5250 50  0001 C CNN
 	1    2800 5250
@@
 F 0 "F7" V 2750 5550 50  0000 C CNN
 F 1 "0.25A" V 2750 5100 50  0000 C CNN
-F 2 "Fuse_Holders_and_Fuses:Fuse_SMD1206_HandSoldering" V 2730 5350 50  0001 C CNN
+F 2 "ENNOID:FUSE" V 2730 5350 50  0001 C CNN
 F 3 "~" H 2800 5350 50  0001 C CNN
 	1    2800 5350
@@
 F 0 "F8" V 2750 5650 50  0000 C CNN
 F 1 "0.25A" V 2750 5200 50  0000 C CNN
-F 2 "Fuse_Holders_and_Fuses:Fuse_SMD1206_HandSoldering" V 2730 5450 50  0001 C CNN
+F 2 "ENNOID:FUSE" V 2730 5450 50  0001 C CNN
 F 3 "~" H 2800 5450 50  0001 C CNN
 	1    2800 5450
@@
 F 0 "F9" V 2750 5750 50  0000 C CNN
 F 1 "0.25A" V 2750 5300 50  0000 C CNN
-F 2 "Fuse_Holders_and_Fuses:Fuse_SMD1206_HandSoldering" V 2730 5550 50  0001 C CNN
+F 2 "ENNOID:FUSE" V 2730 5550 50  0001 C CNN
 F 3 "~" H 2800 5550 50  0001 C CNN
 	1    2800 5550
@@
 F 0 "F10" V 2750 5850 50  0000 C CNN
 F 1 "0.25A" V 2750 5400 50  0000 C CNN
-F 2 "Fuse_Holders_and_Fuses:Fuse_SMD1206_HandSoldering" V 2730 5650 50  0001 C CNN
+F 2 "ENNOID:FUSE" V 2730 5650 50  0001 C CNN
 F 3 "~" H 2800 5650 50  0001 C CNN
 	1    2800 5650
@@
 F 0 "F11" V 2750 5950 50  0000 C CNN
 F 1 "0.25A" V 2750 5500 50  0000 C CNN
-F 2 "Fuse_Holders_and_Fuses:Fuse_SMD1206_HandSoldering" V 2730 5750 50  0001 C CNN
+F 2 "ENNOID:FUSE" V 2730 5750 50  0001 C CNN
 F 3 "~" H 2800 5750 50  0001 C CNN
 	1    2800 5750
@@
 F 0 "F12" V 2750 6050 50  0000 C CNN
 F 1 "0.25A" V 2750 5600 50  0000 C CNN
-F 2 "Fuse_Holders_and_Fuses:Fuse_SMD1206_HandSoldering" V 2730 5850 50  0001 C CNN
+F 2 "ENNOID:FUSE" V 2730 5850 50  0001 C CNN
 F 3 "~" H 2800 5850 50  0001 C CNN
 	1    2800 5850
@@
 F 0 "F13" V 2750 6150 50  0000 C CNN
 F 1 "0.25A" V 2750 5700 50  0000 C CNN
-F 2 "Fuse_Holders_and_Fuses:Fuse_SMD1206_HandSoldering" V 2730 5950 50  0001 C CNN
+F 2 "ENNOID:FUSE" V 2730 5950 50  0001 C CNN
 F 3 "~" H 2800 5950 50  0001 C CNN
 	1    2800 5950

Commit message: Update current sensor connector + LTC6811
Parts:
- added C? (x2): 1u, Capacitors_SMD:C_0805_HandSoldering, symbol Device:C
- added D?: BZT52Bxx, Diode_SMD:D_SOD-123, symbol Diode:BZT52Bxx
- added D? (x2): 1N4148W, Diode_SMD:D_SOD-123, symbol Diode:1N4148W
- added FB?: Ferrite_Bead, Resistor_SMD:R_0603_1608Metric, symbol Device:Ferrite_Bead
- J4: footprint Pin_Headers:Pin_Header_Straight_1x10_Pitch2.54mm -> Pin_Headers:Pin_Header_Angled_1x10_Pitch2.54mm
- R10, R11, R7, R8, R9: value 10k -> 100k
Connections:
- wire segments 335 -> 352
Changed lines of the file:
@@
 	4500 1900 3450 1900
 Wire Wire Line
-	3450 1900 3450 2300
+	3450 1900 3450 1950
 Connection ~ 3450 2300
 Wire Wire Line
@@
 P 13800 3050
 F 0 "R7" H 13900 3100 50  0000 L CNN
-F 1 "10k" H 13900 3000 50  0000 L CNN
+F 1 "100k" H 13900 3000 50  0000 L CNN
 F 2 "Resistors_SMD:R_0603_HandSoldering" V 13730 3050 50  0001 C CNN
 F 3 "~" H 13800 3050 50  0001 C CNN
@@
 P 13800 4500
 F 0 "R8" H 13900 4550 50  0000 L CNN
-F 1 "10k" H 13900 4450 50  0000 L CNN
+F 1 "100k" H 13900 4450 50  0000 L CNN
 F 2 "Resistors_SMD:R_0603_HandSoldering" V 13730 4500 50  0001 C CNN
 F 3 "~" H 13800 4500 50  0001 C CNN
@@
 P 13800 6000
 F 0 "R9" H 13900 6050 50  0000 L CNN
-F 1 "10k" H 13900 5950 50  0000 L CNN
+F 1 "100k" H 13900 5950 50  0000 L CNN
 F 2 "Resistors_SMD:R_0603_HandSoldering" V 13730 6000 50  0001 C CNN
 F 3 "~" H 13800 6000 50  0001 C CNN
@@
 P 13800 7450
 F 0 "R10" H 13900 7500 50  0000 L CNN
-F 1 "10k" H 13900 7400 50  0000 L CNN
+F 1 "100k" H 13900 7400 50  0000 L CNN
 F 2 "Resistors_SMD:R_0603_HandSoldering" V 13730 7450 50  0001 C CNN
 F 3 "~" H 13800 7450 50  0001 C CNN
@@
 P 13800 8850
 F 0 "R11" H 13900 8900 50  0000 L CNN
-F 1 "10k" H 13900 8800 50  0000 L CNN
+F 1 "100k" H 13900 8800 50  0000 L CNN
 F 2 "Resistors_SMD:R_0603_HandSoldering" V 13730 8850 50  0001 C CNN
 F 3 "~" H 13800 8850 50  0001 C CNN
@@
 F 0 "J4" H 15230 6342 50  0000 L CNN
 F 1 "Temperature" H 15230 6251 50  0000 L CNN
-F 2 "Pin_Headers:Pin_Header_Straight_1x10_Pitch2.54mm" H 15150 6350 50  0001 C CNN
+F 2 "Pin_Headers:Pin_Header_Angled_1x10_Pitch2.54mm" H 15150 6350 50  0001 C CNN
 F 3 "~" H 15150 6350 50  0001 C CNN
 	1    15150 6350
@@
 NoConn ~ 1150 3300
 NoConn ~ 1150 3550
+$Comp
+L Diode:BZT52Bxx D?
+U 1 1 5CCBA78B
+P 2900 2700
+F 0 "D?" V 2854 2779 50  0000 L CNN
+F 1 "BZT52Bxx" V 2945 2779 50  0000 L CNN
+F 2 "Diode_SMD:D_SOD-123" H 2900 2525 50  0001 C CNN
+F 3 "https://diotec.com/tl_files/diotec/files/pdf/datasheets/bzt52b2v4.pdf" H 2900 2700 50  0001 C CNN
+	1    2900 2700
+	0    1    1    0
+$EndComp
+Wire Wire Line
+	2900 1650 3450 1650
+Connection ~ 3450 1650
+$Comp
+L power:GND #PWR?
+U 1 1 5CCDBC4F
+P 2900 3150
+F 0 "#PWR?" H 2900 2900 50  0001 C CNN
+F 1 "GND" H 2905 2977 50  0000 C CNN
+F 2 "" H 2900 3150 50  0001 C CNN
+F 3 "" H 2900 3150 50  0001 C CNN
+	1    2900 3150
+	1    0    0    -1
+$EndComp
+$Comp
+L Diode:1N4148W D?
+U 1 1 5CCFC663
+P 2400 2700
+F 0 "D?" V 2354 2780 50  0000 L CNN
+F 1 "1N4148W" V 2445 2780 50  0000 L CNN
+F 2 "Diode_SMD:D_SOD-123" H 2400 2525 50  0001 C CNN
+F 3 "https://www.vishay.com/docs/85748/1n4148w.pdf" H 2400 2700 50  0001 C CNN
+	1    2400 2700
+	0    1    1    0
+$EndComp
+$Comp
+L Diode:1N4148W D?
+U 1 1 5CCFD72B
+P 1900 2700
+F 0 "D?" V 1854 2780 50  0000 L CNN
+F 1 "1N4148W" V 1945 2780 50  0000 L CNN
+F 2 "Diode_SMD:D_SOD-123" H 1900 2525 50  0001 C CNN
+F 3 "https://www.vishay.com/docs/85748/1n4148w.pdf" H 1900 2700 50  0001 C CNN
+	1    1900 2700
+	0    1    1    0
+$EndComp
+Wire Wire Line
+	2900 1650 2900 2300
+Wire Wire Line
+	1900 2550 1900 2300
+Wire Wire Line
+	1900 2300 2400 2300
+Connection ~ 2900 2300
+Wire Wire Line
+	2900 2300 2900 2550
+Wire Wire Line
+	2400 2550 2400 2300
+Connection ~ 2400 2300
+Wire Wire Line
+	2400 2300 2900 2300
+Wire Wire Line
+	1900 2850 1900 3150
+Wire Wire Line
+	2400 2850 2400 3150
+$Comp
+L power:GND #PWR?
+U 1 1 5CDE7639
+P 2400 3150
+F 0 "#PWR?" H 2400 2900 50  0001 C CNN
+F 1 "GND" H 2405 2977 50  0000 C CNN
+F 2 "" H 2400 3150 50  0001 C CNN
+F 3 "" H 2400 3150 50  0001 C CNN
+	1    2400 3150
+	1    0    0    -1
+$EndComp
+$Comp
+L power:GND #PWR?
+U 1 1 5CDE7903
+P 1900 3150
+F 0 "#PWR?" H 1900 2900 50  0001 C CNN
+F 1 "GND" H 1905 2977 50  0000 C CNN
+F 2 "" H 1900 3150 50  0001 C CNN
+F 3 "" H 1900 3150 50  0001 C CNN
+	1    1900 3150
+	1    0    0    -1
+$EndComp
+Wire Wire Line
+	2900 2850 2900 3150
+$Comp
+L Device:Ferrite_Bead FB?
+U 1 1 5CE2B099
+P 3450 2100
+F 0 "FB?" H 3587 2146 50  0000 L CNN
+F 1 "Ferrite_Bead" H 3587 2055 50  0000 L CNN
+F 2 "Resistor_SMD:R_0603_1608Metric" V 3380 2100 50  0001 C CNN
+F 3 "~" H 3450 2100 50  0001 C CNN
+	1    3450 2100
+	1    0    0    -1
+$EndComp
+Wire Wire Line
+	3450 2250 3450 2300
+$Comp
+L Device:C C?
+U 1 1 5CE2C6B5
+P 10200 5700
+F 0 "C?" H 10315 5746 50  0000 L CNN
+F 1 "1u" H 10315 5655 50  0000 L CNN
+F 2 "Capacitors_SMD:C_0805_HandSoldering" H 10238 5550 50  0001 C CNN
+F 3 "~" H 10200 5700 50  0001 C CNN
+	1    10200 5700
+	1    0    0    -1
+$EndComp
+$Comp
+L Device:C C?
+U 1 1 5CE2C9EA
+P 10550 5700
+F 0 "C?" H 10665 5746 50  0000 L CNN
+F 1 "1u" H 10665 5655 50  0000 L CNN
+F 2 "Capacitors_SMD:C_0805_HandSoldering" H 10588 5550 50  0001 C CNN
+F 3 "~" H 10550 5700 50  0001 C CNN
+	1    10550 5700
+	1    0    0    -1
+$EndComp
+Wire Wire Line
+	9850 5450 10200 5450
+Wire Wire Line
+	10200 5450 10200 5550
+Wire Wire Line
+	10200 5450 10550 5450
+Wire Wire Line
+	10550 5450 10550 5550
+Connection ~ 10200 5450
+Wire Wire Line
+	10550 5850 10200 5850
+Connection ~ 9850 5850
+Connection ~ 10200 5850
+Wire Wire Line
+	10200 5850 9850 5850
 $EndSCHEMATC

Commit message: ltc6811
Parts:
- D13, D14, D15: renamed from D?; footprint Diode_SMD:D_SOD-123 -> Diodes_SMD:D_SOD-123
- FB1: renamed from FB?; footprint Resistor_SMD:R_0603_1608Metric -> Resistors_SMD:R_0603_HandSoldering
- gave numbers to parts that had none: 2
Changed lines of the file:
@@
-EESchema Schematic File Version 4
+EESchema Schematic File Version 5
 LIBS:LTC6811-cache
 EELAYER 29 0
@@
 NoConn ~ 1150 3550
 $Comp
-L Diode:BZT52Bxx D?
+L Diode:BZT52Bxx D15
 U 1 1 5CCBA78B
 P 2900 2700
-F 0 "D?" V 2854 2779 50  0000 L CNN
+F 0 "D15" V 2854 2779 50  0000 L CNN
 F 1 "BZT52Bxx" V 2945 2779 50  0000 L CNN
-F 2 "Diode_SMD:D_SOD-123" H 2900 2525 50  0001 C CNN
+F 2 "Diodes_SMD:D_SOD-123" H 2900 2525 50  0001 C CNN
 F 3 "https://diotec.com/tl_files/diotec/files/pdf/datasheets/bzt52b2v4.pdf" H 2900 2700 50  0001 C CNN
 	1    2900 2700
@@
 Connection ~ 3450 1650
 $Comp
-L power:GND #PWR?
+L power:GND #PWR0123
 U 1 1 5CCDBC4F
 P 2900 3150
-F 0 "#PWR?" H 2900 2900 50  0001 C CNN
+F 0 "#PWR0123" H 2900 2900 50  0001 C CNN
 F 1 "GND" H 2905 2977 50  0000 C CNN
 F 2 "" H 2900 3150 50  0001 C CNN
@@
 $EndComp
 $Comp
-L Diode:1N4148W D?
+L Diode:1N4148W D14
 U 1 1 5CCFC663
 P 2400 2700
-F 0 "D?" V 2354 2780 50  0000 L CNN
+F 0 "D14" V 2354 2780 50  0000 L CNN
 F 1 "1N4148W" V 2445 2780 50  0000 L CNN
-F 2 "Diode_SMD:D_SOD-123" H 2400 2525 50  0001 C CNN
+F 2 "Diodes_SMD:D_SOD-123" H 2400 2525 50  0001 C CNN
 F 3 "https://www.vishay.com/docs/85748/1n4148w.pdf" H 2400 2700 50  0001 C CNN
 	1    2400 2700
@@
 $EndComp
 $Comp
-L Diode:1N4148W D?
+L Diode:1N4148W D13
 U 1 1 5CCFD72B
 P 1900 2700
-F 0 "D?" V 1854 2780 50  0000 L CNN
+F 0 "D13" V 1854 2780 50  0000 L CNN
 F 1 "1N4148W" V 1945 2780 50  0000 L CNN
-F 2 "Diode_SMD:D_SOD-123" H 1900 2525 50  0001 C CNN
+F 2 "Diodes_SMD:D_SOD-123" H 1900 2525 50  0001 C CNN
 F 3 "https://www.vishay.com/docs/85748/1n4148w.pdf" H 1900 2700 50  0001 C CNN
 	1    1900 2700
@@
 	2400 2850 2400 3150
 $Comp
-L power:GND #PWR?
+L power:GND #PWR0124
 U 1 1 5CDE7639
 P 2400 3150
-F 0 "#PWR?" H 2400 2900 50  0001 C CNN
+F 0 "#PWR0124" H 2400 2900 50  0001 C CNN
 F 1 "GND" H 2405 2977 50  0000 C CNN
 F 2 "" H 2400 3150 50  0001 C CNN
@@
 $EndComp
 $Comp
-L power:GND #PWR?
+L power:GND #PWR0125
 U 1 1 5CDE7903
 P 1900 3150
-F 0 "#PWR?" H 1900 2900 50  0001 C CNN
+F 0 "#PWR0125" H 1900 2900 50  0001 C CNN
 F 1 "GND" H 1905 2977 50  0000 C CNN
 F 2 "" H 1900 3150 50  0001 C CNN
@@
 	2900 2850 2900 3150
 $Comp
-L Device:Ferrite_Bead FB?
+L Device:Ferrite_Bead FB1
 U 1 1 5CE2B099
 P 3450 2100
-F 0 "FB?" H 3587 2146 50  0000 L CNN
+F 0 "FB1" H 3587 2146 50  0000 L CNN
 F 1 "Ferrite_Bead" H 3587 2055 50  0000 L CNN
-F 2 "Resistor_SMD:R_0603_1608Metric" V 3380 2100 50  0001 C CNN
+F 2 "Resistors_SMD:R_0603_HandSoldering" V 3380 2100 50  0001 C CNN
 F 3 "~" H 3450 2100 50  0001 C CNN
 	1    3450 2100
@@
 	3450 2250 3450 2300
 $Comp
-L Device:C C?
+L Device:C C25
 U 1 1 5CE2C6B5
 P 10200 5700
-F 0 "C?" H 10315 5746 50  0000 L CNN
+F 0 "C25" H 10315 5746 50  0000 L CNN
 F 1 "1u" H 10315 5655 50  0000 L CNN
 F 2 "Capacitors_SMD:C_0805_HandSoldering" H 10238 5550 50  0001 C CNN
@@
 $EndComp
 $Comp
-L Device:C C?
+L Device:C C26
 U 1 1 5CE2C9EA
 P 10550 5700
-F 0 "C?" H 10665 5746 50  0000 L CNN
+F 0 "C26" H 10665 5746 50  0000 L CNN
 F 1 "1u" H 10665 5655 50  0000 L CNN
 F 2 "Capacitors_SMD:C_0805_HandSoldering" H 10588 5550 50  0001 C CNN

Commit message: LTC6811 minor changes
Parts:
- removed C10, C11, C8, C9: 100n, Capacitors_SMD:C_0603_HandSoldering, symbol Device:C
- removed J4: Temperature, Pin_Headers:Pin_Header_Angled_1x10_Pitch2.54mm, symbol Connector_Generic:Conn_01x10
- removed R10, R7, R8, R9: 100k, Resistors_SMD:R_0603_HandSoldering, symbol Device:R
- added J4: Conn_01x04_Female, symbol Connector:Conn_01x04_Female
- added J? (x2): Conn_01x03_Female, symbol Connector:Conn_01x03_Female
Connections:
- net labels added: Analog, GPIO, SCL, SDA
- net labels removed: T2, T3, T4, T5
- wire segments 352 -> 323

Commit message: LTC6811 now more compact
Parts:
- removed J4: Conn_01x04_Female, symbol Connector:Conn_01x04_Female
- removed J? (x2): Conn_01x03_Female, symbol Connector:Conn_01x03_Female
- added J10, J9: Conn_01x03, Pin_Headers:Pin_Header_Angled_1x03_Pitch2.54mm, symbol Connector_Generic:Conn_01x03
- added J11: Conn_01x04, Pin_Headers:Pin_Header_Straight_1x04_Pitch2.54mm, symbol Connector_Generic:Conn_01x04
- added J4: Conn_01x04, Pin_Headers:Pin_Header_Angled_1x04_Pitch2.54mm, symbol Connector_Generic:Conn_01x04
Connections:
- wire segments 323 -> 335
Changed lines of the file:
@@
-EESchema Schematic File Version 4
+EESchema Schematic File Version 5
 LIBS:LTC6811-cache
 EELAYER 29 0
@@
 Connection ~ 10750 1250
 Wire Wire Line
-	10750 1250 12050 1250
+	10750 1250 12000 1250
 Wire Wire Line
 	10750 1600 10750 1650
@@
 Connection ~ 10750 2250
 Wire Wire Line
-	10750 2250 12050 2250
+	10750 2250 11800 2250
 $Comp
 L Device:C C7
@@
 $EndComp
 Wire Wire Line
-	11800 1450 12050 1450
-Wire Wire Line
-	12050 2050 11800 2050
+	11800 1450 11950 1450
+Wire Wire Line
+	12050 2050 11850 2050
 $Comp
 L power:GND #PWR0101
@@
 Text Label 7900 5750 2    50   ~ 0
 SDA
-Wire Wire Line
-	7900 5650 7650 5650
-Text Label 7900 5650 2    50   ~ 0
-SCL
 Connection ~ 8900 6350
 Text Label 7950 4150 0    50   ~ 0
@@
 Wire Wire Line
 	10200 5850 9850 5850
-$Comp
-L Connector:Conn_01x04_Female J4
-U 1 1 5DC5EEB7
-P 14100 5450
-F 0 "J4" H 14128 5426 50  0000 L CNN
-F 1 "Conn_01x04_Female" H 14128 5335 50  0000 L CNN
-F 2 "" H 14100 5450 50  0001 C CNN
-F 3 "~" H 14100 5450 50  0001 C CNN
-	1    14100 5450
-	1    0    0    -1
-$EndComp
 Wire Wire Line
 	13650 5350 13900 5350
@@
 Wire Wire Line
 	13900 5450 13650 5450
-Text Label 13650 5450 2    50   ~ 0
-SCL
 Wire Wire Line
 	13650 5800 13650 5650
@@
 	1    0    0    -1
 $EndComp
-$Comp
-L Connector:Conn_01x03_Female J?
-U 1 1 5DF0E297
-P 13750 6700
-F 0 "J?" H 13778 6726 50  0000 L CNN
-F 1 "Conn_01x03_Female" H 13778 6635 50  0000 L CNN
-F 2 "" H 13750 6700 50  0001 C CNN
-F 3 "~" H 13750 6700 50  0001 C CNN
-	1    13750 6700
-	1    0    0    -1
-$EndComp
-$Comp
-L Connector:Conn_01x03_Female J?
-U 1 1 5DF0ED74
-P 13750 7400
-F 0 "J?" H 13778 7426 50  0000 L CNN
-F 1 "Conn_01x03_Female" H 13778 7335 50  0000 L CNN
-F 2 "" H 13750 7400 50  0001 C CNN
-F 3 "~" H 13750 7400 50  0001 C CNN
-	1    13750 7400
-	1    0    0    -1
-$EndComp
 Text Label 13350 6700 2    50   ~ 0
 GPIO
@@
 	13350 7400 13550 7400
 $Comp
-L power:GND #PWR?
+L power:GND #PWR0103
 U 1 1 5DF4AF4A
 P 13450 6900
-F 0 "#PWR?" H 13450 6650 50  0001 C CNN
+F 0 "#PWR0103" H 13450 6650 50  0001 C CNN
 F 1 "GND" H 13455 6727 50  0000 C CNN
 F 2 "" H 13450 6900 50  0001 C CNN
@@
 	13450 6800 13550 6800
 $Comp
-L power:GND #PWR?
+L power:GND #PWR0104
 U 1 1 5DF698CB
 P 13450 7550
-F 0 "#PWR?" H 13450 7300 50  0001 C CNN
+F 0 "#PWR0104" H 13450 7300 50  0001 C CNN
 F 1 "GND" H 13455 7377 50  0000 C CNN
 F 2 "" H 13450 7550 50  0001 C CNN
@@
 Wire Wire Line
 	13350 7300 13550 7300
+$Comp
+L Connector_Generic:Conn_01x04 J4
+U 1 1 5CCE4863
+P 14100 5450
+F 0 "J4" H 14180 5442 50  0000 L CNN
+F 1 "Conn_01x04" H 14180 5351 50  0000 L CNN
+F 2 "Pin_Headers:Pin_Header_Angled_1x04_Pitch2.54mm" H 14100 5450 50  0001 C CNN
+F 3 "~" H 14100 5450 50  0001 C CNN
+	1    14100 5450
+	1    0    0    -1
+$EndComp
+$Comp
+L Connector_Generic:Conn_01x03 J9
+U 1 1 5CCE6461
+P 13750 6700
+F 0 "J9" H 13830 6742 50  0000 L CNN
+F 1 "Conn_01x03" H 13830 6651 50  0000 L CNN
+F 2 "Pin_Headers:Pin_Header_Angled_1x03_Pitch2.54mm" H 13750 6700 50  0001 C CNN
+F 3 "~" H 13750 6700 50  0001 C CNN
+	1    13750 6700
+	1    0    0    -1
+$EndComp
+$Comp
+L Connector_Generic:Conn_01x03 J10
+U 1 1 5CCE74BE
+P 13750 7400
+F 0 "J10" H 13830 7442 50  0000 L CNN
+F 1 "Conn_01x03" H 13830 7351 50  0000 L CNN
+F 2 "Pin_Headers:Pin_Header_Angled_1x03_Pitch2.54mm" H 13750 7400 50  0001 C CNN
+F 3 "~" H 13750 7400 50  0001 C CNN
+	1    13750 7400
+	1    0    0    -1
+$EndComp
+Text Label 13650 5450 2    50   ~ 0
+SCL
+Text Label 7900 5650 2    50   ~ 0
+SCL
+Wire Wire Line
+	7650 5650 7900 5650
+$Comp
+L Connector_Generic:Conn_01x04 J11
+U 1 1 5CDB7EDD
+P 12250 2650
+F 0 "J11" H 12330 2642 50  0000 L CNN
+F 1 "Conn_01x04" H 12330 2551 50  0000 L CNN
+F 2 "Pin_Headers:Pin_Header_Straight_1x04_Pitch2.54mm" H 12250 2650 50  0001 C CNN
+F 3 "~" H 12250 2650 50  0001 C CNN
+	1    12250 2650
+	1    0    0    -1
+$EndComp
+Wire Wire Line
+	12000 1250 12000 2550
+Wire Wire Line
+	12000 2550 12050 2550
+Connection ~ 12000 1250
+Wire Wire Line
+	12000 1250 12050 1250
+Wire Wire Line
+	11950 1450 11950 2650
+Wire Wire Line
+	11950 2650 12050 2650
+Connection ~ 11950 1450
+Wire Wire Line
+	11950 1450 12050 1450
+Wire Wire Line
+	11850 2050 11850 2750
+Wire Wire Line
+	11850 2750 12050 2750
+Connection ~ 11850 2050
+Wire Wire Line
+	11850 2050 11800 2050
+Wire Wire Line
+	11800 2250 11800 2850
+Wire Wire Line
+	11800 2850 12050 2850
+Connection ~ 11800 2250
+Wire Wire Line
+	11800 2250 12050 2250
 $EndSCHEMATC

Commit message: readme
Parts:
- added TH?: 100k, Resistors_SMD:R_0805_HandSoldering, symbol Device:Thermistor
Connections:
- net GND: now also TH?.2
- net T1: now also TH?.1
Changed lines of the file:
@@
 	13800 9200 13800 9300
 Wire Wire Line
-	14300 9200 13800 9200
+	14400 9200 14250 9200
 Connection ~ 13800 9200
 Wire Wire Line
@@
 	1    0    0    -1
 $EndComp
-Text Label 14300 9200 2    50   ~ 0
+Text Label 14400 9200 2    50   ~ 0
 T1
 Wire Wire Line
@@
 Wire Wire Line
 	11800 2250 12050 2250
+$Comp
+L Device:Thermistor TH?
+U 1 1 5CD17B07
+P 14250 9450
+F 0 "TH?" H 14355 9496 50  0000 L CNN
+F 1 "100k" H 14355 9405 50  0000 L CNN
+F 2 "Resistors_SMD:R_0805_HandSoldering" H 14250 9450 50  0001 C CNN
+F 3 "~" H 14250 9450 50  0001 C CNN
+	1    14250 9450
+	1    0    0    -1
+$EndComp
+Wire Wire Line
+	14250 9250 14250 9200
+Connection ~ 14250 9200
+Wire Wire Line
+	14250 9200 13800 9200
+Wire Wire Line
+	14250 9650 13800 9650
+Connection ~ 13800 9650
 $EndSCHEMATC

Commit message: pic changes
Parts:
- removed JP1, JP2: Jumper_NC_Dual, Pin_Headers:Pin_Header_Straight_1x03_Pitch2.54mm, symbol Device:Jumper_NC_Dual
- added R7: 1k, Resistors_SMD:R_0603_HandSoldering, symbol Device:R
- gave numbers to parts that had none: 1
Connections:
- net DTEN is gone; now on net GND: U1.36 (DTEN)
- net Vreg: now also R7.2
- net WDT: no longer names the net of U1.39 (WDT)
- net WDT: now also R7.1
Changed lines of the file:
@@
-EESchema Schematic File Version 5
+EESchema Schematic File Version 4
 LIBS:LTC6811-cache
 EELAYER 29 0
@@
 	7650 4950 8350 4950
 Wire Wire Line
-	8350 4950 8350 5250
+	8350 4950 8350 5050
 Wire Wire Line
 	7650 5250 8350 5250
@@
 NoConn ~ 7650 4550
 NoConn ~ 7650 4650
-Text Label 8000 5050 0    50   ~ 0
-WDT
-Wire Wire Line
-	8000 5050 7650 5050
-Text Label 2150 1450 0    50   ~ 0
-WDT
-Text Label 8000 5350 0    50   ~ 0
-DTEN
 Wire Wire Line
 	8900 4450 8900 5850
-Wire Wire Line
-	8000 5350 7650 5350
-Text Label 850  1400 0    50   ~ 0
-DTEN
-$Comp
-L power:GND #PWR0121
-U 1 1 5CD4DCEC
-P 1850 1900
-F 0 "#PWR0121" H 1850 1650 50  0001 C CNN
-F 1 "GND" H 1855 1727 50  0000 C CNN
-F 2 "" H 1850 1900 50  0001 C CNN
-F 3 "" H 1850 1900 50  0001 C CNN
-	1    1850 1900
-	1    0    0    -1
-$EndComp
-$Comp
-L Device:Jumper_NC_Dual JP1
-U 1 1 5CD4E774
-P 1300 1400
-F 0 "JP1" V 1300 1502 50  0000 L CNN
-F 1 "Jumper_NC_Dual" V 1345 1502 50  0001 L CNN
-F 2 "Pin_Headers:Pin_Header_Straight_1x03_Pitch2.54mm" H 1300 1400 50  0001 C CNN
-F 3 "~" H 1300 1400 50  0001 C CNN
-	1    1300 1400
-	0    1    1    0
-$EndComp
-Wire Wire Line
-	1300 1650 1300 1900
-Wire Wire Line
-	1300 1900 1850 1900
-$Comp
-L Device:Jumper_NC_Dual JP2
-U 1 1 5CD79FAF
-P 2550 1450
-F 0 "JP2" V 2550 1552 50  0000 L CNN
-F 1 "Jumper_NC_Dual" V 2595 1552 50  0001 L CNN
-F 2 "Pin_Headers:Pin_Header_Straight_1x03_Pitch2.54mm" H 2550 1450 50  0001 C CNN
-F 3 "~" H 2550 1450 50  0001 C CNN
-	1    2550 1450
-	0    1    1    0
-$EndComp
-Wire Wire Line
-	2550 1700 2550 1900
-Wire Wire Line
-	2550 1900 1850 1900
-Connection ~ 1850 1900
-Wire Wire Line
-	850  1400 1200 1400
-Wire Wire Line
-	2150 1450 2450 1450
-Text Label 2550 950  0    50   ~ 0
-Vreg
-Wire Wire Line
-	2550 950  2550 1200
-Text Label 1300 950  0    50   ~ 0
-Vreg
-Wire Wire Line
-	1300 950  1300 1150
 Wire Wire Line
 	4400 8500 4200 8500
@@
 	11800 2250 12050 2250
 $Comp
-L Device:Thermistor TH?
+L Device:Thermistor TH1
 U 1 1 5CD17B07
 P 14250 9450
-F 0 "TH?" H 14355 9496 50  0000 L CNN
+F 0 "TH1" H 14355 9496 50  0000 L CNN
 F 1 "100k" H 14355 9405 50  0000 L CNN
 F 2 "Resistors_SMD:R_0805_HandSoldering" H 14250 9450 50  0001 C CNN
@@
 	14250 9650 13800 9650
 Connection ~ 13800 9650
+$Comp
+L power:GND #PWR0105
+U 1 1 5CDC06E6
+P 8650 5400
+F 0 "#PWR0105" H 8650 5150 50  0001 C CNN
+F 1 "GND" H 8655 5227 50  0000 C CNN
+F 2 "" H 8650 5400 50  0001 C CNN
+F 3 "" H 8650 5400 50  0001 C CNN
+	1    8650 5400
+	1    0    0    -1
+$EndComp
+Wire Wire Line
+	8650 5350 8650 5400
+Wire Wire Line
+	7650 5350 8650 5350
+Wire Wire Line
+	7650 5050 7750 5050
+Connection ~ 8350 5050
+Wire Wire Line
+	8350 5050 8350 5250
+$Comp
+L Device:R R7
+U 1 1 5CE23298
+P 7900 5050
+F 0 "R7" V 7950 5200 50  0000 L CNN
+F 1 "1k" V 7950 4800 50  0000 L CNN
+F 2 "Resistors_SMD:R_0603_HandSoldering" V 7830 5050 50  0001 C CNN
+F 3 "~" H 7900 5050 50  0001 C CNN
+	1    7900 5050
+	0    -1   -1   0
+$EndComp
+Wire Wire Line
+	8050 5050 8350 5050
 $EndSCHEMATC
