File: current_sensor/PCB/isolated_current_sensor.sch (KiCad schematic (older format))
At the start: 7 parts, among them U3 AMC1303

Commit message: update
Parts:
- U3: value AMC1303 -> AMC1303E0510
Changed lines of the file:
@@
 AR Path="/598FD705/585AEFF8" Ref="U3"  Part="1"
 F 0 "U3" H 5900 4537 60  0000 C CNN
-F 1 "AMC1303" H 5900 4431 60  0000 C CNN
+F 1 "AMC1303E0510" H 5900 4431 60  0000 C CNN
 F 2 "IPC7351-Nominal:SOIC127P1032X265-8" H 5800 3200 60  0001 C CNN
 F 3 "http://www.ti.com/lit/ds/symlink/amc1301.pdf" H 5900 3850 60  0001 C CNN
