File: PSU/24-150V DC in/PSU.sch (KiCad schematic (older format))
At the start: 40 parts, among them J1 12V OUT, J2 0-150V IN, Q1 FDMS86252L, Q2 BSC110N15NS5, U1 LTC7801

Commit message: Readme update
No more sd card & wireless options
Parts:
- U1: symbol PSU-rescue:LTC7801-moje-besc-g2-rescue -> PSU-rescue:LTC7801-moje-besc-g2-rescue-PSU-rescue
Changed lines of the file:
@@
 $EndComp
 $Comp
-L PSU-rescue:LTC7801-moje-besc-g2-rescue U1
+L PSU-rescue:LTC7801-moje-besc-g2-rescue-PSU-rescue U1
 U 1 1 5D5ACCCE
 P 4550 4750
