File: Master/LV/PCB/PowerSupply.sch (KiCad schematic (older format))
At the start: 30 parts, among them Q28 BSS138, Q29 BSS138, Q30 BSS138, U19 LM5165YDRC

Commit message: LVupdates
Parts:
- C88: footprint Capacitors_SMD:C_0603_HandSoldering -> Capacitor_SMD:C_0603_1608Metric; MPN (none) -> GRM188R61A225KE34D; Volatge 50V -> (none)
- C89, C90: footprint Capacitors_SMD:C_0805_HandSoldering -> Capacitor_SMD:C_0805_2012Metric; MPN (none) -> CL21A226MOQNNNE; Volatge 50V -> (none); Voltage (none) -> 50V
- C91: footprint Capacitors_SMD:C_0603_HandSoldering -> Capacitor_SMD:C_0603_1608Metric; MPN (none) -> GCM188R71H473KA55D; Volatge 50V -> (none); Voltage (none) -> 50V
- C92, C93, C94: footprint Capacitors_SMD:C_0603_HandSoldering -> Capacitor_SMD:C_0603_1608Metric; MPN (none) -> CL10A106MQ8NNNC; Volatge 50V -> (none); Voltage (none) -> 50V
- D10, D7: MPN (none) -> BZT52C16-E3-08
- D11, D12, D13, D8, D9: MPN (none) -> 1N4148W-7-F
- L3: MPN (none) -> 744043151
- Q28, Q29, Q30: MPN (none) -> BSS138
- R172: footprint Resistors_SMD:R_0603_HandSoldering -> Resistor_SMD:R_0603_1608Metric; MPN (none) -> RC0603FR-07100RL
- R173, R176, R178: footprint Resistors_SMD:R_0603_HandSoldering -> Resistor_SMD:R_0603_1608Metric; MPN (none) -> RMCF2512JT10K0
- R174: footprint Resistors_SMD:R_0603_HandSoldering -> Resistor_SMD:R_0603_1608Metric; MPN (none) -> RC0603JR-071ML
- R175, R177: footprint Resistors_SMD:R_0805_HandSoldering -> Resistor_SMD:R_0603_1608Metric; MPN (none) -> RC0603FR-074M7L
- R179: footprint Resistors_SMD:R_0603_HandSoldering -> Resistor_SMD:R_0603_1608Metric; MPN (none) -> RC0603FR-07130KL
- R180, R181, R182: footprint Resistors_SMD:R_0603_HandSoldering -> Resistor_SMD:R_0603_1608Metric; MPN (none) -> RC0603FR-071RL
- U19: MPN (none) -> LM5165YDRCT
Connections:
- net Power renamed 12V
Other:
- moved on the sheet: C88, C89, C90, C91, C92, C93, C94, D10, D11, D12, D13, D7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
