File: Master/LV/PCB/switches.sch (KiCad schematic (older format))
At the start: 15 parts, among them Q3 BSS138, Q4 BUK98150-55A, Q5 BUK98150-55A, Q6 BUK98150-55A, Q7 BUK98150-55A

Commit message: LVupdates
Parts:
- Q3: MPN (none) -> BSS138
- Q4, Q5, Q6, Q7: MPN (none) -> BUK98150-55A/CUF
- R19: footprint Resistors_SMD:R_0603_HandSoldering -> Resistor_SMD:R_0603_1608Metric; MPN (none) -> RMCF2512JT10K0
- R23, R24, R25, R32: footprint Resistors_SMD:R_0603_HandSoldering -> Resistor_SMD:R_0603_1608Metric; MPN (none) -> RC0603JR-0710RL
- R27, R28, R33, R8: footprint Resistors_SMD:R_0603_HandSoldering -> Resistor_SMD:R_0603_1608Metric; MPN (none) -> RC0603FR-074M7L
- TH1: footprint Resistors_SMD:R_0805_HandSoldering -> Resistor_SMD:R_0805_2012Metric; MPN (none) -> SDNT2012X104F4250FTF
Other:
- moved on the sheet: R19
Changed lines of the file:
@@
 $Descr A3 16535 11693
 encoding utf-8
-Sheet 6 7
+Sheet 5 7
 Title ""
 Date ""
@@
 F 2 "TO_SOT_Packages_SMD:SOT-23" H 5900 6625 50  0001 L CIN
 F 3 "https://www.fairchildsemi.com/datasheets/BS/BSS138.pdf" H 5700 6700 50  0001 L CNN
+F 4 "BSS138" H 5700 6700 50  0001 C CNN "MPN"
 	1    5700 6700
 	1    0    0    -1
 $EndComp
-Text HLabel 3450 7450 0    50   Input ~ 0
+Text HLabel 3700 6700 0    50   Input ~ 0
 Safety
-Wire Wire Line
-	5250 7450 5250 7100
-Wire Wire Line
-	5250 7100 5500 7100
-Wire Wire Line
-	5500 6700 5500 7100
 Wire Wire Line
 	5800 6900 5800 7050
@@
 F 0 "TH1" H 3147 9304 50  0000 R CNN
 F 1 "Thermistor_NTC 100k" H 3147 9395 50  0000 R CNN
-F 2 "Resistors_SMD:R_0805_HandSoldering" H 3300 9400 50  0001 C CNN
+F 2 "Resistor_SMD:R_0805_2012Metric" H 3300 9400 50  0001 C CNN
 F 3 "~" H 3300 9400 50  0001 C CNN
+F 4 "SDNT2012X104F4250FTF" H 3300 9350 50  0001 C CNN "MPN"
 	1    3300 9350
 	-1   0    0    1
@@
 F 2 "Package_TO_SOT_SMD:SOT-223" H 13600 3850 50  0001 C CNN
 F 3 "~" H 13400 3750 50  0001 C CNN
+F 4 "BUK98150-55A/CUF" H 13400 3750 50  0001 C CNN "MPN"
 	1    13400 3750
 	1    0    0    -1
@@
 F 2 "Package_TO_SOT_SMD:SOT-223" H 13600 5650 50  0001 C CNN
 F 3 "~" H 13400 5550 50  0001 C CNN
+F 4 "BUK98150-55A/CUF" H 13400 5550 50  0001 C CNN "MPN"
 	1    13400 5550
 	1    0    0    -1
@@
 F 2 "Package_TO_SOT_SMD:SOT-223" H 13600 7600 50  0001 C CNN
 F 3 "~" H 13400 7500 50  0001 C CNN
+F 4 "BUK98150-55A/CUF" H 13400 7500 50  0001 C CNN "MPN"
 	1    13400 7500
 	1    0    0    -1
@@
 L power:+3.3V #PWR0138
 U 1 1 5D4B45BC
-P 3800 7150
-F 0 "#PWR0138" H 3800 7000 50  0001 C CNN
-F 1 "+3.3V" H 3815 7323 50  0000 C CNN
-F 2 "" H 3800 7150 50  0001 C CNN
-F 3 "" H 3800 7150 50  0001 C CNN
-	1    3800 7150
+P 4050 6400
+F 0 "#PWR0138" H 4050 6250 50  0001 C CNN
+F 1 "+3.3V" H 4065 6573 50  0000 C CNN
+F 2 "" H 4050 6400 50  0001 C CNN
+F 3 "" H 4050 6400 50  0001 C CNN
+	1    4050 6400
 	1    0    0    -1
 $EndComp
@@
 F 2 "Package_TO_SOT_SMD:SOT-223" H 13600 1950 50  0001 C CNN
 F 3 "~" H 13400 1850 50  0001 C CNN
+F 4 "BUK98150-55A/CUF" H 13400 1850 50  0001 C CNN "MPN"
 	1    13400 1850
 	1    0    0    -1
@@
 	3450 4250 8900 4250
 Wire Wire Line
-	3450 7450 3800 7450
+	3700 6700 4050 6700
 $Comp
 L power:GND #PWR0116
@@
 L Device:R R?
 U 1 1 5DC6C211
-P 3800 7300
+P 4050 6550
 AR Path="/5C519BA0/5DC6C211" Ref="R?"  Part="1"
 AR Path="/5D7DC460/5DC6C211" Ref="R?"  Part="1"
 AR Path="/5AC7323C/5DC6C211" Ref="R19"  Part="1"
-F 0 "R19" V 4007 7300 50  0000 C CNN
-F 1 "10k" V 3916 7300 50  0000 C CNN
-F 2 "Resistors_SMD:R_0603_HandSoldering" V 3730 7300 50  0001 C CNN
-F 3 "~" H 3800 7300 50  0001 C CNN
-	1    3800 7300
+F 0 "R19" V 4257 6550 50  0000 C CNN
+F 1 "10k" V 4166 6550 50  0000 C CNN
+F 2 "Resistor_SMD:R_0603_1608Metric" V 3980 6550 50  0001 C CNN
+F 3 "~" H 4050 6550 50  0001 C CNN
+F 4 "RMCF2512JT10K0" H 4050 6550 50  0001 C CNN "MPN"
+	1    4050 6550
 	1    0    0    -1
 $EndComp
@@
 F 0 "R23" V 12257 7500 50  0000 C CNN
 F 1 "10" V 12166 7500 50  0000 C CNN
-F 2 "Resistors_SMD:R_0603_HandSoldering" V 11980 7500 50  0001 C CNN
+F 2 "Resistor_SMD:R_0603_1608Metric" V 11980 7500 50  0001 C CNN
 F 3 "~" H 12050 7500 50  0001 C CNN
+F 4 "RC0603JR-0710RL" H 12050 7500 50  0001 C CNN "MPN"
 	1    12050 7500
 	0    1    1    0
@@
 F 0 "R25" V 12257 5550 50  0000 C CNN
 F 1 "10" V 12166 5550 50  0000 C CNN
-F 2 "Resistors_SMD:R_0603_HandSoldering" V 11980 5550 50  0001 C CNN
+F 2 "Resistor_SMD:R_0603_1608Metric" V 11980 5550 50  0001 C CNN
 F 3 "~" H 12050 5550 50  0001 C CNN
+F 4 "RC0603JR-0710RL" H 12050 5550 50  0001 C CNN "MPN"
 	1    12050 5550
 	0    1    1    0
@@
 F 0 "R24" V 12257 3750 50  0000 C CNN
 F 1 "10" V 12166 3750 50  0000 C CNN
-F 2 "Resistors_SMD:R_0603_HandSoldering" V 11980 3750 50  0001 C CNN
+F 2 "Resistor_SMD:R_0603_1608Metric" V 11980 3750 50  0001 C CNN
 F 3 "~" H 12050 3750 50  0001 C CNN
+F 4 "RC0603JR-0710RL" H 12050 3750 50  0001 C CNN "MPN"
 	1    12050 3750
 	0    1    1    0
@@
 F 0 "R32" V 12257 1850 50  0000 C CNN
 F 1 "10" V 12166 1850 50  0000 C CNN
-F 2 "Resistors_SMD:R_0603_HandSoldering" V 11980 1850 50  0001 C CNN
+F 2 "Resistor_SMD:R_0603_1608Metric" V 11980 1850 50  0001 C CNN
 F 3 "~" H 12050 1850 50  0001 C CNN
+F 4 "RC0603JR-0710RL" H 12050 1850 50  0001 C CNN "MPN"
 	1    12050 1850
 	0    1    1    0
@@
 F 0 "R33" V 13057 2100 50  0000 C CNN
 F 1 "4.7M" V 12966 2100 50  0000 C CNN
-F 2 "Resistors_SMD:R_0603_HandSoldering" V 12780 2100 50  0001 C CNN
+F 2 "Resistor_SMD:R_0603_1608Metric" V 12780 2100 50  0001 C CNN
 F 3 "~" H 12850 2100 50  0001 C CNN
+F 4 "RC0603FR-074M7L" H 12850 2100 50  0001 C CNN "MPN"
 	1    12850 2100
 	-1   0    0    1
@@
 F 0 "R27" V 13057 4000 50  0000 C CNN
 F 1 "4.7M" V 12966 4000 50  0000 C CNN
-F 2 "Resistors_SMD:R_0603_HandSoldering" V 12780 4000 50  0001 C CNN
+F 2 "Resistor_SMD:R_0603_1608Metric" V 12780 4000 50  0001 C CNN
 F 3 "~" H 12850 4000 50  0001 C CNN
+F 4 "RC0603FR-074M7L" H 12850 4000 50  0001 C CNN "MPN"
 	1    12850 4000
 	-1   0    0    1
@@
 F 0 "R28" V 13157 5800 50  0000 C CNN
 F 1 "4.7M" V 13066 5800 50  0000 C CNN
-F 2 "Resistors_SMD:R_0603_HandSoldering" V 12880 5800 50  0001 C CNN
+F 2 "Resistor_SMD:R_0603_1608Metric" V 12880 5800 50  0001 C CNN
 F 3 "~" H 12950 5800 50  0001 C CNN
+F 4 "RC0603FR-074M7L" H 12950 5800 50  0001 C CNN "MPN"
 	1    12950 5800
 	-1   0    0    1
@@
 F 0 "R8" V 13157 7750 50  0000 C CNN
 F 1 "4.7M" V 13066 7750 50  0000 C CNN
-F 2 "Resistors_SMD:R_0603_HandSoldering" V 12880 7750 50  0001 C CNN
+F 2 "Resistor_SMD:R_0603_1608Metric" V 12880 7750 50  0001 C CNN
 F 3 "~" H 12950 7750 50  0001 C CNN
+F 4 "RC0603FR-074M7L" H 12950 7750 50  0001 C CNN "MPN"
 	1    12950 7750
 	-1   0    0    1
 $EndComp
-Connection ~ 3800 7450
-Wire Wire Line
-	3800 7450 5250 7450
+Connection ~ 4050 6700
+Wire Wire Line
+	4050 6700 5500 6700
 $EndSCHEMATC

Commit message: Schematics updates & improvements
Changed lines of the file:
@@
 	1    0    0    -1
 $EndComp
-Text HLabel 3700 6700 0    50   Input ~ 0
+Text HLabel 2850 6700 0    50   Input ~ 0
 Safety
 Wire Wire Line
@@
 Wire Wire Line
 	3450 5050 5800 5050
-Wire Wire Line
-	5800 6500 5800 5050
 Connection ~ 5800 5050
 $Comp
@@
 Connection ~ 13500 7300
 Wire Wire Line
-	3450 3750 11900 3750
-Wire Wire Line
 	5800 5050 8600 5050
 Wire Wire Line
@@
 	3450 4250 8900 4250
 Wire Wire Line
-	3700 6700 4050 6700
+	2850 6700 4050 6700
 $Comp
 L power:GND #PWR0116
@@
 Wire Wire Line
 	4050 6700 5500 6700
+Wire Wire Line
+	5800 5050 5800 6500
+Wire Wire Line
+	3450 3750 11900 3750
 $EndSCHEMATC
