File: Slaves/LTC6813/18W/PCB/LTC6813.sch (KiCad schematic (older format))
At the start: 73 parts, among them J1 Conn_01x01, J10 Slave, J11 Master, J2 Conn_01x01, J3 Conn_01x01, J4 Conn_01x01, J5 Cells, J6 Temp, Q1 DZTT5551, U1 LTC6813

Commit message: Small changes to resistor & connectors
Now with vertical USB connectors & clip connectors
Parts:
- D3: value BZT52H-C62 -> MMSZ5268BT1G
- R2: value 1k -> 806
- R5: value 1k -> 1.2k
Changed lines of the file:
@@
 P 9300 3000
 F 0 "R5" V 9093 3000 50  0000 C CNN
-F 1 "1k" V 9184 3000 50  0000 C CNN
+F 1 "1.2k" V 9184 3000 50  0000 C CNN
 F 2 "Resistor_SMD:R_0603_1608Metric" V 9230 3000 50  0001 C CNN
 F 3 "~" H 9300 3000 50  0001 C CNN
@@
 P 8750 3000
 F 0 "R2" V 8543 3000 50  0000 C CNN
-F 1 "1k" V 8634 3000 50  0000 C CNN
+F 1 "806" V 8634 3000 50  0000 C CNN
 F 2 "Resistor_SMD:R_0603_1608Metric" V 8680 3000 50  0001 C CNN
 F 3 "~" H 8750 3000 50  0001 C CNN
@@
 P 4200 2850
 F 0 "D3" V 4154 2929 50  0000 L CNN
-F 1 "BZT52H-C62" V 4245 2929 50  0000 L CNN
+F 1 "MMSZ5268BT1G " V 4245 2929 50  0000 L CNN
 F 2 "Diodes_SMD:D_SOD-123" H 4200 2675 50  0001 C CNN
-F 3 "https://diotec.com/tl_files/diotec/files/pdf/datasheets/bzt52b2v4.pdf" H 4200 2850 50  0001 C CNN
+F 3 "" H 4200 2850 50  0001 C CNN
 	1    4200 2850
 	0    1    1    0
