File: Master/HV/PCB/PowerSupply.sch (KiCad schematic (older format))
At the start: 34 parts, among them J13 Charger 12V, Q2 BSS138, Q28 BSS138, Q29 BSS138, Q30 BSS138, U19 LM5165YDRC

Commit message: maintenance update
Parts:
- C88, C91, C92, C93, C94: footprint Capacitors_SMD:C_0603_HandSoldering -> Capacitor_SMD:C_0603_1608Metric
- C89, C90: footprint Capacitors_SMD:C_0805_HandSoldering -> Capacitor_SMD:C_0805_2012Metric
- R172, R173, R174, R175, R176, R177, R178, R179, R180, R181, R182, R41: footprint Resistors_SMD:R_0603_HandSoldering -> Resistor_SMD:R_0603_1608Metric
Changed lines of the file:
@@
 F 0 "C90" H 12200 6800 50  0000 L CNN
 F 1 "22u" H 12200 6900 50  0000 L CNN
-F 2 "Capacitors_SMD:C_0805_HandSoldering" H 12438 6700 50  0001 C CNN
+F 2 "Capacitor_SMD:C_0805_2012Metric" H 12438 6700 50  0001 C CNN
 F 3 "~" H 12400 6850 50  0001 C CNN
 F 4 "CL21A226MOQNNNE" H 12400 6850 50  0001 C CNN "MPN"
@@
 F 0 "C89" H 11700 6800 50  0000 L CNN
 F 1 "22u" H 11700 6900 50  0000 L CNN
-F 2 "Capacitors_SMD:C_0805_HandSoldering" H 11938 6700 50  0001 C CNN
+F 2 "Capacitor_SMD:C_0805_2012Metric" H 11938 6700 50  0001 C CNN
 F 3 "~" H 11900 6850 50  0001 C CNN
 F 4 "CL21A226MOQNNNE" H 11900 6850 50  0001 C CNN "MPN"
@@
 F 0 "R179" H 14330 7204 50  0000 R CNN
 F 1 "130k" H 14330 7295 50  0000 R CNN
-F 2 "Resistors_SMD:R_0603_HandSoldering" V 14330 7250 50  0001 C CNN
+F 2 "Resistor_SMD:R_0603_1608Metric" V 14330 7250 50  0001 C CNN
 F 3 "~" H 14400 7250 50  0001 C CNN
 F 4 "RC0603FR-07130KL" H 14400 7250 50  0001 C CNN "MPN"
@@
 F 0 "R177" H 13680 6754 50  0000 R CNN
 F 1 "4.7M" H 13680 6845 50  0000 R CNN
-F 2 "Resistors_SMD:R_0603_HandSoldering" V 13680 6800 50  0001 C CNN
+F 2 "Resistor_SMD:R_0603_1608Metric" V 13680 6800 50  0001 C CNN
 F 3 "~" H 13750 6800 50  0001 C CNN
 F 4 "RC0603FR-074M7L" H 13750 6800 50  0001 C CNN "MPN"
@@
 F 0 "R175" H 13280 6754 50  0000 R CNN
 F 1 "4.7M" H 13280 6845 50  0000 R CNN
-F 2 "Resistors_SMD:R_0603_HandSoldering" V 13280 6800 50  0001 C CNN
+F 2 "Resistor_SMD:R_0603_1608Metric" V 13280 6800 50  0001 C CNN
 F 3 "~" H 13350 6800 50  0001 C CNN
 F 4 "RC0603FR-074M7L" H 13350 6800 50  0001 C CNN "MPN"
@@
 F 0 "R176" H 13580 10804 50  0000 R CNN
 F 1 "10k" H 13580 10895 50  0000 R CNN
-F 2 "Resistors_SMD:R_0603_HandSoldering" V 13580 10850 50  0001 C CNN
+F 2 "Resistor_SMD:R_0603_1608Metric" V 13580 10850 50  0001 C CNN
 F 3 "~" H 13650 10850 50  0001 C CNN
 F 4 "RC0603FR-0710KL" H 13650 10850 50  0001 C CNN "MPN"
@@
 F 0 "R182" H 16830 6354 50  0000 R CNN
 F 1 "1" H 16830 6445 50  0000 R CNN
-F 2 "Resistors_SMD:R_0603_HandSoldering" V 16830 6400 50  0001 C CNN
+F 2 "Resistor_SMD:R_0603_1608Metric" V 16830 6400 50  0001 C CNN
 F 3 "~" H 16900 6400 50  0001 C CNN
 F 4 "RC0603FR-071RL" H 16900 6400 50  0001 C CNN "MPN"
@@
 F 0 "R180" H 16180 6804 50  0000 R CNN
 F 1 "1" H 16180 6895 50  0000 R CNN
-F 2 "Resistors_SMD:R_0603_HandSoldering" V 16180 6850 50  0001 C CNN
+F 2 "Resistor_SMD:R_0603_1608Metric" V 16180 6850 50  0001 C CNN
 F 3 "~" H 16250 6850 50  0001 C CNN
 F 4 "RC0603FR-071RL" H 16250 6850 50  0001 C CNN "MPN"
@@
 F 0 "C92" H 16050 7300 50  0000 L CNN
 F 1 "10u" H 16050 7400 50  0000 L CNN
-F 2 "Capacitors_SMD:C_0603_HandSoldering" H 16288 7200 50  0001 C CNN
+F 2 "Capacitor_SMD:C_0603_1608Metric" H 16288 7200 50  0001 C CNN
 F 3 "~" H 16250 7350 50  0001 C CNN
 F 4 "" H 16250 7350 50  0001 C CNN "Volatge"
@@
 F 0 "C93" H 16350 7300 50  0000 L CNN
 F 1 "10u" H 16350 7400 50  0000 L CNN
-F 2 "Capacitors_SMD:C_0603_HandSoldering" H 16588 7200 50  0001 C CNN
+F 2 "Capacitor_SMD:C_0603_1608Metric" H 16588 7200 50  0001 C CNN
 F 3 "~" H 16550 7350 50  0001 C CNN
 F 4 "" H 16550 7350 50  0001 C CNN "Volatge"
@@
 F 0 "R181" H 16480 6804 50  0000 R CNN
 F 1 "1" H 16480 6895 50  0000 R CNN
-F 2 "Resistors_SMD:R_0603_HandSoldering" V 16480 6850 50  0001 C CNN
+F 2 "Resistor_SMD:R_0603_1608Metric" V 16480 6850 50  0001 C CNN
 F 3 "~" H 16550 6850 50  0001 C CNN
 F 4 "RC0603FR-071RL" H 16550 6850 50  0001 C CNN "MPN"
@@
 F 0 "C94" H 17250 7300 50  0000 L CNN
 F 1 "10u" H 17250 7400 50  0000 L CNN
-F 2 "Capacitors_SMD:C_0603_HandSoldering" H 17488 7200 50  0001 C CNN
+F 2 "Capacitor_SMD:C_0603_1608Metric" H 17488 7200 50  0001 C CNN
 F 3 "~" H 17450 7350 50  0001 C CNN
 F 4 "" H 17450 7350 50  0001 C CNN "Volatge"
@@
 F 0 "C91" H 15400 7250 50  0000 L CNN
 F 1 "47n" H 15400 7350 50  0000 L CNN
-F 2 "Capacitors_SMD:C_0603_HandSoldering" H 15638 7150 50  0001 C CNN
+F 2 "Capacitor_SMD:C_0603_1608Metric" H 15638 7150 50  0001 C CNN
 F 3 "~" H 15600 7300 50  0001 C CNN
 F 4 "100V" H 15600 7300 50  0001 C CNN "Voltage"
@@
 F 0 "R174" H 11480 10104 50  0000 R CNN
 F 1 "1M" H 11480 10195 50  0000 R CNN
-F 2 "Resistors_SMD:R_0603_HandSoldering" V 11480 10150 50  0001 C CNN
+F 2 "Resistor_SMD:R_0603_1608Metric" V 11480 10150 50  0001 C CNN
 F 3 "~" H 11550 10150 50  0001 C CNN
 F 4 "RC0603JR-071ML" H 11550 10150 50  0001 C CNN "MPN"
@@
 F 0 "C88" H 11350 9750 50  0000 L CNN
 F 1 "2.2u" H 11350 9850 50  0000 L CNN
-F 2 "Capacitors_SMD:C_0603_HandSoldering" H 11588 9650 50  0001 C CNN
+F 2 "Capacitor_SMD:C_0603_1608Metric" H 11588 9650 50  0001 C CNN
 F 3 "~" H 11550 9800 50  0001 C CNN
 F 4 "50V" H 11550 9800 50  0001 C CNN "Volatge"
@@
 F 0 "R172" H 9830 9754 50  0000 R CNN
 F 1 "100" H 9830 9845 50  0000 R CNN
-F 2 "Resistors_SMD:R_0603_HandSoldering" V 9830 9800 50  0001 C CNN
+F 2 "Resistor_SMD:R_0603_1608Metric" V 9830 9800 50  0001 C CNN
 F 3 "~" H 9900 9800 50  0001 C CNN
 F 4 "RC0603FR-07100RL" H 9900 9800 50  0001 C CNN "MPN"
@@
 F 0 "R173" H 10730 9104 50  0000 R CNN
 F 1 "10k" H 10730 9195 50  0000 R CNN
-F 2 "Resistors_SMD:R_0603_HandSoldering" V 10730 9150 50  0001 C CNN
+F 2 "Resistor_SMD:R_0603_1608Metric" V 10730 9150 50  0001 C CNN
 F 3 "~" H 10800 9150 50  0001 C CNN
 F 4 "RC0603FR-0710KL" H 10800 9150 50  0001 C CNN "MPN"
@@
 F 0 "R178" H 14080 9054 50  0000 R CNN
 F 1 "10k" H 14080 9145 50  0000 R CNN
-F 2 "Resistors_SMD:R_0603_HandSoldering" V 14080 9100 50  0001 C CNN
+F 2 "Resistor_SMD:R_0603_1608Metric" V 14080 9100 50  0001 C CNN
 F 3 "~" H 14150 9100 50  0001 C CNN
 F 4 "RC0603FR-0710KL" H 14150 9100 50  0001 C CNN "MPN"
@@
 F 0 "R41" H 9180 8304 50  0000 R CNN
 F 1 "10k" H 9180 8395 50  0000 R CNN
-F 2 "Resistors_SMD:R_0603_HandSoldering" V 9180 8350 50  0001 C CNN
+F 2 "Resistor_SMD:R_0603_1608Metric" V 9180 8350 50  0001 C CNN
 F 3 "~" H 9250 8350 50  0001 C CNN
 F 4 "RC0603FR-0710KL" H 9250 8350 50  0001 C CNN "MPN"

Commit message: Schematics updates & improvements
Parts:
- removed D6: B220, Diode_SMD:D_SMB, symbol Diode:B220
- J13: value Charger 12V -> Charger; footprint Connectors_Molex:Molex_KK-6410-02_02x2.54mm_Straight -> ENNOID:Pin_1x02-XL
Changed lines of the file:
@@
 Wire Wire Line
 	8650 5800 8650 6400
-Wire Wire Line
-	8650 6400 10250 6400
 $Comp
 L BMS-Master-rescue:Conn_01x02-Connector_Generic-BMS-Master-rescue J13
@@
 P 8650 7550
 F 0 "J13" H 8729 7542 50  0000 L CNN
-F 1 "Charger 12V" H 8729 7451 50  0000 L CNN
-F 2 "Connectors_Molex:Molex_KK-6410-02_02x2.54mm_Straight" H 8650 7550 50  0001 C CNN
+F 1 "Charger" H 8729 7451 50  0000 L CNN
+F 2 "ENNOID:Pin_1x02-XL" H 8650 7550 50  0001 C CNN
 F 3 "~" H 8650 7550 50  0001 C CNN
 F 4 "282834-2 " H 8650 7550 50  0001 C CNN "MPN"
@@
 Wire Wire Line
 	8850 7650 8950 7650
-Wire Wire Line
-	10250 7550 10250 6400
-Connection ~ 10250 6400
 $Comp
 L BMS-Master-rescue:R-Device-BMS-Master-rescue R178
@@
 Wire Wire Line
 	13750 9800 14600 9800
-Wire Wire Line
-	9850 7550 10250 7550
-$Comp
-L Diode:B220 D6
-U 1 1 5D83524C
-P 9700 7550
-F 0 "D6" H 9700 7334 50  0000 C CNN
-F 1 "B220" H 9700 7425 50  0000 C CNN
-F 2 "Diode_SMD:D_SMB" H 9700 7375 50  0001 C CNN
-F 3 "http://www.jameco.com/Jameco/Products/ProdDS/1538777.pdf" H 9700 7550 50  0001 C CNN
-F 4 "N/A" H 9700 7550 50  0001 C CNN "MPN"
-	1    9700 7550
-	-1   0    0    1
-$EndComp
 Wire Wire Line
 	8850 7550 9250 7550
@@
 Wire Wire Line
 	9250 8200 9400 8200
-Connection ~ 9250 7550
-Wire Wire Line
-	9250 7550 9550 7550
 $Comp
 L BMS-Master-rescue:R-Device-BMS-Master-rescue R41
@@
 	17450 6400 17450 7200
 Wire Wire Line
-	10250 6400 11900 6400
+	17450 6400 18000 6400
 Wire Wire Line
-	17450 6400 18000 6400
+	8650 6400 11900 6400
+Text Label 14600 9100 0    50   ~ 0
+ChargeDetect
 $EndSCHEMATC
