File: Master/HV/PCB/switches.sch (KiCad schematic (older format))
At the start: 15 parts, among them Q3 BSS138, Q4 BUK98150-55A, Q5 BUK98150-55A, Q6 BUK98150-55A, Q7 BUK98150-55A

Commit message: maintenance update
Parts:
- R11, R23, R24, R25, R27, R28, R32, R33, R8: footprint Resistors_SMD:R_0603_HandSoldering -> Resistor_SMD:R_0603_1608Metric
- TH1: footprint Resistors_SMD:R_0805_HandSoldering -> Resistor_SMD:R_0805_2012Metric
Changed lines of the file:
@@
 F 0 "R24" V 12257 3750 50  0000 C CNN
 F 1 "10" V 12166 3750 50  0000 C CNN
-F 2 "Resistors_SMD:R_0603_HandSoldering" V 11980 3750 50  0001 C CNN
+F 2 "Resistor_SMD:R_0603_1608Metric" V 11980 3750 50  0001 C CNN
 F 3 "~" H 12050 3750 50  0001 C CNN
 F 4 "RC0603JR-0710RL" H 12050 3750 50  0001 C CNN "MPN"
@@
 F 0 "R23" V 12257 7500 50  0000 C CNN
 F 1 "10" V 12166 7500 50  0000 C CNN
-F 2 "Resistors_SMD:R_0603_HandSoldering" V 11980 7500 50  0001 C CNN
+F 2 "Resistor_SMD:R_0603_1608Metric" V 11980 7500 50  0001 C CNN
 F 3 "~" H 12050 7500 50  0001 C CNN
 F 4 "RC0603JR-0710RL" H 12050 7500 50  0001 C CNN "MPN"
@@
 F 0 "R25" V 12257 5550 50  0000 C CNN
 F 1 "10" V 12166 5550 50  0000 C CNN
-F 2 "Resistors_SMD:R_0603_HandSoldering" V 11980 5550 50  0001 C CNN
+F 2 "Resistor_SMD:R_0603_1608Metric" V 11980 5550 50  0001 C CNN
 F 3 "~" H 12050 5550 50  0001 C CNN
 F 4 "RC0603JR-0710RL" H 12050 5550 50  0001 C CNN "MPN"
@@
 F 0 "TH1" H 3147 9304 50  0000 R CNN
 F 1 "Thermistor_NTC 100K" H 3147 9395 50  0000 R CNN
-F 2 "Resistors_SMD:R_0805_HandSoldering" H 3300 9400 50  0001 C CNN
+F 2 "Resistor_SMD:R_0805_2012Metric" H 3300 9400 50  0001 C CNN
 F 3 "~" H 3300 9400 50  0001 C CNN
 F 4 "SDNT2012X104F4250FTF" H 3300 9350 50  0001 C CNN "MPN"
@@
 F 0 "R28" V 13157 5800 50  0000 C CNN
 F 1 "4.7M" V 13066 5800 50  0000 C CNN
-F 2 "Resistors_SMD:R_0603_HandSoldering" V 12880 5800 50  0001 C CNN
+F 2 "Resistor_SMD:R_0603_1608Metric" V 12880 5800 50  0001 C CNN
 F 3 "~" H 12950 5800 50  0001 C CNN
 F 4 "RC0603FR-074M7L" H 12950 5800 50  0001 C CNN "MPN"
@@
 F 0 "R27" V 13057 4000 50  0000 C CNN
 F 1 "4.7M" V 12966 4000 50  0000 C CNN
-F 2 "Resistors_SMD:R_0603_HandSoldering" V 12780 4000 50  0001 C CNN
+F 2 "Resistor_SMD:R_0603_1608Metric" V 12780 4000 50  0001 C CNN
 F 3 "~" H 12850 4000 50  0001 C CNN
 F 4 "RC0603FR-074M7L" H 12850 4000 50  0001 C CNN "MPN"
@@
 F 0 "R8" V 13157 7750 50  0000 C CNN
 F 1 "4.7M" V 13066 7750 50  0000 C CNN
-F 2 "Resistors_SMD:R_0603_HandSoldering" V 12880 7750 50  0001 C CNN
+F 2 "Resistor_SMD:R_0603_1608Metric" V 12880 7750 50  0001 C CNN
 F 3 "~" H 12950 7750 50  0001 C CNN
 F 4 "RC0603FR-074M7L" H 12950 7750 50  0001 C CNN "MPN"
@@
 F 0 "R11" V 4007 7300 50  0000 C CNN
 F 1 "10k" V 3916 7300 50  0000 C CNN
-F 2 "Resistors_SMD:R_0603_HandSoldering" V 3730 7300 50  0001 C CNN
+F 2 "Resistor_SMD:R_0603_1608Metric" V 3730 7300 50  0001 C CNN
 F 3 "~" H 3800 7300 50  0001 C CNN
 F 4 "RC0603FR-0710KL" H 3800 7300 50  0001 C CNN "MPN"
@@
 F 0 "R32" V 12257 1850 50  0000 C CNN
 F 1 "10" V 12166 1850 50  0000 C CNN
-F 2 "Resistors_SMD:R_0603_HandSoldering" V 11980 1850 50  0001 C CNN
+F 2 "Resistor_SMD:R_0603_1608Metric" V 11980 1850 50  0001 C CNN
 F 3 "~" H 12050 1850 50  0001 C CNN
 F 4 "RC0603JR-0710RL" H 12050 1850 50  0001 C CNN "MPN"
@@
 F 0 "R33" V 13057 2100 50  0000 C CNN
 F 1 "4.7M" V 12966 2100 50  0000 C CNN
-F 2 "Resistors_SMD:R_0603_HandSoldering" V 12780 2100 50  0001 C CNN
+F 2 "Resistor_SMD:R_0603_1608Metric" V 12780 2100 50  0001 C CNN
 F 3 "~" H 12850 2100 50  0001 C CNN
 F 4 "RC0603FR-074M7L" H 12850 2100 50  0001 C CNN "MPN"

Commit message: Schematics updates & improvements
Parts:
- added Q8: BUK98150-55A, Package_TO_SOT_SMD:SOT-223, symbol Device:Q_NMOS_GDSD
- added Q9: BSS138, TO_SOT_Packages_SMD:SOT-23, symbol Transistor_FET:BSS138
- added R45: 10, Resistor_SMD:R_0603_1608Metric, symbol BMS-Master-rescue:R-Device-BMS-Master-rescue
- added R47: 4.7M, Resistor_SMD:R_0603_1608Metric, symbol BMS-Master-rescue:R-Device-BMS-Master-rescue
Connections:
- net GND: now also Q8.3 (S), Q9.2 (S), R47.2
- net Precharge: now also Q8.2 (D), Q8.4 (D); no longer Q4.2 (D), Q4.4 (D)
- net PrechargeEnable: now also R45.1; no longer R24.1
- net Safety: now also Q9.1 (G)
- net Discharge renamed DischargePos
- net DischargeEnable renamed DischargePosEnable
- new net: Q8.1 (G), R45.2, R47.1
- new net DischargeNeg: Q4.2 (D), Q4.4 (D)
- new net DischargeNegEnable: Q9.3 (D), R24.1
Changed lines of the file:
@@
 $Descr A3 16535 11693
 encoding utf-8
-Sheet 5 7
+Sheet 7 7
 Title ""
 Date ""
@@
 ChargeEnable
 Text HLabel 14550 7150 2    50   Input ~ 0
-Discharge
+DischargePos
 Text HLabel 14550 3550 2    50   Input ~ 0
-Precharge
+DischargeNeg
 Text HLabel 14650 4950 2    50   Input ~ 0
 Charge
@@
 Wire Wire Line
 	3450 5050 5800 5050
-Wire Wire Line
-	5800 6500 5800 5050
 Connection ~ 5800 5050
 $Comp
@@
 	8600 7500 11900 7500
 Text HLabel 3450 5050 0    50   Input ~ 0
-DischargeEnable
+DischargePosEnable
 Text HLabel 3450 3750 0    50   Input ~ 0
-PrechargeEnable
+DischargeNegEnable
 $Comp
 L Device:Q_NMOS_GDSD Q4
@@
 	13600 7300 13500 7300
 Connection ~ 13500 7300
-Wire Wire Line
-	3450 3750 11900 3750
 Wire Wire Line
 	5800 5050 8600 5050
@@
 	13150 2450 13150 2350
 Wire Wire Line
-	3450 1850 11900 1850
-Wire Wire Line
 	13500 2050 13500 2350
 Wire Wire Line
@@
 Wire Wire Line
 	5250 6700 5250 7450
+Connection ~ 13175 9300
+Connection ~ 13625 8600
+Connection ~ 12875 8800
+$Comp
+L Device:Q_NMOS_GDSD Q8
+U 1 1 5E5898FF
+P 13425 8800
+F 0 "Q8" H 13713 8846 50  0000 L CNN
+F 1 "BUK98150-55A" H 13713 8755 50  0000 L CNN
+F 2 "Package_TO_SOT_SMD:SOT-223" H 13625 8900 50  0001 C CNN
+F 3 "~" H 13425 8800 50  0001 C CNN
+F 4 "BUK98150-55A/CUF" H 13425 8800 50  0001 C CNN "MPN"
+	1    13425 8800
+	1    0    0    -1
+$EndComp
+$Comp
+L BMS-Master-rescue:GND-power-BMS-Master-rescue #PWR0158
+U 1 1 5E58990C
+P 13175 9400
+F 0 "#PWR0158" H 13175 9150 50  0001 C CNN
+F 1 "GND" H 13180 9227 50  0000 C CNN
+F 2 "" H 13175 9400 50  0001 C CNN
+F 3 "" H 13175 9400 50  0001 C CNN
+	1    13175 9400
+	1    0    0    -1
+$EndComp
+$Comp
+L BMS-Master-rescue:R-Device-BMS-Master-rescue R45
+U 1 1 5E58991B
+P 12075 8800
+F 0 "R45" V 12282 8800 50  0000 C CNN
+F 1 "10" V 12191 8800 50  0000 C CNN
+F 2 "Resistor_SMD:R_0603_1608Metric" V 12005 8800 50  0001 C CNN
+F 3 "~" H 12075 8800 50  0001 C CNN
+F 4 "RC0603JR-0710RL" H 12075 8800 50  0001 C CNN "MPN"
+	1    12075 8800
+	0    -1   -1   0
+$EndComp
+$Comp
+L BMS-Master-rescue:R-Device-BMS-Master-rescue R47
+U 1 1 5E58992A
+P 12875 9050
+F 0 "R47" V 13082 9050 50  0000 C CNN
+F 1 "4.7M" V 12991 9050 50  0000 C CNN
+F 2 "Resistor_SMD:R_0603_1608Metric" V 12805 9050 50  0001 C CNN
+F 3 "~" H 12875 9050 50  0001 C CNN
+F 4 "RC0603FR-074M7L" H 12875 9050 50  0001 C CNN "MPN"
+	1    12875 9050
+	1    0    0    -1
+$EndComp
+Wire Wire Line
+	13175 9300 13525 9300
+Wire Wire Line
+	12875 8900 12875 8800
+Wire Wire Line
+	13175 9400 13175 9300
+Wire Wire Line
+	12875 9200 12875 9300
+Wire Wire Line
+	13625 8600 14575 8600
+Wire Wire Line
+	13525 8600 13625 8600
+Wire Wire Line
+	12875 9300 13175 9300
+Wire Wire Line
+	12225 8800 12875 8800
+Wire Wire Line
+	13525 9000 13525 9300
+Wire Wire Line
+	12875 8800 13225 8800
+Text HLabel 11775 8800 0    50   Input ~ 0
+PrechargeEnable
+Wire Wire Line
+	11775 8800 11925 8800
+Text HLabel 14575 8600 2    50   Input ~ 0
+Precharge
+Wire Wire Line
+	5800 5050 5800 6500
+Wire Wire Line
+	6800 6900 6800 7050
+$Comp
+L BMS-Master-rescue:GND-power-BMS-Master-rescue #PWR0159
+U 1 1 5E6109CD
+P 6800 7050
+F 0 "#PWR0159" H 6800 6800 50  0001 C CNN
+F 1 "GND" H 6805 6877 50  0000 C CNN
+F 2 "" H 6800 7050 50  0001 C CNN
+F 3 "" H 6800 7050 50  0001 C CNN
+	1    6800 7050
+	1    0    0    -1
+$EndComp
+$Comp
+L Transistor_FET:BSS138 Q9
+U 1 1 5E6109DD
+P 6700 6700
+F 0 "Q9" H 6906 6746 50  0000 L CNN
+F 1 "BSS138" H 6906 6655 50  0000 L CNN
+F 2 "TO_SOT_Packages_SMD:SOT-23" H 6900 6625 50  0001 L CIN
+F 3 "https://www.fairchildsemi.com/datasheets/BS/BSS138.pdf" H 6700 6700 50  0001 L CNN
+F 4 "BSS138" H 6700 6700 50  0001 C CNN "MPN"
+	1    6700 6700
+	1    0    0    -1
+$EndComp
+Wire Wire Line
+	5250 7450 6400 7450
+Wire Wire Line
+	6400 7450 6400 6700
+Wire Wire Line
+	6400 6700 6500 6700
+Connection ~ 5250 7450
+Wire Wire Line
+	3450 3750 6800 3750
+Wire Wire Line
+	3450 1850 11900 1850
+Wire Wire Line
+	6800 6500 6800 3750
+Connection ~ 6800 3750
+Wire Wire Line
+	6800 3750 11900 3750
 $EndSCHEMATC
