File: Master/HV/PCB/CAN.sch (KiCad schematic (older format))
At the start: 10 parts, among them U8 ISO1050DUBR, U9 SFH617A-2X009T

Commit message: maintenance update
Parts:
- C43, C45, C46: footprint Capacitors_SMD:C_0805_HandSoldering -> Capacitor_SMD:C_0805_2012Metric
- C44, C47: footprint Capacitors_SMD:C_0603_HandSoldering -> Capacitor_SMD:C_0603_1608Metric
- R115: footprint Resistors_SMD:R_0805_HandSoldering -> Resistor_SMD:R_0603_1608Metric
- R116: footprint Resistor_SMD:R_0603_1608Metric_Pad1.05x0.95mm_HandSolder -> Resistor_SMD:R_0603_1608Metric
Changed lines of the file:
@@
 F 0 "C44" H 3865 3546 50  0000 L CNN
 F 1 "100n" H 3865 3455 50  0000 L CNN
-F 2 "Capacitors_SMD:C_0603_HandSoldering" H 3788 3350 50  0001 C CNN
+F 2 "Capacitor_SMD:C_0603_1608Metric" H 3788 3350 50  0001 C CNN
 F 3 "~" H 3750 3500 50  0001 C CNN
 F 4 "GRM188R71E104KA01D" H 3750 3500 50  0001 C CNN "MPN"
@@
 F 0 "C43" H 3415 3546 50  0000 L CNN
 F 1 "1u" H 3415 3455 50  0000 L CNN
-F 2 "Capacitors_SMD:C_0805_HandSoldering" H 3338 3350 50  0001 C CNN
+F 2 "Capacitor_SMD:C_0805_2012Metric" H 3338 3350 50  0001 C CNN
 F 3 "~" H 3300 3500 50  0001 C CNN
 F 4 "GRM188R71E105KA12D" H 3300 3500 50  0001 C CNN "MPN"
@@
 F 0 "C47" V 6748 1850 50  0000 C CNN
 F 1 "100n" V 6839 1850 50  0000 C CNN
-F 2 "Capacitors_SMD:C_0603_HandSoldering" H 7038 1700 50  0001 C CNN
+F 2 "Capacitor_SMD:C_0603_1608Metric" H 7038 1700 50  0001 C CNN
 F 3 "~" H 7000 1850 50  0001 C CNN
 F 4 "GRM188R71E104KA01D" H 7000 1850 50  0001 C CNN "MPN"
@@
 F 0 "C46" H 6765 1896 50  0000 L CNN
 F 1 "1u" H 6765 1805 50  0000 L CNN
-F 2 "Capacitors_SMD:C_0805_HandSoldering" H 6688 1700 50  0001 C CNN
+F 2 "Capacitor_SMD:C_0805_2012Metric" H 6688 1700 50  0001 C CNN
 F 3 "~" H 6650 1850 50  0001 C CNN
 F 4 "GRM188R71E105KA12D" H 6650 1850 50  0001 C CNN "MPN"
@@
 F 0 "R115" V 5550 4000 50  0000 L CNN
 F 1 "4.7M" V 5450 4000 50  0000 L CNN
-F 2 "Resistors_SMD:R_0805_HandSoldering" V 5530 4300 50  0001 C CNN
+F 2 "Resistor_SMD:R_0603_1608Metric" V 5530 4300 50  0001 C CNN
 F 3 "~" H 5600 4300 50  0001 C CNN
 F 4 "RC0805JR-0710ML" H 5600 4300 50  0001 C CNN "MPN"
@@
 F 0 "C45" V 5350 4750 50  0000 C CNN
 F 1 "10n" V 5450 4800 50  0000 C CNN
-F 2 "Capacitors_SMD:C_0805_HandSoldering" H 5638 4800 50  0001 C CNN
+F 2 "Capacitor_SMD:C_0805_2012Metric" H 5638 4800 50  0001 C CNN
 F 3 "~" H 5600 4950 50  0001 C CNN
 F 4 "100V" V 5600 4950 50  0001 C CNN "Voltage"
@@
 F 0 "R116" V 6400 5700 50  0000 L CNN
 F 1 "2.2k" V 6300 5700 50  0000 L CNN
-F 2 "Resistor_SMD:R_0603_1608Metric_Pad1.05x0.95mm_HandSolder" V 6380 6000 50  0001 C CNN
+F 2 "Resistor_SMD:R_0603_1608Metric" V 6380 6000 50  0001 C CNN
 F 3 "~" H 6450 6000 50  0001 C CNN
 F 4 "RC0603JR-072K2L" H 6450 6000 50  0001 C CNN "MPN"

Commit message: Master-HV changes
Parts:
- removed C45: 10n, Capacitor_SMD:C_0805_2012Metric, symbol BMS-Master-rescue:C-Device-BMS-Master-rescue
- removed R115: 4.7M, Resistor_SMD:R_0603_1608Metric, symbol BMS-Master-rescue:R-Device-BMS-Master-rescue
- C43, C46: footprint Capacitor_SMD:C_0805_2012Metric -> Capacitor_SMD:C_0603_1608Metric
Changed lines of the file:
@@
 Wire Wire Line
 	5200 3650 5000 3650
-Wire Wire Line
-	5000 3650 5000 4300
-$Comp
-L BMS-Master-rescue:C-Device-BMS-Master-rescue C44
-U 1 1 5A91EB41
-P 3750 3500
-F 0 "C44" H 3865 3546 50  0000 L CNN
-F 1 "100n" H 3865 3455 50  0000 L CNN
-F 2 "Capacitor_SMD:C_0603_1608Metric" H 3788 3350 50  0001 C CNN
-F 3 "~" H 3750 3500 50  0001 C CNN
-F 4 "GRM188R71E104KA01D" H 3750 3500 50  0001 C CNN "MPN"
-	1    3750 3500
-	1    0    0    -1
-$EndComp
 $Comp
 L BMS-Master-rescue:+3.3V-power-BMS-Master-rescue #PWR0185
@@
 Text HLabel 7550 3450 2    50   Input ~ 0
 CANL
-Wire Wire Line
-	6000 3650 6000 4300
-$Comp
-L BMS-Master-rescue:C-Device-BMS-Master-rescue C43
-U 1 1 5A924642
-P 3300 3500
-F 0 "C43" H 3415 3546 50  0000 L CNN
-F 1 "1u" H 3415 3455 50  0000 L CNN
-F 2 "Capacitor_SMD:C_0805_2012Metric" H 3338 3350 50  0001 C CNN
-F 3 "~" H 3300 3500 50  0001 C CNN
-F 4 "GRM188R71E105KA12D" H 3300 3500 50  0001 C CNN "MPN"
-	1    3300 3500
-	1    0    0    -1
-$EndComp
 $Comp
 L BMS-Master-rescue:+3.3V-power-BMS-Master-rescue #PWR0187
@@
 Text HLabel 7700 1700 2    50   Input ~ 0
 5V_CAN
+Wire Wire Line
+	7700 1700 7000 1700
+Connection ~ 7000 1700
+Wire Wire Line
+	7000 1700 6650 1700
+Wire Wire Line
+	6650 1700 6200 1700
+Wire Wire Line
+	6200 1700 6200 3350
+Wire Wire Line
+	6200 3350 6000 3350
+Connection ~ 6650 1700
+Text Label 7350 2100 0    50   ~ 0
+CAN_GND
+Wire Wire Line
+	6650 2000 6650 2100
+Wire Wire Line
+	6650 2100 7000 2100
+Wire Wire Line
+	7000 2000 7000 2100
+Connection ~ 7000 2100
+Wire Wire Line
+	7000 2100 7350 2100
+Text Label 6100 5150 0    50   ~ 0
+CAN_GND
+Wire Wire Line
+	6000 5150 6100 5150
+Text HLabel 6050 5300 2    50   Input ~ 0
+CAN_GND
+Wire Wire Line
+	6050 5300 6000 5300
+Wire Wire Line
+	6000 5300 6000 5150
+Connection ~ 6000 5150
+$Comp
+L Power_Protection:SZNUP2105L D4
+U 1 1 5C258D40
+P 7000 3900
+F 0 "D4" H 7205 3946 50  0000 L CNN
+F 1 "SZNUP2105L" H 7205 3855 50  0000 L CNN
+F 2 "TO_SOT_Packages_SMD:SOT-23" H 7225 3850 50  0001 L CNN
+F 3 "http://www.onsemi.com/pub_link/Collateral/NUP2105L-D.PDF" H 7125 4025 50  0001 C CNN
+F 4 "SZNUP2105LT1G" H 7000 3900 50  0001 C CNN "MPN"
+	1    7000 3900
+	1    0    0    -1
+$EndComp
+Text Label 7150 4200 0    50   ~ 0
+CAN_GND
+Wire Wire Line
+	7000 4100 7000 4200
+Wire Wire Line
+	7000 4200 7150 4200
+Wire Notes Line
+	5650 2350 5650 6300
+Wire Notes Line
+	5550 2350 5550 6300
+$Comp
+L Isolator:SFH617A-2X017T U9
+U 1 1 5C25CD2F
+P 5600 6100
+F 0 "U9" H 5600 6425 50  0000 C CNN
+F 1 "SFH617A-2X009T" H 5600 6334 50  0000 C CNN
+F 2 "Housings_DIP:SMDIP-4_W9.53mm_Clearance8mm" H 5600 5750 50  0001 C CIN
+F 3 "http://www.vishay.com/docs/83740/sfh617a.pdf" H 5600 6050 50  0001 L CNN
+F 4 "SFH617A-2X009T" H 5600 6100 50  0001 C CNN "MPN"
+	1    5600 6100
+	-1   0    0    -1
+$EndComp
+$Comp
+L BMS-Master-rescue:GND-power-BMS-Master-rescue #PWR0189
+U 1 1 5C25DB56
+P 5100 6400
+F 0 "#PWR0189" H 5100 6150 50  0001 C CNN
+F 1 "GND" H 5105 6227 50  0000 C CNN
+F 2 "" H 5100 6400 50  0001 C CNN
+F 3 "" H 5100 6400 50  0001 C CNN
+	1    5100 6400
+	1    0    0    -1
+$EndComp
+Text HLabel 4300 6000 0    50   Input ~ 0
+EnableRequest
+Wire Wire Line
+	5300 6000 4300 6000
+Wire Wire Line
+	5300 6200 5100 6200
+Wire Wire Line
+	5100 6200 5100 6400
+$Comp
+L BMS-Master-rescue:R-Device-BMS-Master-rescue R116
+U 1 1 5C25FA4A
+P 6450 6000
+F 0 "R116" V 6400 5700 50  0000 L CNN
+F 1 "2.2k" V 6300 5700 50  0000 L CNN
+F 2 "Resistor_SMD:R_0603_1608Metric" V 6380 6000 50  0001 C CNN
+F 3 "~" H 6450 6000 50  0001 C CNN
+F 4 "RC0603JR-072K2L" H 6450 6000 50  0001 C CNN "MPN"
+	1    6450 6000
+	0    1    1    0
+$EndComp
+Wire Wire Line
+	5900 6000 6300 6000
+Text Label 6200 6200 0    50   ~ 0
+CAN_GND
+Wire Wire Line
+	5900 6200 6200 6200
+Text HLabel 7450 6000 2    50   Input ~ 0
+Enable_CAN
+Wire Wire Line
+	6600 6000 7450 6000
+Wire Wire Line
+	6000 3450 6900 3450
+Wire Wire Line
+	6000 3550 7100 3550
+Wire Wire Line
+	6900 3700 6900 3450
+Connection ~ 6900 3450
+Wire Wire Line
+	6900 3450 7550 3450
+Wire Wire Line
+	7100 3700 7100 3550
+Connection ~ 7100 3550
+Wire Wire Line
+	7100 3550 7550 3550
 $Comp
 L BMS-Master-rescue:C-Device-BMS-Master-rescue C47
@@
 F 0 "C46" H 6765 1896 50  0000 L CNN
 F 1 "1u" H 6765 1805 50  0000 L CNN
-F 2 "Capacitor_SMD:C_0805_2012Metric" H 6688 1700 50  0001 C CNN
+F 2 "Capacitor_SMD:C_0603_1608Metric" H 6688 1700 50  0001 C CNN
 F 3 "~" H 6650 1850 50  0001 C CNN
 F 4 "GRM188R71E105KA12D" H 6650 1850 50  0001 C CNN "MPN"
@@
 $EndComp
 $Comp
-L BMS-Master-rescue:R-Device-BMS-Master-rescue R115
-U 1 1 5C24E192
-P 5600 4300
-F 0 "R115" V 5550 4000 50  0000 L CNN
-F 1 "4.7M" V 5450 4000 50  0000 L CNN
-F 2 "Resistor_SMD:R_0603_1608Metric" V 5530 4300 50  0001 C CNN
-F 3 "~" H 5600 4300 50  0001 C CNN
-F 4 "RC0805JR-0710ML" H 5600 4300 50  0001 C CNN "MPN"
-	1    5600 4300
-	0    1    1    0
-$EndComp
-$Comp
-L BMS-Master-rescue:C-Device-BMS-Master-rescue C45
-U 1 1 5C24E7DA
-P 5600 4950
-F 0 "C45" V 5350 4750 50  0000 C CNN
-F 1 "10n" V 5450 4800 50  0000 C CNN
-F 2 "Capacitor_SMD:C_0805_2012Metric" H 5638 4800 50  0001 C CNN
-F 3 "~" H 5600 4950 50  0001 C CNN
-F 4 "100V" V 5600 4950 50  0001 C CNN "Voltage"
-F 5 "GRM188R71H103KA01D" H 5600 4950 50  0001 C CNN "MPN"
-	1    5600 4950
-	0    1    1    0
-$EndComp
-Wire Wire Line
-	5450 4300 5000 4300
-Connection ~ 5000 4300
-Wire Wire Line
-	5000 4300 5000 4950
-Wire Wire Line
-	5450 4950 5000 4950
-Connection ~ 5000 4950
-Wire Wire Line
-	5000 4950 5000 5150
-Wire Wire Line
-	5750 4950 6000 4950
-Wire Wire Line
-	5750 4300 6000 4300
-Connection ~ 6000 4300
-Wire Wire Line
-	6000 4300 6000 4950
-Wire Wire Line
-	7700 1700 7000 1700
-Connection ~ 7000 1700
-Wire Wire Line
-	7000 1700 6650 1700
-Wire Wire Line
-	6650 1700 6200 1700
-Wire Wire Line
-	6200 1700 6200 3350
-Wire Wire Line
-	6200 3350 6000 3350
-Connection ~ 6650 1700
-Wire Wire Line
-	6000 4950 6000 5150
-Connection ~ 6000 4950
-Text Label 7350 2100 0    50   ~ 0
-CAN_GND
-Wire Wire Line
-	6650 2000 6650 2100
-Wire Wire Line
-	6650 2100 7000 2100
-Wire Wire Line
-	7000 2000 7000 2100
-Connection ~ 7000 2100
-Wire Wire Line
-	7000 2100 7350 2100
-Text Label 6100 5150 0    50   ~ 0
-CAN_GND
-Wire Wire Line
-	6000 5150 6100 5150
-Text HLabel 6050 5300 2    50   Input ~ 0
-CAN_GND
-Wire Wire Line
-	6050 5300 6000 5300
-Wire Wire Line
-	6000 5300 6000 5150
-Connection ~ 6000 5150
-$Comp
-L Power_Protection:SZNUP2105L D4
-U 1 1 5C258D40
-P 7000 3900
-F 0 "D4" H 7205 3946 50  0000 L CNN
-F 1 "SZNUP2105L" H 7205 3855 50  0000 L CNN
-F 2 "TO_SOT_Packages_SMD:SOT-23" H 7225 3850 50  0001 L CNN
-F 3 "http://www.onsemi.com/pub_link/Collateral/NUP2105L-D.PDF" H 7125 4025 50  0001 C CNN
-F 4 "SZNUP2105LT1G" H 7000 3900 50  0001 C CNN "MPN"
-	1    7000 3900
-	1    0    0    -1
-$EndComp
-Text Label 7150 4200 0    50   ~ 0
-CAN_GND
-Wire Wire Line
-	7000 4100 7000 4200
-Wire Wire Line
-	7000 4200 7150 4200
-Wire Notes Line
-	5650 2350 5650 6300
-Wire Notes Line
-	5550 2350 5550 6300
-$Comp
-L Isolator:SFH617A-2X017T U9
-U 1 1 5C25CD2F
-P 5600 6100
-F 0 "U9" H 5600 6425 50  0000 C CNN
-F 1 "SFH617A-2X009T" H 5600 6334 50  0000 C CNN
-F 2 "Housings_DIP:SMDIP-4_W9.53mm_Clearance8mm" H 5600 5750 50  0001 C CIN
-F 3 "http://www.vishay.com/docs/83740/sfh617a.pdf" H 5600 6050 50  0001 L CNN
-F 4 "SFH617A-2X009T" H 5600 6100 50  0001 C CNN "MPN"
-	1    5600 6100
-	-1   0    0    -1
-$EndComp
-$Comp
-L BMS-Master-rescue:GND-power-BMS-Master-rescue #PWR0189
-U 1 1 5C25DB56
-P 5100 6400
-F 0 "#PWR0189" H 5100 6150 50  0001 C CNN
-F 1 "GND" H 5105 6227 50  0000 C CNN
-F 2 "" H 5100 6400 50  0001 C CNN
-F 3 "" H 5100 6400 50  0001 C CNN
-	1    5100 6400
-	1    0    0    -1
-$EndComp
-Text HLabel 4300 6000 0    50   Input ~ 0
-EnableRequest
-Wire Wire Line
-	5300 6000 4300 6000
-Wire Wire Line
-	5300 6200 5100 6200
-Wire Wire Line
-	5100 6200 5100 6400
-$Comp
-L BMS-Master-rescue:R-Device-BMS-Master-rescue R116
-U 1 1 5C25FA4A
-P 6450 6000
-F 0 "R116" V 6400 5700 50  0000 L CNN
-F 1 "2.2k" V 6300 5700 50  0000 L CNN
-F 2 "Resistor_SMD:R_0603_1608Metric" V 6380 6000 50  0001 C CNN
-F 3 "~" H 6450 6000 50  0001 C CNN
-F 4 "RC0603JR-072K2L" H 6450 6000 50  0001 C CNN "MPN"
-	1    6450 6000
-	0    1    1    0
-$EndComp
-Wire Wire Line
-	5900 6000 6300 6000
-Text Label 6200 6200 0    50   ~ 0
-CAN_GND
-Wire Wire Line
-	5900 6200 6200 6200
-Text HLabel 7450 6000 2    50   Input ~ 0
-Enable_CAN
-Wire Wire Line
-	6600 6000 7450 6000
-Wire Wire Line
-	6000 3450 6900 3450
-Wire Wire Line
-	6000 3550 7100 3550
-Wire Wire Line
-	6900 3700 6900 3450
-Connection ~ 6900 3450
-Wire Wire Line
-	6900 3450 7550 3450
-Wire Wire Line
-	7100 3700 7100 3550
-Connection ~ 7100 3550
-Wire Wire Line
-	7100 3550 7550 3550
+L BMS-Master-rescue:C-Device-BMS-Master-rescue C43
+U 1 1 5A924642
+P 3300 3500
+F 0 "C43" H 3415 3546 50  0000 L CNN
+F 1 "1u" H 3415 3455 50  0000 L CNN
+F 2 "Capacitor_SMD:C_0603_1608Metric" H 3338 3350 50  0001 C CNN
+F 3 "~" H 3300 3500 50  0001 C CNN
+F 4 "GRM188R71E105KA12D" H 3300 3500 50  0001 C CNN "MPN"
+	1    3300 3500
+	1    0    0    -1
+$EndComp
+$Comp
+L BMS-Master-rescue:C-Device-BMS-Master-rescue C44
+U 1 1 5A91EB41
+P 3750 3500
+F 0 "C44" H 3865 3546 50  0000 L CNN
+F 1 "100n" H 3865 3455 50  0000 L CNN
+F 2 "Capacitor_SMD:C_0603_1608Metric" H 3788 3350 50  0001 C CNN
+F 3 "~" H 3750 3500 50  0001 C CNN
+F 4 "GRM188R71E104KA01D" H 3750 3500 50  0001 C CNN "MPN"
+	1    3750 3500
+	1    0    0    -1
+$EndComp
+Wire Wire Line
+	5000 3650 5000 5150
+Wire Wire Line
+	6000 3650 6000 5150
 $EndSCHEMATC
