File: Master/HV/PCB/USB.sch (KiCad schematic (older format))
At the start: 12 parts, among them J14 SERIAL, Q26 BSS138, U7 CP2104

Commit message: maintenance update
Parts:
- C39, C40, C41, C42: footprint Capacitors_SMD:C_0603_HandSoldering -> Capacitor_SMD:C_0603_1608Metric
- R111, R112, R113, R114: footprint Resistors_SMD:R_0603_HandSoldering -> Resistor_SMD:R_0603_1608Metric
Changed lines of the file:
@@
 F 0 "R111" V 3850 3700 50  0000 C CNN
 F 1 "240" V 3850 3300 50  0000 C CNN
-F 2 "Resistors_SMD:R_0603_HandSoldering" V 3830 3500 50  0001 C CNN
+F 2 "Resistor_SMD:R_0603_1608Metric" V 3830 3500 50  0001 C CNN
 F 3 "~" H 3900 3500 50  0001 C CNN
 F 4 "RC0603FR-07240RL" H 3900 3500 50  0001 C CNN "MPN"
@@
 F 0 "R112" V 3850 3800 50  0000 C CNN
 F 1 "240" V 3850 3400 50  0000 C CNN
-F 2 "Resistors_SMD:R_0603_HandSoldering" V 3830 3600 50  0001 C CNN
+F 2 "Resistor_SMD:R_0603_1608Metric" V 3830 3600 50  0001 C CNN
 F 3 "~" H 3900 3600 50  0001 C CNN
 F 4 "RC0603FR-07240RL" H 3900 3600 50  0001 C CNN "MPN"
@@
 F 0 "R113" V 4000 4300 50  0000 C CNN
 F 1 "10k" V 4000 3900 50  0000 C CNN
-F 2 "Resistors_SMD:R_0603_HandSoldering" V 3980 4100 50  0001 C CNN
+F 2 "Resistor_SMD:R_0603_1608Metric" V 3980 4100 50  0001 C CNN
 F 3 "~" H 4050 4100 50  0001 C CNN
 F 4 "RC0603FR-0710KL" H 4050 4100 50  0001 C CNN "MPN"
@@
 F 0 "C40" H 6265 4646 50  0000 L CNN
 F 1 "2.2u" H 6265 4555 50  0000 L CNN
-F 2 "Capacitors_SMD:C_0603_HandSoldering" H 6188 4450 50  0001 C CNN
+F 2 "Capacitor_SMD:C_0603_1608Metric" H 6188 4450 50  0001 C CNN
 F 3 "~" H 6150 4600 50  0001 C CNN
 F 4 "GRM188R61A225KE34D" H 6150 4600 50  0001 C CNN "MPN"
@@
 F 0 "C39" H 4415 2096 50  0000 L CNN
 F 1 "2.2u" H 4415 2005 50  0000 L CNN
-F 2 "Capacitors_SMD:C_0603_HandSoldering" H 4338 1900 50  0001 C CNN
+F 2 "Capacitor_SMD:C_0603_1608Metric" H 4338 1900 50  0001 C CNN
 F 3 "~" H 4300 2050 50  0001 C CNN
 F 4 "GRM188R61A225KE34D" H 4300 2050 50  0001 C CNN "MPN"
@@
 F 0 "C42" H 6915 1946 50  0000 L CNN
 F 1 "2.2u" H 6915 1855 50  0000 L CNN
-F 2 "Capacitors_SMD:C_0603_HandSoldering" H 6838 1750 50  0001 C CNN
+F 2 "Capacitor_SMD:C_0603_1608Metric" H 6838 1750 50  0001 C CNN
 F 3 "~" H 6800 1900 50  0001 C CNN
 F 4 "GRM188R61A225KE34D" H 6800 1900 50  0001 C CNN "MPN"
@@
 F 0 "C41" H 6515 1946 50  0000 L CNN
 F 1 "100n" H 6515 1855 50  0000 L CNN
-F 2 "Capacitors_SMD:C_0603_HandSoldering" H 6438 1750 50  0001 C CNN
+F 2 "Capacitor_SMD:C_0603_1608Metric" H 6438 1750 50  0001 C CNN
 F 3 "~" H 6400 1900 50  0001 C CNN
 F 4 "GRM188R71E104KA01D" H 6400 1900 50  0001 C CNN "MPN"
@@
 F 0 "R114" H 7500 1950 50  0000 C CNN
 F 1 "10k" H 7500 1850 50  0000 C CNN
-F 2 "Resistors_SMD:R_0603_HandSoldering" V 7280 1900 50  0001 C CNN
+F 2 "Resistor_SMD:R_0603_1608Metric" V 7280 1900 50  0001 C CNN
 F 3 "~" H 7350 1900 50  0001 C CNN
 F 4 "RC0603FR-0710KL" H 7350 1900 50  0001 C CNN "MPN"

Commit message: New parts for precharge circuit
Parts:
- J14: MPN 282834-5 -> 70543-0004
Changed lines of the file:
@@
 F 2 "Connectors_Molex:Molex_KK-6410-05_05x2.54mm_Straight" H 3300 4700 50  0001 C CNN
 F 3 "" H 3300 4700 50  0001 C CNN
-F 4 "282834-5 " H 3300 4700 50  0001 C CNN "MPN"
+F 4 "70543-0004" H 3300 4700 50  0001 C CNN "MPN"
 	1    3300 4700
 	1    0    0    -1
