File: Master/HV/PCB/MCU.sch (KiCad schematic (older format))
At the start: 25 parts, among them J17 DEBUG, Q27 BSS138, U17 STM32F303CCTx, U2 LTC6820, Y1 8MHz

Commit message: maintenance update
Parts:
- C20, C6, C7, C76, C77, C78, C80, C81, C82, C83, C84: footprint Capacitors_SMD:C_0603_HandSoldering -> Capacitor_SMD:C_0603_1608Metric
- C8: footprint Capacitor_SMD:C_0603_1608Metric_Pad0.99x1.00mm_HandSolder -> Capacitor_SMD:C_0603_1608Metric
- R168, R170, R36, R37, R5, R6, R7: footprint Resistors_SMD:R_0603_HandSoldering -> Resistor_SMD:R_0603_1608Metric
Changed lines of the file:
@@
 F 0 "C77" H 7115 9446 50  0000 L CNN
 F 1 "18p" H 7115 9355 50  0000 L CNN
-F 2 "Capacitors_SMD:C_0603_HandSoldering" H 7038 9250 50  0001 C CNN
+F 2 "Capacitor_SMD:C_0603_1608Metric" H 7038 9250 50  0001 C CNN
 F 3 "~" H 7000 9400 50  0001 C CNN
 F 4 "50V" H 7000 9400 50  0001 C CNN "Voltage"
@@
 F 0 "C76" H 6115 9446 50  0000 L CNN
 F 1 "18p" H 6115 9355 50  0000 L CNN
-F 2 "Capacitors_SMD:C_0603_HandSoldering" H 6038 9250 50  0001 C CNN
+F 2 "Capacitor_SMD:C_0603_1608Metric" H 6038 9250 50  0001 C CNN
 F 3 "~" H 6000 9400 50  0001 C CNN
 F 4 "50V" H 6000 9400 50  0001 C CNN "Voltage"
@@
 F 0 "C78" H 7165 8396 50  0000 L CNN
 F 1 "100n" H 7165 8305 50  0000 L CNN
-F 2 "Capacitors_SMD:C_0603_HandSoldering" H 7088 8200 50  0001 C CNN
+F 2 "Capacitor_SMD:C_0603_1608Metric" H 7088 8200 50  0001 C CNN
 F 3 "~" H 7050 8350 50  0001 C CNN
 F 4 "GRM188R71E104KA01D" H 7050 8350 50  0001 C CNN "MPN"
@@
 F 0 "C80" H 20715 7441 50  0000 L CNN
 F 1 "100n" H 20715 7350 50  0000 L CNN
-F 2 "Capacitors_SMD:C_0603_HandSoldering" H 20638 7200 50  0001 C CNN
+F 2 "Capacitor_SMD:C_0603_1608Metric" H 20638 7200 50  0001 C CNN
 F 3 "~" H 20600 7350 50  0001 C CNN
 F 4 "25V" H 20715 7259 50  0000 L CNN "Voltage"
@@
 F 0 "C81" H 21315 7441 50  0000 L CNN
 F 1 "100n" H 21315 7350 50  0000 L CNN
-F 2 "Capacitors_SMD:C_0603_HandSoldering" H 21238 7200 50  0001 C CNN
+F 2 "Capacitor_SMD:C_0603_1608Metric" H 21238 7200 50  0001 C CNN
 F 3 "~" H 21200 7350 50  0001 C CNN
 F 4 "25V" H 21315 7259 50  0000 L CNN "Voltage"
@@
 F 0 "C82" H 21915 7441 50  0000 L CNN
 F 1 "100n" H 21915 7350 50  0000 L CNN
-F 2 "Capacitors_SMD:C_0603_HandSoldering" H 21838 7200 50  0001 C CNN
+F 2 "Capacitor_SMD:C_0603_1608Metric" H 21838 7200 50  0001 C CNN
 F 3 "~" H 21800 7350 50  0001 C CNN
 F 4 "25V" H 21915 7259 50  0000 L CNN "Voltage"
@@
 F 0 "C83" H 22515 7441 50  0000 L CNN
 F 1 "100n" H 22515 7350 50  0000 L CNN
-F 2 "Capacitors_SMD:C_0603_HandSoldering" H 22438 7200 50  0001 C CNN
+F 2 "Capacitor_SMD:C_0603_1608Metric" H 22438 7200 50  0001 C CNN
 F 3 "~" H 22400 7350 50  0001 C CNN
 F 4 "25V" H 22515 7259 50  0000 L CNN "Voltage"
@@
 F 0 "C84" H 24215 9641 50  0000 L CNN
 F 1 "100n" H 24215 9550 50  0000 L CNN
-F 2 "Capacitors_SMD:C_0603_HandSoldering" H 24138 9400 50  0001 C CNN
+F 2 "Capacitor_SMD:C_0603_1608Metric" H 24138 9400 50  0001 C CNN
 F 3 "~" H 24100 9550 50  0001 C CNN
 F 4 "25V" H 24215 9459 50  0000 L CNN "Voltage"
@@
 F 0 "R168" H 7120 7846 50  0000 L CNN
 F 1 "10k" H 7120 7755 50  0000 L CNN
-F 2 "Resistors_SMD:R_0603_HandSoldering" V 6980 7800 50  0001 C CNN
+F 2 "Resistor_SMD:R_0603_1608Metric" V 6980 7800 50  0001 C CNN
 F 3 "~" H 7050 7800 50  0001 C CNN
 F 4 "RC0603FR-0710KL" H 7050 7800 50  0001 C CNN "MPN"
@@
 F 0 "R170" H 24670 9596 50  0000 L CNN
 F 1 "100k" H 24670 9505 50  0000 L CNN
-F 2 "Resistors_SMD:R_0603_HandSoldering" V 24530 9550 50  0001 C CNN
+F 2 "Resistor_SMD:R_0603_1608Metric" V 24530 9550 50  0001 C CNN
 F 3 "~" H 24600 9550 50  0001 C CNN
 F 4 "RC0603JR-07100KL" H 24600 9550 50  0001 C CNN "MPN"
@@
 F 0 "R36" V 15750 2900 50  0000 C CNN
 F 1 "1.2k" V 15534 2900 50  0000 C CNN
-F 2 "Resistors_SMD:R_0603_HandSoldering" V 15580 2900 50  0001 C CNN
+F 2 "Resistor_SMD:R_0603_1608Metric" V 15580 2900 50  0001 C CNN
 F 3 "~" H 15650 2900 50  0001 C CNN
 F 4 "RC0603JR-071K2L" H 15650 2900 50  0001 C CNN "MPN"
@@
 F 0 "R5" V 15200 2900 50  0000 C CNN
 F 1 "806" V 14984 2900 50  0000 C CNN
-F 2 "Resistors_SMD:R_0603_HandSoldering" V 15030 2900 50  0001 C CNN
+F 2 "Resistor_SMD:R_0603_1608Metric" V 15030 2900 50  0001 C CNN
 F 3 "~" H 15100 2900 50  0001 C CNN
 F 4 "RC0603FR-07806RL" H 15100 2900 50  0001 C CNN "MPN"
@@
 F 0 "C20" H 17135 4004 50  0000 R CNN
 F 1 "1u" H 17135 4095 50  0000 R CNN
-F 2 "Capacitors_SMD:C_0603_HandSoldering" H 17288 3900 50  0001 C CNN
+F 2 "Capacitor_SMD:C_0603_1608Metric" H 17288 3900 50  0001 C CNN
 F 3 "~" H 17250 4050 50  0001 C CNN
 F 4 "GRM188R71E105KA12D" H 17250 4050 50  0001 C CNN "MPN"
@@
 F 0 "R37" V 17743 2950 50  0000 C CNN
 F 1 "2k" V 17834 2950 50  0000 C CNN
-F 2 "Resistors_SMD:R_0603_HandSoldering" V 17880 2950 50  0001 C CNN
+F 2 "Resistor_SMD:R_0603_1608Metric" V 17880 2950 50  0001 C CNN
 F 3 "~" H 17950 2950 50  0001 C CNN
 F 4 "RC0603FR-072KL" H 17950 2950 50  0001 C CNN "MPN"
@@
 F 0 "R6" V 15450 2200 50  0000 C CNN
 F 1 "51" V 15234 2200 50  0000 C CNN
-F 2 "Resistors_SMD:R_0603_HandSoldering" V 15280 2200 50  0001 C CNN
+F 2 "Resistor_SMD:R_0603_1608Metric" V 15280 2200 50  0001 C CNN
 F 3 "~" H 15350 2200 50  0001 C CNN
 F 4 "RC0603JR-0751RL" H 15350 2200 50  0001 C CNN "MPN"
@@
 F 0 "R7" V 15450 2600 50  0000 C CNN
 F 1 "51" V 15234 2600 50  0000 C CNN
-F 2 "Resistors_SMD:R_0603_HandSoldering" V 15280 2600 50  0001 C CNN
+F 2 "Resistor_SMD:R_0603_1608Metric" V 15280 2600 50  0001 C CNN
 F 3 "~" H 15350 2600 50  0001 C CNN
 F 4 "RC0603JR-0751RL" H 15350 2600 50  0001 C CNN "MPN"
@@
 F 0 "C7" H 14735 2354 50  0000 R CNN
 F 1 "10n" H 14735 2445 50  0000 R CNN
-F 2 "Capacitors_SMD:C_0603_HandSoldering" H 14888 2250 50  0001 C CNN
+F 2 "Capacitor_SMD:C_0603_1608Metric" H 14888 2250 50  0001 C CNN
 F 3 "~" H 14850 2400 50  0001 C CNN
 F 4 "GRM188R71H103KA01D" H 14850 2400 50  0001 C CNN "MPN"
@@
 F 0 "C6" H 14185 2354 50  0000 R CNN
 F 1 "10n" H 14185 2445 50  0000 R CNN
-F 2 "Capacitors_SMD:C_0603_HandSoldering" H 14338 2250 50  0001 C CNN
+F 2 "Capacitor_SMD:C_0603_1608Metric" H 14338 2250 50  0001 C CNN
 F 3 "~" H 14300 2400 50  0001 C CNN
 F 4 "GRM188R71H103KA01D" H 14300 2400 50  0001 C CNN "MPN"
@@
 F 0 "C8" H 18015 4141 50  0000 L CNN
 F 1 "100n" H 18015 4050 50  0000 L CNN
-F 2 "Capacitor_SMD:C_0603_1608Metric_Pad0.99x1.00mm_HandSolder" H 17938 3900 50  0001 C CNN
+F 2 "Capacitor_SMD:C_0603_1608Metric" H 17938 3900 50  0001 C CNN
 F 3 "~" H 17900 4050 50  0001 C CNN
 F 4 "25V" H 18015 3959 50  0001 L CNN "Voltage"

Commit message: Schematics updates & improvements
Connections:
- net CoolingEnable: now also U17.20 (PB2/ADC2_IN12/ADC3_EXTI2/ADC4_EXTI2/COMP4_INM/OPAMP3_VINM/OPAMP3_VINM_SEC/TSC_G3_IO4); no longer U17.4 (PC15/ADC1_EXTI15/ADC2_EXTI15/RCC_OSC32_OUT)
- net PreChargeEnable: now also U17.4 (PC15/ADC1_EXTI15/ADC2_EXTI15/RCC_OSC32_OUT); no longer U17.22 (PB11/ADC1_EXTI11/ADC2_EXTI11/COMP6_INP/OPAMP4_VINP/OPAMP4_VINP_SEC/TIM2_CH4/TSC_G6_IO1/USART3_RX)
- net DischargeEnable renamed DischargePosEnable
- new net DischargeNegEnable: U17.22 (PB11/ADC1_EXTI11/ADC2_EXTI11/COMP6_INP/OPAMP4_VINP/OPAMP4_VINP_SEC/TIM2_CH4/TSC_G6_IO1/USART3_RX)
- no-connect marks 3 -> 4
Changed lines of the file:
@@
 $Descr A1 33110 23386
 encoding utf-8
-Sheet 6 7
+Sheet 5 7
 Title ""
 Date ""
@@
 Text HLabel 24450 10000 2    50   Input ~ 0
 RX_USB
-Text HLabel 9100 9300 0    50   Input ~ 0
+Text HLabel 8525 9300 0    50   Input ~ 0
 Safety
 Wire Wire Line
@@
 	6000 9550 6000 9600
 Wire Wire Line
-	9100 9300 9200 9300
+	8525 9300 9200 9300
 Text HLabel 7200 9950 0    50   BiDi ~ 0
 ChargeDetect
 Wire Wire Line
-	9200 9400 8600 9400
+	9200 9400 8125 9400
 Wire Wire Line
 	7000 9100 9200 9100
@@
 $EndComp
 Wire Wire Line
-	8600 9200 8600 9400
+	8125 9200 8125 9400
 Text HLabel 8950 10800 0    50   Input ~ 0
-PreChargeEnable
-Wire Wire Line
-	9200 10800 8950 10800
+DischargeNegEnable
 Text HLabel 8950 10700 0    50   Input ~ 0
-DischargeEnable
-Wire Wire Line
-	8950 10700 9200 10700
+DischargePosEnable
 Text HLabel 8950 10200 0    50   Input ~ 0
 PowerEnable
@@
 	8950 10300 9200 10300
 Wire Wire Line
-	7800 9200 8600 9200
+	7800 9200 8125 9200
 Wire Wire Line
 	7800 9600 7800 9650
@@
 Text Label 24450 10100 0    50   ~ 0
 SS
+Text HLabel 8950 9900 0    50   Input ~ 0
+CoolingEnable
+Wire Wire Line
+	8950 9900 9200 9900
 Text HLabel 8950 9500 0    50   Input ~ 0
-CoolingEnable
+PreChargeEnable
 Wire Wire Line
 	8950 9500 9200 9500
+Wire Wire Line
+	8950 10700 9200 10700
+Wire Wire Line
+	8950 10800 9200 10800
+NoConn ~ 9200 10600
 $EndSCHEMATC

Commit message: Schematic Master-HV minor change
DischargeNeg has been switched to precharge for better code compatibility
Connections:
- net DischargeNegEnable: now also U17.4 (PC15/ADC1_EXTI15/ADC2_EXTI15/RCC_OSC32_OUT); no longer U17.22 (PB11/ADC1_EXTI11/ADC2_EXTI11/COMP6_INP/OPAMP4_VINP/OPAMP4_VINP_SEC/TIM2_CH4/TSC_G6_IO1/USART3_RX)
- net PreChargeEnable: now also U17.22 (PB11/ADC1_EXTI11/ADC2_EXTI11/COMP6_INP/OPAMP4_VINP/OPAMP4_VINP_SEC/TIM2_CH4/TSC_G6_IO1/USART3_RX); no longer U17.4 (PC15/ADC1_EXTI15/ADC2_EXTI15/RCC_OSC32_OUT)
Changed lines of the file:
@@
 Wire Wire Line
 	8125 9200 8125 9400
-Text HLabel 8950 10800 0    50   Input ~ 0
-DischargeNegEnable
 Text HLabel 8950 10700 0    50   Input ~ 0
 DischargePosEnable
@@
 Wire Wire Line
 	8950 9900 9200 9900
-Text HLabel 8950 9500 0    50   Input ~ 0
-PreChargeEnable
 Wire Wire Line
 	8950 9500 9200 9500
@@
 	8950 10800 9200 10800
 NoConn ~ 9200 10600
+Text HLabel 8950 10800 0    50   Input ~ 0
+PreChargeEnable
+Text HLabel 8950 9500 0    50   Input ~ 0
+DischargeNegEnable
 $EndSCHEMATC
