File: Slaves/LTC6811/12W/PCB/LTC6811.sch (KiCad schematic (older format))
At the start: 52 parts, among them J1 Cells, J2 Slave, J3 Master, J4 Temp, J5 Conn_01x01, J6 Conn_01x01, J8 Conn_01x01, Q1 NSV1C201MZ4, U1 LTC6811-1

Commit message: Readme changes
Parts:
- added C10, C11, C8, C9: 100n, Capacitors_SMD:C_0603_HandSoldering, symbol Device:C
- added R60, R61, R62, R63: 100k, Resistors_SMD:R_0603_HandSoldering, symbol Device:R
Connections:
- net GND: now also C10.2, C11.2, C8.2, C9.2
- net T2: now also C8.1, R60.1
- net T3: now also C9.1, R61.1
- net T4: now also C10.1, R62.1
- net T5: now also C11.1, R63.1
- net Vref2: now also R60.2, R61.2, R62.2, R63.2
Other:
- moved on the sheet: C12, R11, TH1

Commit message: Datasheet update for V1.0
Parts:
- added J7: Conn_01x01, Mounting_Holes:MountingHole_3.2mm_M3_ISO7380_Pad, symbol Connector_Generic:Conn_01x01
- C1, C2, C25, C26, C5: MPN (none) -> CL21B105KBFNNNE
- C10, C11, C12, C3, C4, C8, C9: MPN (none) -> CC0603KRX7R0BB104
- C6, C7: MPN (none) -> CL10C101JB8NNNC
- D13, D14: MPN (none) -> 1N4148W-7-F
- D15: MPN (none) -> BZT52H-C62,115
- D16: MPN (none) -> SML-D12P8WT86C
- F1, F10, F11, F12, F13, F2, F3, F4, F5, F6, F7, F8, F9, J5, J6, J8, LOGO1: MPN (none) -> N/A
- J2, J3: MPN (none) -> 282834-2
- R1, R2, R5, R6: MPN (none) -> RC0603FR-07100RL
- R10, R4: MPN (none) -> RC0603JR-071K2L
- R11, R60, R61, R62, R63: MPN (none) -> RC0603JR-07100KL
- R3: value 806 -> 1K; MPN (none) -> MCR03EZPFX1001
- R7: MPN (none) -> RC0603JR-071ML
- TH1: MPN (none) -> SDNT2012X104F4250FTF
- TR1: MPN (none) -> HM2102NLT
- U1: MPN (none) -> LTC6811HG-1#PBF
Connections:
- net Vref2: now also J4.6 (Pin_6)
- net Vreg: no longer J4.6 (Pin_6)
- no-connect marks 7 -> 8

Commit message: LV-BMS design started
Parts:
- R3: value 1K -> 1.2k
- R4: value 1.2k -> 806
Changed lines of the file:
@@
 P 8000 4450
 F 0 "R3" V 8050 4600 50  0000 L CNN
-F 1 "1K" V 8050 4200 50  0000 L CNN
+F 1 "1.2k" V 8050 4200 50  0000 L CNN
 F 2 "Resistors_SMD:R_0603_HandSoldering" V 7930 4450 50  0001 C CNN
 F 3 "~" H 8000 4450 50  0001 C CNN
@@
 P 8600 4450
 F 0 "R4" V 8650 4600 50  0000 L CNN
-F 1 "1.2k" V 8650 4150 50  0000 L CNN
+F 1 "806" V 8650 4150 50  0000 L CNN
 F 2 "Resistors_SMD:R_0603_HandSoldering" V 8530 4450 50  0001 C CNN
 F 3 "~" H 8600 4450 50  0001 C CNN

Commit message: maintenance update
Parts:
- removed J4: Temp, Pin_Headers:Pin_Header_Angled_1x06_Pitch2.54mm, symbol Connector_Generic:Conn_01x06
- removed JP1: ~Last?, Pin_Headers:Pin_Header_Straight_1x02_Pitch2.54mm, symbol Device:Jumper
- added J4: Temp, Connector_PinHeader_2.54mm:PinHeader_1x05_P2.54mm_Horizontal, symbol Connector:Conn_01x05_Male
- C1, C2, C25, C26, C5: footprint Capacitors_SMD:C_0805_HandSoldering -> Capacitor_SMD:C_0805_2012Metric
- C10, C11, C12, C3, C4, C6, C7, C8, C9: footprint Capacitors_SMD:C_0603_HandSoldering -> Capacitor_SMD:C_0603_1608Metric
- D13, D14, D15: footprint Diodes_SMD:D_SOD-123 -> Diode_SMD:D_SOD-123
- D16: footprint LED_SMD:LED_0603_1608Metric_Pad1.05x0.95mm_HandSolder -> LED_SMD:LED_0603_1608Metric
- FB1: footprint Resistors_SMD:R_0603_HandSoldering -> Resistor_SMD:R_0603_1608Metric; MPN (none) -> BLM18PG330SN1D
- J1: MPN (none) -> N/A
- J2, J3: footprint Connectors_Molex:Molex_KK-6410-02_02x2.54mm_Straight -> ENNOID:Pin_1x02-XL; MPN 282834-2 -> 70543-0001
- Q1: MPN (none) -> NSV1C201MZ4T1G
- R1, R10, R11, R2, R5, R6, R60, R61, R62, R63, R7: footprint Resistors_SMD:R_0603_HandSoldering -> Resistor_SMD:R_0603_1608Metric
- R3: footprint Resistors_SMD:R_0603_HandSoldering -> Resistor_SMD:R_0603_1608Metric; MPN MCR03EZPFX1001 -> RC0603JR-071K2L
- R4: footprint Resistors_SMD:R_0603_HandSoldering -> Resistor_SMD:R_0603_1608Metric; MPN RC0603JR-071K2L -> RC0603FR-07806RL
- R8, R9: footprint Resistors_SMD:R_0603_HandSoldering -> Resistor_SMD:R_0603_1608Metric; MPN (none) -> RC0603JR-070RL
- TH1: footprint Resistors_SMD:R_0805_HandSoldering -> Resistor_SMD:R_0805_2012Metric
Connections:
- net GND: now also J4.1 (Pin_1)
- net IPB: now also TR1.7
- net T2: now also J4.2 (Pin_2)
- net T3: now also J4.3 (Pin_3)
- net T4: now also J4.4 (Pin_4)
- net T5: now also J4.5 (Pin_5)
- net at TR1.1: now also J3.1 (Pin_1); no longer J3.2 (Pin_2)
- net at TR1.3: now also J3.2 (Pin_2); no longer J3.1 (Pin_1)
- net at TR1.4: now also J2.1 (Pin_1); no longer J2.2 (Pin_2)
- net at TR1.6: now also J2.2 (Pin_2); no longer J2.1 (Pin_1)

Commit message: Schematics updates & improvements
Parts:
- J2: value Slave -> PB MB
- J3: value Master -> PA MA
Changed lines of the file:
@@
 P 13700 2150
 F 0 "J3" H 13780 2142 50  0000 L CNN
-F 1 "Master" H 13780 2051 50  0000 L CNN
+F 1 "PA MA" H 13780 2051 50  0000 L CNN
 F 2 "ENNOID:Pin_1x02-XL" H 13700 2150 50  0001 C CNN
 F 3 "~" H 13700 2150 50  0001 C CNN
@@
 P 13700 1450
 F 0 "J2" H 13780 1442 50  0000 L CNN
-F 1 "Slave" H 13780 1351 50  0000 L CNN
+F 1 "PB MB" H 13780 1351 50  0000 L CNN
 F 2 "ENNOID:Pin_1x02-XL" H 13700 1450 50  0001 C CNN
 F 3 "~" H 13700 1450 50  0001 C CNN
