File: Slaves/LTC6811/12W/PCB/cell.sch (KiCad schematic (older format))
At the start: 7 parts, among them Q2 TSM2323

Commit message: Datasheet update for V1.0
Parts:
- C13: footprint Capacitors_SMD:C_0805_HandSoldering -> Capacitor_SMD:C_0603_1608Metric_Pad0.99x1.00mm_HandSolder; MPN (none) -> CC0603KRX7R0BB104
- D1: MPN (none) -> PDZ7.5BZ
- R13: MPN (none) -> RC0603FR-07100RL
Changed lines of the file:
@@
 $Descr A4 11693 8268
 encoding utf-8
-Sheet 2 13
+Sheet 12 13
 Title ""
 Date ""
@@
 Comment3 ""
 Comment4 ""
-Comment5 ""
-Comment6 ""
-Comment7 ""
-Comment8 ""
-Comment9 ""
 $EndDescr
 $Comp
@@
 F 2 "Resistors_SMD:R_0603_HandSoldering" V 4580 2700 50  0001 C CNN
 F 3 "~" H 4650 2700 50  0001 C CNN
+F 4 "RC0603FR-07100RL" H 4650 2700 50  0001 C CNN "MPN"
 	1    4650 2700
 	0    1    1    0
@@
 F 0 "C24" H 5515 3996 50  0000 L CNN
 F 1 "100n" H 5515 3905 50  0000 L CNN
-F 2 "Capacitors_SMD:C_0805_HandSoldering" H 5438 3800 50  0001 C CNN
+F 2 "Capacitor_SMD:C_0603_1608Metric_Pad0.99x1.00mm_HandSolder" H 5438 3800 50  0001 C CNN
 F 3 "~" H 5400 3950 50  0001 C CNN
+F 4 "CC0603KRX7R0BB104" H 5400 3950 50  0001 C CNN "MPN"
 	1    5400 3950
 	1    0    0    -1
@@
 F 2 "Diode_SMD:D_SOD-323_HandSoldering" H 6000 3300 50  0001 C CNN
 F 3 "~" H 6000 3300 50  0001 C CNN
+F 4 "PDZ7.5BZ" H 6000 3300 50  0001 C CNN "MPN"
 	1    6000 3300
 	0    1    1    0

Commit message: LV-BMS design started
Changed lines of the file:
@@
 $Descr A4 11693 8268
 encoding utf-8
-Sheet 12 13
+Sheet 2 13
 Title ""
 Date ""
@@
 AR Path="/5C4FFA3D/5D2EBE6E" Ref="R?"  Part="1"
 AR Path="/5C4FFA43/5D2EBE6E" Ref="R?"  Part="1"
-F 0 "R46" V 4443 2700 50  0000 C CNN
+F 0 "R13" V 4443 2700 50  0000 C CNN
 F 1 "100" V 4534 2700 50  0000 C CNN
 F 2 "Resistors_SMD:R_0603_HandSoldering" V 4580 2700 50  0001 C CNN
@@
 AR Path="/5C4FFA3D/5D2EBE7D" Ref="R?"  Part="1"
 AR Path="/5C4FFA43/5D2EBE7D" Ref="R?"  Part="1"
-F 0 "R47" V 4443 3350 50  0000 C CNN
+F 0 "R14" V 4443 3350 50  0000 C CNN
 F 1 "3.3k" V 4534 3350 50  0000 C CNN
 F 2 "Resistors_SMD:R_0603_HandSoldering" V 4580 3350 50  0001 C CNN
@@
 AR Path="/5C4FFA3D/5D2EBE8A" Ref="Q?"  Part="1"
 AR Path="/5C4FFA43/5D2EBE8A" Ref="Q?"  Part="1"
-F 0 "Q13" H 4105 3304 50  0000 L CNN
+F 0 "Q2" H 4105 3304 50  0000 L CNN
 F 1 "TSM2323" H 4105 3395 50  0000 L CNN
 F 2 "TO_SOT_Packages_SMD:SOT-23" H 4100 3450 50  0001 C CNN
@@
 AR Path="/5C4FFA3D/5D2EBE98" Ref="R?"  Part="1"
 AR Path="/5C4FFA43/5D2EBE98" Ref="R?"  Part="1"
-F 0 "R45" H 3730 3954 50  0000 R CNN
+F 0 "R12" H 3730 3954 50  0000 R CNN
 F 1 "15" H 3730 4045 50  0000 R CNN
 F 2 "Resistors_SMD:R_2512" V 3730 4000 50  0001 C CNN
@@
 AR Path="/5C4FFA3D/5D2EBE9F" Ref="C?"  Part="1"
 AR Path="/5C4FFA43/5D2EBE9F" Ref="C?"  Part="1"
-F 0 "C24" H 5515 3996 50  0000 L CNN
+F 0 "C13" H 5515 3996 50  0000 L CNN
 F 1 "100n" H 5515 3905 50  0000 L CNN
 F 2 "Capacitor_SMD:C_0603_1608Metric_Pad0.99x1.00mm_HandSolder" H 5438 3800 50  0001 C CNN
@@
 AR Path="/5C4FFA3D/5D2EBEAA" Ref="#PWR?"  Part="1"
 AR Path="/5C4FFA43/5D2EBEAA" Ref="#PWR?"  Part="1"
-F 0 "#PWR0120" H 5400 3950 50  0001 C CNN
+F 0 "#PWR0109" H 5400 3950 50  0001 C CNN
 F 1 "GND" H 5405 4027 50  0000 C CNN
 F 2 "" H 5400 4200 50  0001 C CNN
@@
 AR Path="/5C4FFA31/5D2EBEB0" Ref="D11"  Part="1"
 AR Path="/5C4FFA37/5D2EBEB0" Ref="D12"  Part="1"
-F 0 "D12" V 5954 3379 50  0000 L CNN
+F 0 "D1" V 5954 3379 50  0000 L CNN
 F 1 "PDZ7.5B" V 6045 3379 50  0000 L CNN
 F 2 "Diode_SMD:D_SOD-323_HandSoldering" H 6000 3300 50  0001 C CNN
@@
 AR Path="/5C4FFA3D/5D2EBEBA" Ref="R?"  Part="1"
 AR Path="/5C4FFA43/5D2EBEBA" Ref="R?"  Part="1"
-F 0 "R59" H 3480 3954 50  0000 R CNN
+F 0 "R48" H 3480 3954 50  0000 R CNN
 F 1 "15" H 3480 4045 50  0000 R CNN
 F 2 "Resistors_SMD:R_2512" V 3480 4000 50  0001 C CNN

Commit message: maintenance update
Parts:
- removed R48: 15, Resistors_SMD:R_2512, symbol Device:R
- C13: footprint Capacitor_SMD:C_0603_1608Metric_Pad0.99x1.00mm_HandSolder -> Capacitor_SMD:C_0603_1608Metric
- D1: footprint Diode_SMD:D_SOD-323_HandSoldering -> Diode_SMD:D_SOD-323
- Q2: MPN (none) -> TSM2323CX RFG
- R12: value 15 -> 36; footprint Resistors_SMD:R_2512 -> Resistor_SMD:R_2512_6332Metric; MPN (none) -> RTT25360JTE
- R13: footprint Resistors_SMD:R_0603_HandSoldering -> Resistor_SMD:R_0603_1608Metric
- R14: footprint Resistors_SMD:R_0603_HandSoldering -> Resistor_SMD:R_0603_1608Metric; MPN (none) -> RC0603JR-073K3L
Changed lines of the file:
@@
 $Descr A4 11693 8268
 encoding utf-8
-Sheet 2 13
+Sheet 9 13
 Title ""
 Date ""
@@
 AR Path="/5C4FFA3D/5D2EBE6E" Ref="R?"  Part="1"
 AR Path="/5C4FFA43/5D2EBE6E" Ref="R?"  Part="1"
-F 0 "R13" V 4443 2700 50  0000 C CNN
+F 0 "R34" V 4443 2700 50  0000 C CNN
 F 1 "100" V 4534 2700 50  0000 C CNN
-F 2 "Resistors_SMD:R_0603_HandSoldering" V 4580 2700 50  0001 C CNN
+F 2 "Resistor_SMD:R_0603_1608Metric" V 4580 2700 50  0001 C CNN
 F 3 "~" H 4650 2700 50  0001 C CNN
 F 4 "RC0603FR-07100RL" H 4650 2700 50  0001 C CNN "MPN"
@@
 AR Path="/5C4FFA3D/5D2EBE7D" Ref="R?"  Part="1"
 AR Path="/5C4FFA43/5D2EBE7D" Ref="R?"  Part="1"
-F 0 "R14" V 4443 3350 50  0000 C CNN
+F 0 "R35" V 4443 3350 50  0000 C CNN
 F 1 "3.3k" V 4534 3350 50  0000 C CNN
-F 2 "Resistors_SMD:R_0603_HandSoldering" V 4580 3350 50  0001 C CNN
+F 2 "Resistor_SMD:R_0603_1608Metric" V 4580 3350 50  0001 C CNN
 F 3 "~" H 4650 3350 50  0001 C CNN
+F 4 "RC0603JR-073K3L" H 4650 3350 50  0001 C CNN "MPN"
 	1    4650 3350
 	0    1    1    0
@@
 AR Path="/5C4FFA3D/5D2EBE8A" Ref="Q?"  Part="1"
 AR Path="/5C4FFA43/5D2EBE8A" Ref="Q?"  Part="1"
-F 0 "Q2" H 4105 3304 50  0000 L CNN
+F 0 "Q9" H 4105 3304 50  0000 L CNN
 F 1 "TSM2323" H 4105 3395 50  0000 L CNN
 F 2 "TO_SOT_Packages_SMD:SOT-23" H 4100 3450 50  0001 C CNN
 F 3 "~" H 3900 3350 50  0001 C CNN
+F 4 "TSM2323CX RFG " H 3900 3350 50  0001 C CNN "MPN"
 	1    3900 3350
 	-1   0    0    1
@@
 AR Path="/5C4FFA3D/5D2EBE98" Ref="R?"  Part="1"
 AR Path="/5C4FFA43/5D2EBE98" Ref="R?"  Part="1"
-F 0 "R12" H 3730 3954 50  0000 R CNN
-F 1 "15" H 3730 4045 50  0000 R CNN
-F 2 "Resistors_SMD:R_2512" V 3730 4000 50  0001 C CNN
+F 0 "R33" H 3730 3954 50  0000 R CNN
+F 1 "36" H 3730 4045 50  0000 R CNN
+F 2 "Resistor_SMD:R_2512_6332Metric" V 3730 4000 50  0001 C CNN
 F 3 "~" H 3800 4000 50  0001 C CNN
+F 4 "RTT25360JTE" H 3800 4000 50  0001 C CNN "MPN"
 	1    3800 4000
 	-1   0    0    1
 $EndComp
-Wire Wire Line
-	3800 3550 3800 3750
 Text HLabel 5100 3350 2    50   Input ~ 0
 S
@@
 AR Path="/5C4FFA3D/5D2EBE9F" Ref="C?"  Part="1"
 AR Path="/5C4FFA43/5D2EBE9F" Ref="C?"  Part="1"
-F 0 "C13" H 5515 3996 50  0000 L CNN
+F 0 "C20" H 5515 3996 50  0000 L CNN
 F 1 "100n" H 5515 3905 50  0000 L CNN
-F 2 "Capacitor_SMD:C_0603_1608Metric_Pad0.99x1.00mm_HandSolder" H 5438 3800 50  0001 C CNN
+F 2 "Capacitor_SMD:C_0603_1608Metric" H 5438 3800 50  0001 C CNN
 F 3 "~" H 5400 3950 50  0001 C CNN
 F 4 "CC0603KRX7R0BB104" H 5400 3950 50  0001 C CNN "MPN"
@@
 AR Path="/5C4FFA3D/5D2EBEAA" Ref="#PWR?"  Part="1"
 AR Path="/5C4FFA43/5D2EBEAA" Ref="#PWR?"  Part="1"
-F 0 "#PWR0109" H 5400 3950 50  0001 C CNN
+F 0 "#PWR0116" H 5400 3950 50  0001 C CNN
 F 1 "GND" H 5405 4027 50  0000 C CNN
 F 2 "" H 5400 4200 50  0001 C CNN
@@
 Wire Wire Line
 	3800 4150 3800 4350
-Wire Wire Line
-	3800 4350 3550 4350
 $Comp
 L Device:D_Zener D1
@@
 AR Path="/5C4FFA31/5D2EBEB0" Ref="D11"  Part="1"
 AR Path="/5C4FFA37/5D2EBEB0" Ref="D12"  Part="1"
-F 0 "D1" V 5954 3379 50  0000 L CNN
+F 0 "D8" V 5954 3379 50  0000 L CNN
 F 1 "PDZ7.5B" V 6045 3379 50  0000 L CNN
-F 2 "Diode_SMD:D_SOD-323_HandSoldering" H 6000 3300 50  0001 C CNN
+F 2 "Diode_SMD:D_SOD-323" H 6000 3300 50  0001 C CNN
 F 3 "~" H 6000 3300 50  0001 C CNN
 F 4 "PDZ7.5BZ" H 6000 3300 50  0001 C CNN "MPN"
@@
 Wire Wire Line
 	6000 4250 6250 4250
-$Comp
-L Device:R R48
-U 1 1 5D2EBEBA
-P 3550 4000
-AR Path="/5C4F59F4/5D2EBEBA" Ref="R48"  Part="1"
-AR Path="/5C4FCBE0/5D2EBEBA" Ref="R49"  Part="1"
-AR Path="/5C4FCED2/5D2EBEBA" Ref="R50"  Part="1"
-AR Path="/5C4FCED8/5D2EBEBA" Ref="R51"  Part="1"
-AR Path="/5C4FD32A/5D2EBEBA" Ref="R52"  Part="1"
-AR Path="/5C4FD330/5D2EBEBA" Ref="R53"  Part="1"
-AR Path="/5C4FD336/5D2EBEBA" Ref="R54"  Part="1"
-AR Path="/5C4FD33C/5D2EBEBA" Ref="R55"  Part="1"
-AR Path="/5C4FFA25/5D2EBEBA" Ref="R56"  Part="1"
-AR Path="/5C4FFA2B/5D2EBEBA" Ref="R57"  Part="1"
-AR Path="/5C4FFA31/5D2EBEBA" Ref="R58"  Part="1"
-AR Path="/5C4FFA37/5D2EBEBA" Ref="R59"  Part="1"
-AR Path="/5C4FFA3D/5D2EBEBA" Ref="R?"  Part="1"
-AR Path="/5C4FFA43/5D2EBEBA" Ref="R?"  Part="1"
-F 0 "R48" H 3480 3954 50  0000 R CNN
-F 1 "15" H 3480 4045 50  0000 R CNN
-F 2 "Resistors_SMD:R_2512" V 3480 4000 50  0001 C CNN
-F 3 "~" H 3550 4000 50  0001 C CNN
-	1    3550 4000
-	-1   0    0    1
-$EndComp
-Wire Wire Line
-	3550 3850 3550 3750
-Wire Wire Line
-	3550 3750 3800 3750
-Connection ~ 3800 3750
-Wire Wire Line
-	3800 3750 3800 3850
-Wire Wire Line
-	3550 4150 3550 4350
-Connection ~ 3550 4350
-Wire Wire Line
-	3550 4350 2850 4350
+Wire Wire Line
+	2850 4350 3800 4350
+Wire Wire Line
+	3800 3550 3800 3850
 $EndSCHEMATC

Commit message: Schematics updates & improvements
Changed lines of the file:
@@
 AR Path="/5C4FFA3D/5D2EBE6E" Ref="R?"  Part="1"
 AR Path="/5C4FFA43/5D2EBE6E" Ref="R?"  Part="1"
-F 0 "R34" V 4443 2700 50  0000 C CNN
+F 0 "R46" V 4443 2700 50  0000 C CNN
 F 1 "100" V 4534 2700 50  0000 C CNN
 F 2 "Resistor_SMD:R_0603_1608Metric" V 4580 2700 50  0001 C CNN
@@
 AR Path="/5C4FFA3D/5D2EBE7D" Ref="R?"  Part="1"
 AR Path="/5C4FFA43/5D2EBE7D" Ref="R?"  Part="1"
-F 0 "R35" V 4443 3350 50  0000 C CNN
+F 0 "R47" V 4443 3350 50  0000 C CNN
 F 1 "3.3k" V 4534 3350 50  0000 C CNN
 F 2 "Resistor_SMD:R_0603_1608Metric" V 4580 3350 50  0001 C CNN
@@
 AR Path="/5C4FFA3D/5D2EBE8A" Ref="Q?"  Part="1"
 AR Path="/5C4FFA43/5D2EBE8A" Ref="Q?"  Part="1"
-F 0 "Q9" H 4105 3304 50  0000 L CNN
+F 0 "Q13" H 4105 3304 50  0000 L CNN
 F 1 "TSM2323" H 4105 3395 50  0000 L CNN
 F 2 "TO_SOT_Packages_SMD:SOT-23" H 4100 3450 50  0001 C CNN
@@
 AR Path="/5C4FFA3D/5D2EBE98" Ref="R?"  Part="1"
 AR Path="/5C4FFA43/5D2EBE98" Ref="R?"  Part="1"
-F 0 "R33" H 3730 3954 50  0000 R CNN
+F 0 "R45" H 3730 3954 50  0000 R CNN
 F 1 "36" H 3730 4045 50  0000 R CNN
 F 2 "Resistor_SMD:R_2512_6332Metric" V 3730 4000 50  0001 C CNN
@@
 AR Path="/5C4FFA3D/5D2EBE9F" Ref="C?"  Part="1"
 AR Path="/5C4FFA43/5D2EBE9F" Ref="C?"  Part="1"
-F 0 "C20" H 5515 3996 50  0000 L CNN
+F 0 "C24" H 5515 3996 50  0000 L CNN
 F 1 "100n" H 5515 3905 50  0000 L CNN
 F 2 "Capacitor_SMD:C_0603_1608Metric" H 5438 3800 50  0001 C CNN
@@
 AR Path="/5C4FFA3D/5D2EBEAA" Ref="#PWR?"  Part="1"
 AR Path="/5C4FFA43/5D2EBEAA" Ref="#PWR?"  Part="1"
-F 0 "#PWR0116" H 5400 3950 50  0001 C CNN
+F 0 "#PWR0120" H 5400 3950 50  0001 C CNN
 F 1 "GND" H 5405 4027 50  0000 C CNN
 F 2 "" H 5400 4200 50  0001 C CNN
@@
 AR Path="/5C4FFA31/5D2EBEB0" Ref="D11"  Part="1"
 AR Path="/5C4FFA37/5D2EBEB0" Ref="D12"  Part="1"
-F 0 "D8" V 5954 3379 50  0000 L CNN
+F 0 "D12" V 5954 3379 50  0000 L CNN
 F 1 "PDZ7.5B" V 6045 3379 50  0000 L CNN
 F 2 "Diode_SMD:D_SOD-323" H 6000 3300 50  0001 C CNN
